File: BMS_20S/BMS_20S.kicad_pcb (KiCad board)
At the start: 2 copper layers, 242.8 x 149.9 mm, 931 parts, among them J101 IN, J102 OUT, J2101 TEMP_IDC_26_CONN, J401 VOLT_IDC_26_CONN, Q2001 Si2302DS, Q2002 Si2302DS, Q201 BC558, Q3401 Si2302DS, Q3402 Si2302DS, Q3403 Si2302DS, Q3404 Si2302DS, Q3501 Si2302DS, Q3502 Si2302DS, Q3503 Si2302DS, Q3504 Si2302DS, Q3601 Si2302DS, Q3602 Si2302DS, Q3603 Si2302DS, Q3604 Si2302DS, Q3701 Si2302DS, Q3702 Si2302DS, Q3703 Si2302DS, Q3704 Si2302DS, Q3803 Si2302DS, Q3804 Si2302DS, U1001 LM324, U101 74HC595, U102 74HC4051, U103 74HC4051, U104 74HC4051, U1101 LM324, U1201 LM324, U1301 LM324, U1901 TS1851ILT, U1902 TS1851ILT, U1903 TLP290-4, U2001 TS1851ILT, U2002 TS1851ILT, U2003 TLP290-4, U2004 TLP290-4, U201 TL431LP, U202 LM324, U203 TL431LP, U204 TL431LP, U2101 TS1851ILT, U2102 TS1851ILT, U2103 TLP290-4, U2201 TS1851ILT, U2202 TS1851ILT, U2203 TLP290-4, U2301 TS1851ILT, U2302 TS1851ILT, U2303 TLP290-4, U2401 TS1851ILT, U2402 TS1851ILT, U2403 TLP290-4, U2501 TS1851ILT, U2502 TS1851ILT, U2503 TLP290-4, U2601 TS1851ILT, U2602 TS1851ILT, U2603 TLP290-4, U2701 TS1851ILT, U2702 TS1851ILT, U2703 TLP290-4, U2801 TS1851ILT, U2802 TS1851ILT, U2803 TLP290-4, U301 LMC7660, U302 LMC7660, U303 LM317_3PinPackage, U304 LMC7660, U305 LMC7660, U3401 TLP290-4, U3501 TLP290-4, U3601 TLP290-4, U3701 TLP290-4, U501 LM324, U601 LM324, U701 LM324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

Commit message: add e-Power_conventions file
Parts:
- added R314: 0R, Resistor_SMD:R_0805_2012Metric, F.Cu at (359.4, 186.7)
Changed lines of the file:
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@@
     (tracks 6094)
     (zones 0)
-    (modules 931)
+    (modules 932)
     (nets 635)
   )
@@
     (0 F.Cu signal)
     (31 B.Cu signal)
-    (32 B.Adhes user hide)
+    (32 B.Adhes user)
     (33 F.Adhes user)
-    (34 B.Paste user hide)
-    (35 F.Paste user hide)
-    (36 B.SilkS user hide)
-    (37 F.SilkS user hide)
-    (38 B.Mask user hide)
-    (39 F.Mask user hide)
+    (34 B.Paste user)
+    (35 F.Paste user)
+    (36 B.SilkS user)
+    (37 F.SilkS user)
+    (38 B.Mask user)
+    (39 F.Mask user)
     (40 Dwgs.User user)
     (41 Cmts.User user)
-    (42 Eco1.User user hide)
+    (42 Eco1.User user)
     (43 Eco2.User user)
     (44 Edge.Cuts user)
     (45 Margin user)
     (46 B.CrtYd user)
-    (47 F.CrtYd user hide)
-    (48 B.Fab user hide)
-    (49 F.Fab user hide)
+    (47 F.CrtYd user)
+    (48 B.Fab user)
+    (49 F.Fab user)
   )
   (setup
-    (last_trace_width 0.25)
+    (last_trace_width 0.3)
     (user_trace_width 0.3)
     (user_trace_width 0.35)
@@
     (solder_mask_min_width 0.25)
     (aux_axis_origin 157.48 201.676)
-    (visible_elements 7FF9F7FF)
+    (visible_elements 7FFFFFFF)
     (pcbplotparams
       (layerselection 0x010fc_ffffffff)
@@
     (add_net "Net-(U305-Pad7)")
   )
+  (module Resistor_SMD:R_0805_2012Metric (layer F.Cu)
+    (at 359.41 186.69)
+    (descr "Resistor SMD 0805 (2012 Metric), square (rectangular) end terminal, IPC_7351 nominal, (Body size source: https://docs.google.com/spreadsheets/d/1BsfQQcO9C6DZCsRaXUlFlo91Tg2WpOkGARC1WS5S8t0/edit?usp=sharing), generated with kicad-footprint-generator")
+    (tags resistor)
+    (attr smd)
+    (fp_text reference R314 (at 0 -1.65) (layer F.Cu)
+      (effects (font (size 1 1) (thickness 0.15)))
+    )
+    (fp_text value 0R (at 0 1.65) (layer F.Fab)
+      (effects (font (size 1 1) (thickness 0.15)))
+    )
+    (fp_line (start -1 0.6) (end -1 -0.6) (layer F.Fab) (width 0.1))
+    (fp_line (start -1 -0.6) (end 1 -0.6) (layer F.Fab) (width 0.1))
+    (fp_line (start 1 -0.6) (end 1 0.6) (layer F.Fab) (width 0.1))
+    (fp_line (start 1 0.6) (end -1 0.6) (layer F.Fab) (width 0.1))
+    (fp_line (start -0.258578 -0.71) (end 0.258578 -0.71) (layer F.SilkS) (width 0.12))
+    (fp_line (start -0.258578 0.71) (end 0.258578 0.71) (layer F.SilkS) (width 0.12))
+    (fp_line (start -1.68 0.95) (end -1.68 -0.95) (layer F.CrtYd) (width 0.05))
+    (fp_line (start -1.68 -0.95) (end 1.68 -0.95) (layer F.CrtYd) (width 0.05))
+    (fp_line (start 1.68 -0.95) (end 1.68 0.95) (layer F.CrtYd) (width 0.05))
+    (fp_line (start 1.68 0.95) (end -1.68 0.95) (layer F.CrtYd) (width 0.05))
+    (fp_text user %R (at 0 0) (layer F.Fab)
+      (effects (font (size 0.5 0.5) (thickness 0.08)))
+    )
+    (pad 1 smd roundrect (at -0.9375 0) (size 0.975 1.4) (layers F.Cu F.Paste F.Mask) (roundrect_rratio 0.25)
+      (net 596 "Net-(J2101-Pad10)"))
+    (pad 2 smd roundrect (at 0.9375 0) (size 0.975 1.4) (layers F.Cu F.Paste F.Mask) (roundrect_rratio 0.25)
+      (net 51 "/Temperature Sensors/0V"))
+    (model ${KISYS3DMOD}/Resistor_SMD.3dshapes/R_0805_2012Metric.wrl
+      (at (xyz 0 0 0))
+      (scale (xyz 1 1 1))
+      (rotate (xyz 0 0 0))
+    )
+  )
   (module "e-Power:SOIC-16_4.55x10.3mm_P1.27mm(TLP290-4)" (layer B.Cu)

Commit message: rounded corners
Parts:
- removed J101: IN, e-Power:DSUB-9_Female_EdgeMount_P2.77mm
- removed J102: OUT, e-Power:DSUB-9_Female_EdgeMount_P2.77mm
- added C104: 100nF, Capacitor_SMD:C_0805_2012Metric, F.Cu at (384.2, 119.4)
- added C105: 100nF, Capacitor_SMD:C_0805_2012Metric, F.Cu at (379.8, 119.4)
- added C106: 100nF, Capacitor_SMD:C_0805_2012Metric, F.Cu at (379.8, 122.3)
- added C107: 100nF, Capacitor_SMD:C_0805_2012Metric, F.Cu at (370.6, 127.3)
- added C108: 100nF, Capacitor_SMD:C_0805_2012Metric, F.Cu at (367.1, 131.3)
- added C109: 100nF, Capacitor_SMD:C_0805_2012Metric, F.Cu at (362.7, 131.3)
- added C3201: 100nF, Capacitor_SMD:C_0805_2012Metric, F.Cu at (348.8, 155.1)
- added C3202: 100nF, Capacitor_SMD:C_0805_2012Metric, F.Cu at (353.2, 152.2)
- added D301: 1N5819, Diode_SMD:D_SOD-323_HandSoldering, F.Cu at (393.0, 111.4)
- added G***: LOGO, e-Power:Logo_e-Power_41.3x20.0mm_Copper, F.Cu at (348.2, 171.1)
- added G***: LOGO, e-Power:Logo_UFRGS_22.0x12.0mm_Silk, F.Cu at (264.9, 190.2)
- added G***: LOGO, e-Power:Logo_UFRGS_22.0x12.0mm_Copper, F.Cu at (265.0, 190.4)
- added J3201: Current_Conn, Connector_PinHeader_2.54mm:PinHeader_1x04_P2.54mm_Horizontal, F.Cu at (357.9, 140.8)
- added J3202: BSPD_Conn, Connector_PinHeader_2.54mm:PinHeader_1x04_P2.54mm_Horizontal, F.Cu at (344.5, 140.8)
- added JP3201: jumper, e-Power:zero_ohm_resistor_0805, F.Cu at (357.9, 151.8)
- added R101: 1K, Resistor_SMD:R_0805_2012Metric, F.Cu at (375.0, 127.3)
- added R102: 1K, Resistor_SMD:R_0805_2012Metric, F.Cu at (371.5, 130.3)
- added R103: 1K, Resistor_SMD:R_0805_2012Metric, F.Cu at (379.8, 125.3)
- added R104: 1K, Resistor_SMD:R_0805_2012Metric, F.Cu at (371.5, 133.2)
- added R105: 1K, Resistor_SMD:R_0805_2012Metric, F.Cu at (384.2, 122.3)
- added R106: 1K, Resistor_SMD:R_0805_2012Metric, F.Cu at (375.9, 130.3)
- added R3201: 10K, Resistor_SMD:R_0805_2012Metric, F.Cu at (344.4, 152.2)
- added R3202: 10K, Resistor_SMD:R_0805_2012Metric, F.Cu at (371.2, 150.1)
- added R3203: 10K, Resistor_SMD:R_0805_2012Metric, F.Cu at (344.4, 155.1)
- added R3204: 10K, Resistor_SMD:R_0805_2012Metric, F.Cu at (348.8, 152.2)
- added U104: 74HC4051, Package_SO:SOP-16_4.4x10.4mm_P1.27mm, F.Cu at (355.9, 127.9)
- added U105: 74HC4051, Package_SO:SOP-16_4.4x10.4mm_P1.27mm, F.Cu at (365.0, 115.9)
- added U106: 74HC4051, Package_SO:SOP-16_4.4x10.4mm_P1.27mm, F.Cu at (355.9, 115.9)
- added U107: 74HC595, Package_SO:SOP-16_4.4x10.4mm_P1.27mm, F.Cu at (346.7, 127.9)
- added U108: 74HC595, Package_SO:SOP-16_4.4x10.4mm_P1.27mm, F.Cu at (346.7, 115.9)
- added U3201: LM324, Package_SO:SOIC-14_3.9x8.7mm_P1.27mm, F.Cu at (373.2, 143.6)
- H101, H102, H103, H104: footprint MountingHole:MountingHole_4.3mm_M4_Pad_Via -> e-Power:MountingHole_3.2mm_M3_Pad_Via
- R2701: renamed from R3401; value 390R -> 330R
- R2702: renamed from R3402; value 390R -> 330R
- R2703: renamed from R3403; value 390R -> 330R
- R2704: renamed from R3404; value 390R -> 330R
- R2705: renamed from R3405; value 390R -> 330R
- R2706: renamed from R3406; value 390R -> 330R
- R2707: renamed from R3407; value 390R -> 330R
- R2708: renamed from R3408; value 390R -> 330R
- R2745: renamed from R3457; value 390R -> 330R
- R2746: renamed from R3458; value 390R -> 330R
- R2747: renamed from R3459; value 390R -> 330R
- R2748: renamed from R3460; value 390R -> 330R
- R2801: renamed from R3501; value 390R -> 330R
- R2802: renamed from R3502; value 390R -> 330R
- R2803: renamed from R3503; value 390R -> 330R
- R2804: renamed from R3504; value 390R -> 330R
- R2805: renamed from R3505; value 390R -> 330R
- R2806: renamed from R3506; value 390R -> 330R
- R2807: renamed from R3507; value 390R -> 330R
- R2808: renamed from R3508; value 390R -> 330R
- R2845: renamed from R3557; value 390R -> 330R
- R2846: renamed from R3558; value 390R -> 330R
- R2847: renamed from R3559; value 390R -> 330R
- R2848: renamed from R3560; value 390R -> 330R
- R2901: renamed from R3601; value 390R -> 330R
- R2902: renamed from R3602; value 390R -> 330R
- R2903: renamed from R3603; value 390R -> 330R
- R2904: renamed from R3604; value 390R -> 330R
- R2905: renamed from R3605; value 390R -> 330R
- R2906: renamed from R3606; value 390R -> 330R
- R2907: renamed from R3607; value 390R -> 330R
- R2908: renamed from R3608; value 390R -> 330R
- R2945: renamed from R3657; value 390R -> 330R
- R2946: renamed from R3658; value 390R -> 330R
- R2947: renamed from R3659; value 390R -> 330R
- R2948: renamed from R3660; value 390R -> 330R
- R3001: renamed from R3701; value 390R -> 330R
- R3002: renamed from R3702; value 390R -> 330R
- R3003: renamed from R3703; value 390R -> 330R
- R3004: renamed from R3704; value 390R -> 330R
- R3005: renamed from R3705; value 390R -> 330R
- R3006: renamed from R3706; value 390R -> 330R
- R3007: renamed from R3707; value 390R -> 330R
- R3008: renamed from R3708; value 390R -> 330R
- R3045: renamed from R3757; value 390R -> 330R
- R3046: renamed from R3758; value 390R -> 330R
- R3047: renamed from R3759; value 390R -> 330R
- R3048: renamed from R3760; value 390R -> 330R
- R3101: renamed from R2014; value 390R -> 330R
- R3102: renamed from R2018; value 390R -> 330R
- R3103: renamed from R3803; value 390R -> 330R
- R3104: renamed from R3804; value 390R -> 330R
- R3105: renamed from R2019; value 390R -> 330R
- R3106: renamed from R2020; value 390R -> 330R
- R3107: renamed from R3807; value 390R -> 330R
- R3108: renamed from R3808; value 390R -> 330R
- R3145: renamed from R2039; value 390R -> 330R
- R3146: renamed from R2040; value 390R -> 330R
- R3147: renamed from R3859; value 390R -> 330R
- R3148: renamed from R3860; value 390R -> 330R
- moved H101 264.6 mm to (397.3, 58.4)
- moved H104 232.7 mm to (166.1, 198.1)
- moved H103 137.2 mm to (397.3, 198.1)
- moved H102 5.91 mm to (166.1, 58.4)
- moved C1001 2.54 mm to (236.8, 66.7)
- moved C102 2.54 mm to (329.0, 141.2)
- moved C1701 2.54 mm to (292.1, 82.2)
- moved C1702 2.54 mm to (292.1, 85.8)
- moved C1801 2.54 mm to (292.1, 100.4)
- moved C1802 2.54 mm to (292.1, 104.0)
- moved C1901 2.54 mm to (292.1, 119.1)
- moved C1902 2.54 mm to (292.1, 122.6)
- moved C201 2.54 mm to (362.2, 73.2)
- moved C202 2.54 mm to (362.2, 71.1)
- moved C205 2.54 mm to (362.2, 76.3)
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- renumbered C2403 to C1001, C2503 to C1101, C2603 to C1201, C2703 to C1301, C2803 to C1401, C801 to C1601, C802 to C1602, C501 to C1701, C502 to C1702, C601 to C1801, C602 to C1802, C701 to C1901, C702 to C1902, C803 to C2001, C804 to C2002, C901 to C2101, C902 to C2102, C1001 to C2201, C1002 to C2202, C1101 to C2301, C1102 to C2302, C1201 to C2401, C1202 to C2402, C1301 to C2501, C1302 to C2502, C1903 to C501, C2003 to C601, C2103 to C701, C2203 to C801, C2303 to C901, D2401 to D1001, D2402 to D1002, D2403 to D1003, D2404 to D1004, D2405 to D1005, D2406 to D1006, D2501 to D1101, D2502 to D1102, D2503 to D1103, D2504 to D1104, D2505 to D1105, D2506 to D1106, D2601 to D1201, D2602 to D1202, D2603 to D1203, D2604 to D1204, D2605 to D1205, D2606 to D1206, D2701 to D1301, D2702 to D1302, D2703 to D1303, D2704 to D1304, D2705 to D1305, D2706 to D1306, D2801 to D1401, D2802 to D1402, D2803 to D1403, D2804 to D1404, D2805 to D1405, D2806 to D1406, D3401 to D2701, D3402 to D2702, D3403 to D2703, D3404 to D2704, D3405 to D2705, D3406 to D2706, D3407 to D2707, D3408 to D2708, D3501 to D2801, D3502 to D2802, D3503 to D2803, D3504 to D2804, D3505 to D2805, D3506 to D2806, D3507 to D2807, D3508 to D2808, D3601 to D2901, D3602 to D2902, D3603 to D2903, D3604 to D2904, D3605 to D2905, D3606 to D2906, D3607 to D2907, D3608 to D2908, D3701 to D3001, D3702 to D3002, D3703 to D3003, D3704 to D3004, D3705 to D3005, D3706 to D3006, D3707 to D3007, D3708 to D3008, D301 to D302, D302 to D303, D2007 to D3101, D2008 to D3102, D3803 to D3103, D3804 to D3104, D2009 to D3105, D2010 to D3106, D3807 to D3107, D3808 to D3108, D1901 to D501, D1902 to D502, D1903 to D503, D1904 to D504, D1905 to D505, D1906 to D506, D2001 to D601, D2002 to D602, D2003 to D603, D2004 to D604, D2005 to D605, D2006 to D606, D2101 to D701, D2102 to D702, D2103 to D703, D2104 to D704, D2105 to D705, D2106 to D706, D2201 to D801, D2202 to D802, D2203 to D803, D2204 to D804, D2205 to D805, D2206 to D806, D2301 to D901, D2302 to D902, D2303 to D903, D2304 to D904, D2305 to D905, D2306 to D906, F1820 to F401, F1825 to F402, F1819 to F403, F1826 to F404, F1818 to F405, F1827 to F406, F1817 to F407, F1828 to F408, F1816 to F409, F1829 to F410, F1815 to F411, F1830 to F412, F1814 to F413, F1801 to F414, F1813 to F415, F1802 to F416, F1812 to F417, F1803 to F418, F1811 to F419, F1804 to F420, F1810 to F421, F1805 to F422, F1809 to F423, F1806 to F424, F1808 to F425, F1807 to F426, J2101 to J1501, JP2401 to JP1001, JP2404 to JP1002, JP2402 to JP1003, JP2408 to JP1004, JP2501 to JP1101, JP2504 to JP1102, JP2502 to JP1103, JP2508 to JP1104, JP2601 to JP1201, JP2604 to JP1202, JP2602 to JP1203, JP2608 to JP1204, JP2701 to JP1301, JP2704 to JP1302, JP2702 to JP1303, JP2708 to JP1304, JP2801 to JP1401, JP2804 to JP1402, JP2802 to JP1403, JP2808 to JP1404, JP1901 to JP501, JP1904 to JP502, JP1902 to JP503, JP1908 to JP504, JP2001 to JP601, JP2004 to JP602, JP2002 to JP603, JP2008 to JP604, JP2101 to JP701, JP2104 to JP702, JP2102 to JP703, JP2108 to JP704, JP2201 to JP801, JP2204 to JP802, JP2202 to JP803, JP2208 to JP804, JP2301 to JP901, JP2304 to JP902, JP2302 to JP903, JP2308 to JP904, Q3401 to Q2701, Q3402 to Q2702, Q3403 to Q2703, Q3404 to Q2704, Q3501 to Q2801, Q3502 to Q2802, Q3503 to Q2803, Q3504 to Q2804, Q3601 to Q2901, Q3602 to Q2902, Q3603 to Q2903, Q3604 to Q2904, Q3701 to Q3001, Q3702 to Q3002, Q3703 to Q3003, Q3704 to Q3004, Q2001 to Q3101, Q2002 to Q3102, Q3803 to Q3103, Q3804 to Q3104, R2401 to R1001, R2402 to R1002, R2403 to R1003, R2404 to R1004, R2405 to R1005, R2406 to R1006, R2407 to R1007, R2408 to R1008, R2409 to R1009, R2410 to R1010, R2411 to R1011, R2412 to R1012, R2416 to R1013, R2417 to R1014, R2413 to R1015, R2415 to R1016, R2501 to R1101, R2502 to R1102, R2503 to R1103, R2504 to R1104, R2505 to R1105, R2506 to R1106, R2507 to R1107, R2508 to R1108, R2509 to R1109, R2510 to R1110, R2511 to R1111, R2512 to R1112, R2516 to R1113, R2517 to R1114, R2513 to R1115, R2515 to R1116, R2601 to R1201, R2602 to R1202, R2603 to R1203, R2604 to R1204, R2605 to R1205, R2606 to R1206, R2607 to R1207, R2608 to R1208, R2609 to R1209, R2610 to R1210, R2611 to R1211, R2612 to R1212, R2616 to R1213, R2617 to R1214, R2613 to R1215, R2615 to R1216, R2701 to R1301, R2702 to R1302, R2703 to R1303, R2704 to R1304, R2705 to R1305, R2706 to R1306, R2707 to R1307, R2708 to R1308, R2709 to R1309, R2710 to R1310, R2711 to R1311, R2712 to R1312, R2716 to R1313, R2717 to R1314, R2713 to R1315, R2715 to R1316, R2801 to R1401, R2802 to R1402, R2803 to R1403, R2804 to R1404, R2805 to R1405, R2806 to R1406, R2807 to R1407, R2808 to R1408, R2809 to R1409, R2810 to R1410, R2811 to R1411, R2812 to R1412, R2816 to R1413, R2817 to R1414, R2813 to R1415, R2815 to R1416, R305 to R1501, R306 to R1502, R307 to R1503, R308 to R1504, R309 to R1505, R310 to R1506, R311 to R1507, R312 to R1508, R313 to R1509, R314 to R1510, R315 to R1511, R316 to R1512, R317 to R1513, R318 to R1514, R319 to R1515, R320 to R1516, R321 to R1517, R322 to R1518, R323 to R1519, R324 to R1520, R325 to R1521, R326 to R1522, R327 to R1523, R328 to R1524, R329 to R1525, R330 to R1526, R801 to R1601, R802 to R1602, R803 to R1603, R804 to R1604, R805 to R1605, R806 to R1606, R807 to R1607, R808 to R1608, R809 to R1609, R810 to R1610, R811 to R1611, R812 to R1612, R813 to R1613, R814 to R1614, R501 to R1701, R502 to R1702, R503 to R1703, R504 to R1704, R505 to R1705, R506 to R1706, R507 to R1707, R508 to R1708, R509 to R1709, R510 to R1710, R511 to R1711, R512 to R1712, R513 to R1713, R514 to R1714, R601 to R1801, R602 to R1802, R603 to R1803, R604 to R1804, R605 to R1805, R606 to R1806, R607 to R1807, R608 to R1808, R609 to R1809, R610 to R1810, R611 to R1811, R612 to R1812, R613 to R1813, R614 to R1814, R701 to R1901, R702 to R1902, R703 to R1903, R704 to R1904, R705 to R1905, R706 to R1906, R707 to R1907, R708 to R1908, R709 to R1909, R710 to R1910, R711 to R1911, R712 to R1912, R713 to R1913, R714 to R1914, R815 to R2001, R816 to R2002, R817 to R2003, R818 to R2004, R819 to R2005, R820 to R2006, R821 to R2007, R822 to R2008, R823 to R2009, R824 to R2010, R825 to R2011, R826 to R2012, R827 to R2013, R828 to R2014, R901 to R2101, R902 to R2102, R903 to R2103, R904 to R2104, R905 to R2105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
Connections:
- net /Balancing/B_01 renamed /B1
- net /Balancing/B_02 renamed /B2
- net /Balancing/B_03 renamed /B3
- net /Balancing/B_04 renamed /B4
- net /Balancing/B_05 renamed /B5
- net /Balancing/B_06 renamed /B6
- net /Balancing/B_07 renamed /B7
- net /Balancing/B_08 renamed /B8
- net /Balancing/B_09 renamed /B9
- net /Balancing/B_10 renamed /B10
- net /Balancing/B_11 renamed /B11
- net /Balancing/B_12 renamed /B12
- net /Balancing/B_13 renamed /B13
- net /Balancing/B_14 renamed /B14
- net /Balancing/B_15 renamed /B15
- net /Balancing/B_16 renamed /B16
- net /Balancing/B_17 renamed /Balancing/B17
- net /Balancing/B_18 renamed /Balancing/B18
- net /Balancing/B_19 renamed /Balancing/B19
- net /Balancing/B_20 renamed /Balancing/B20
- net /Voltage References/0.850V renamed /0.850V
- net /Voltage References/5.000V renamed /5.000V
- net /Voltage Sensors/V1 renamed /V1
- net /Voltage Sensors/V10 renamed /V10
- net /Voltage Sensors/V11 renamed /V11
- net /Voltage Sensors/V12 renamed /V12
- net /Voltage Sensors/V13 renamed /V13
- net /Voltage Sensors/V14 renamed /V14
- net /Voltage Sensors/V15 renamed /V15
- net /Voltage Sensors/V16 renamed /V16
- net /Voltage Sensors/V2 renamed /V2
- net /Voltage Sensors/V3 renamed /V3
- net /Voltage Sensors/V4 renamed /V4
- net /Voltage Sensors/V5 renamed /V5
- net /Voltage Sensors/V6 renamed /V6
- net /Voltage Sensors/V7 renamed /V7
- net /Voltage Sensors/V8 renamed /V8
- net /Voltage Sensors/V9 renamed /V9
- net Net-(U101-Pad15) renamed /B17
- net Net-(U101-Pad3) renamed /B20
- net Net-(U102-Pad3) renamed /TOUT_1
- net Net-(U103-Pad3) renamed /TOUT_3
- net Net-(U104-Pad3) renamed /TOUT_2
- C1001 pad 1: /Voltage Sensors/1.8V -> /1.8V
- C1101 pad 1: /Voltage Sensors/1.8V -> /1.8V
- C1201 pad 1: /Voltage Sensors/1.8V -> /1.8V
- C1301 pad 1: /Voltage Sensors/1.8V -> /1.8V
- C1401 pad 1: /Voltage Sensors/1.8V -> /1.8V
- C1601 pad 1: -5V -> +5V
- C1701 pad 1: -5V -> +5V
- C1801 pad 1: -5V -> +5V
- C1901 pad 1: -5V -> +5V
- C2001 pad 1: -5V -> +5V
- C2101 pad 1: -5V -> +5V
- C2201 pad 1: -5V -> +5V
- C2301 pad 1: -5V -> +5V
- C2401 pad 1: -5V -> +5V
- C2501 pad 1: -5V -> +5V
- C303 pad 1: -5V -> +5V
- C309 pad 1: -5V -> +5V
- C314 pad 1: -5V -> +5V
- C317 pad 1: -5V -> +5V
- C318 pad 1: -5V -> +5V
- C501 pad 1: /Voltage Sensors/1.8V -> /1.8V
- C601 pad 1: /Voltage Sensors/1.8V -> /1.8V
- C701 pad 1: /Voltage Sensors/1.8V -> /1.8V
- C801 pad 1: /Voltage Sensors/1.8V -> /1.8V
- C901 pad 1: /Voltage Sensors/1.8V -> /1.8V
- F301 pad 1: Net-(F301-Pad1) -> Net-(D301-Pad2)
- FB301 pad 2: Net-(F301-Pad1) -> Net-(D301-Pad1)
- Q2701 pad 1: Net-(Q3401-Pad1) -> Net-(Q2701-Pad1)
- Q2702 pad 1: Net-(Q3402-Pad1) -> Net-(Q2702-Pad1)
- Q2703 pad 1: Net-(Q3403-Pad1) -> Net-(Q2703-Pad1)
- Q2704 pad 1: Net-(Q3404-Pad1) -> Net-(Q2704-Pad1)
- Q2801 pad 1: Net-(Q3501-Pad1) -> Net-(Q2801-Pad1)
- Q2802 pad 1: Net-(Q3502-Pad1) -> Net-(Q2802-Pad1)
- Q2803 pad 1: Net-(Q3503-Pad1) -> Net-(Q2803-Pad1)
- Q2804 pad 1: Net-(Q3504-Pad1) -> Net-(Q2804-Pad1)
- Q2901 pad 1: Net-(Q3601-Pad1) -> Net-(Q2901-Pad1)
- Q2902 pad 1: Net-(Q3602-Pad1) -> Net-(Q2902-Pad1)
- Q2903 pad 1: Net-(Q3603-Pad1) -> Net-(Q2903-Pad1)
- Q2904 pad 1: Net-(Q3604-Pad1) -> Net-(Q2904-Pad1)
- Q3001 pad 1: Net-(Q3701-Pad1) -> Net-(Q3001-Pad1)
- Q3002 pad 1: Net-(Q3702-Pad1) -> Net-(Q3002-Pad1)
- Q3003 pad 1: Net-(Q3703-Pad1) -> Net-(Q3003-Pad1)
- Q3004 pad 1: Net-(Q3704-Pad1) -> Net-(Q3004-Pad1)
- R1604 pad 2: /Temperature Sensors/2.2727V -> /2.2727V
- R1605 pad 1: /Temperature Sensors/2.2727V -> /2.2727V
- R1611 pad 2: /Temperature Sensors/2.2727V -> /2.2727V
- R1612 pad 1: /Temperature Sensors/2.2727V -> /2.2727V
- R1704 pad 2: /Temperature Sensors/2.2727V -> /2.2727V
- R1705 pad 1: /Temperature Sensors/2.2727V -> /2.2727V
- R1711 pad 2: /Temperature Sensors/2.2727V -> /2.2727V
- R1712 pad 1: /Temperature Sensors/2.2727V -> /2.2727V
- R1804 pad 2: /Temperature Sensors/2.2727V -> /2.2727V
- R1805 pad 1: /Temperature Sensors/2.2727V -> /2.2727V
- R1811 pad 2: /Temperature Sensors/2.2727V -> /2.2727V
- R1812 pad 1: /Temperature Sensors/2.2727V -> /2.2727V
- R1904 pad 2: /Temperature Sensors/2.2727V -> /2.2727V
- R1905 pad 1: /Temperature Sensors/2.2727V -> /2.2727V
- R1911 pad 2: /Temperature Sensors/2.2727V -> /2.2727V
- R1912 pad 1: /Temperature Sensors/2.2727V -> /2.2727V
- R2004 pad 2: /Temperature Sensors/2.2727V -> /2.2727V
- R2005 pad 1: /Temperature Sensors/2.2727V -> /2.2727V
- R2011 pad 2: /Temperature Sensors/2.2727V -> /2.2727V
- R2012 pad 1: /Temperature Sensors/2.2727V -> /2.2727V
- R210 pad 2: /Voltage References/2.2727V -> /2.2727V
- R2104 pad 2: /Temperature Sensors/2.2727V -> /2.2727V
- R2105 pad 1: /Temperature Sensors/2.2727V -> /2.2727V
- R211 pad 1: /Voltage References/1.8V -> /1.8V
- R2111 pad 2: /Temperature Sensors/2.2727V -> /2.2727V
- R2112 pad 1: /Temperature Sensors/2.2727V -> /2.2727V
- R2204 pad 2: /Temperature Sensors/2.2727V -> /2.2727V
- R2205 pad 1: /Temperature Sensors/2.2727V -> /2.2727V
- R2211 pad 2: /Temperature Sensors/2.2727V -> /2.2727V
- R2212 pad 1: /Temperature Sensors/2.2727V -> /2.2727V
- R2304 pad 2: /Temperature Sensors/2.2727V -> /2.2727V
- R2305 pad 1: /Temperature Sensors/2.2727V -> /2.2727V
- R2311 pad 2: /Temperature Sensors/2.2727V -> /2.2727V
- R2312 pad 1: /Temperature Sensors/2.2727V -> /2.2727V
- R2404 pad 2: /Temperature Sensors/2.2727V -> /2.2727V
- R2405 pad 1: /Temperature Sensors/2.2727V -> /2.2727V
- R2411 pad 2: /Temperature Sensors/2.2727V -> /2.2727V
- R2412 pad 1: /Temperature Sensors/2.2727V -> /2.2727V
- R2504 pad 2: /Temperature Sensors/2.2727V -> /2.2727V
- R2505 pad 1: /Temperature Sensors/2.2727V -> /2.2727V
- R2511 pad 2: /Temperature Sensors/2.2727V -> /2.2727V
- R2512 pad 1: /Temperature Sensors/2.2727V -> /2.2727V
- R2705 pad 2: Net-(R3405-Pad2) -> Net-(R2705-Pad2)
- R2706 pad 2: Net-(R3406-Pad2) -> Net-(R2706-Pad2)
- R2707 pad 2: Net-(R3407-Pad2) -> Net-(R2707-Pad2)
- R2708 pad 2: Net-(R3408-Pad2) -> Net-(R2708-Pad2)
- R2709 pad 1: Net-(R3409-Pad1) -> Net-(R2709-Pad1)
- R2710 pad 1: Net-(R3410-Pad1) -> Net-(R2710-Pad1)
- R2711 pad 1: Net-(R3411-Pad1) -> Net-(R2711-Pad1)
- R2712 pad 1: Net-(R3412-Pad1) -> Net-(R2712-Pad1)
- R2717 pad 2: Net-(Q3401-Pad1) -> Net-(Q2701-Pad1)
- R2718 pad 2: Net-(Q3402-Pad1) -> Net-(Q2702-Pad1)
- R2719 pad 2: Net-(Q3403-Pad1) -> Net-(Q2703-Pad1)
- R2720 pad 2: Net-(Q3404-Pad1) -> Net-(Q2704-Pad1)
- R2805 pad 2: Net-(R3505-Pad2) -> Net-(R2805-Pad2)
- R2806 pad 2: Net-(R3506-Pad2) -> Net-(R2806-Pad2)
- R2807 pad 2: Net-(R3507-Pad2) -> Net-(R2807-Pad2)
- R2808 pad 2: Net-(R3508-Pad2) -> Net-(R2808-Pad2)
- R2809 pad 1: Net-(R3509-Pad1) -> Net-(R2809-Pad1)
- R2810 pad 1: Net-(R3510-Pad1) -> Net-(R2810-Pad1)
- R2811 pad 1: Net-(R3511-Pad1) -> Net-(R2811-Pad1)
- R2812 pad 1: Net-(R3512-Pad1) -> Net-(R2812-Pad1)
- R2817 pad 2: Net-(Q3501-Pad1) -> Net-(Q2801-Pad1)
- R2818 pad 2: Net-(Q3502-Pad1) -> Net-(Q2802-Pad1)
- R2819 pad 2: Net-(Q3503-Pad1) -> Net-(Q2803-Pad1)
- R2820 pad 2: Net-(Q3504-Pad1) -> Net-(Q2804-Pad1)
- R2905 pad 2: Net-(R3605-Pad2) -> Net-(R2905-Pad2)
- R2906 pad 2: Net-(R3606-Pad2) -> Net-(R2906-Pad2)
- R2907 pad 2: Net-(R3607-Pad2) -> Net-(R2907-Pad2)
- R2908 pad 2: Net-(R3608-Pad2) -> Net-(R2908-Pad2)
- R2909 pad 1: Net-(R3609-Pad1) -> Net-(R2909-Pad1)
- R2910 pad 1: Net-(R3610-Pad1) -> Net-(R2910-Pad1)
- R2911 pad 1: Net-(R3611-Pad1) -> Net-(R2911-Pad1)
- R2912 pad 1: Net-(R3612-Pad1) -> Net-(R2912-Pad1)
- R2917 pad 2: Net-(Q3601-Pad1) -> Net-(Q2901-Pad1)
- R2918 pad 2: Net-(Q3602-Pad1) -> Net-(Q2902-Pad1)
- R2919 pad 2: Net-(Q3603-Pad1) -> Net-(Q2903-Pad1)
- R2920 pad 2: Net-(Q3604-Pad1) -> Net-(Q2904-Pad1)
- R3005 pad 2: Net-(R3705-Pad2) -> Net-(R3005-Pad2)
- R3006 pad 2: Net-(R3706-Pad2) -> Net-(R3006-Pad2)
- R3007 pad 2: Net-(R3707-Pad2) -> Net-(R3007-Pad2)
- R3008 pad 2: Net-(R3708-Pad2) -> Net-(R3008-Pad2)
- R3009 pad 1: Net-(R3709-Pad1) -> Net-(R3009-Pad1)
- R3010 pad 1: Net-(R3710-Pad1) -> Net-(R3010-Pad1)
- R3011 pad 1: Net-(R3711-Pad1) -> Net-(R3011-Pad1)
- R3012 pad 1: Net-(R3712-Pad1) -> Net-(R3012-Pad1)
- R3017 pad 2: Net-(Q3701-Pad1) -> Net-(Q3001-Pad1)
- R3018 pad 2: Net-(Q3702-Pad1) -> Net-(Q3002-Pad1)
- R3019 pad 2: Net-(Q3703-Pad1) -> Net-(Q3003-Pad1)
- R3020 pad 2: Net-(Q3704-Pad1) -> Net-(Q3004-Pad1)
- R306 pad 1: -5V -> +5V
- TP201 pad 1: /Voltage References/2.2727V -> /2.2727V
- TP202 pad 1: /Voltage References/1.8V -> /1.8V
- TP303 pad 1: -5V -> +5V
- U1003 pad 10: /Voltage Sensors/1.8V -> /1.8V
- U1003 pad 14: /Voltage Sensors/1.8V -> /1.8V
- U101 pad 10: Net-(U103-Pad10) -> /S1
- U101 pad 11: Net-(U103-Pad11) -> /S0
- U101 pad 9: Net-(U103-Pad9) -> /S2
- U102 pad 10: Net-(U104-Pad10) -> /S1
- U102 pad 11: Net-(U104-Pad11) -> /S0
- U102 pad 9: Net-(U104-Pad9) -> /S2
- U103 pad 10: Net-(U102-Pad10) -> /S1
- U103 pad 11: Net-(U102-Pad11) -> /S0
- U103 pad 9: Net-(U102-Pad9) -> /S2
- U109 pad 1: Net-(U101-Pad1) (its old number) -> /B18
- U109 pad 10: Net-(U101-Pad10) -> /~RESET
- U109 pad 11: Net-(U101-Pad11) -> /SCLK
- U109 pad 12: Net-(U101-Pad12) -> /RCLK
- U109 pad 13: Net-(U101-Pad13) -> /~OE
- U109 pad 16: Net-(U101-Pad16) -> +5V
- U109 pad 2: Net-(U101-Pad2) (its old number) -> /B19
- U109 pad 8: Net-(U101-Pad8) -> GND
- U1103 pad 10: /Voltage Sensors/1.8V -> /1.8V
- U1103 pad 14: /Voltage Sensors/1.8V -> /1.8V
- U1203 pad 10: /Voltage Sensors/1.8V -> /1.8V
- U1203 pad 14: /Voltage Sensors/1.8V -> /1.8V
- U1303 pad 10: /Voltage Sensors/1.8V -> /1.8V
- U1303 pad 14: /Voltage Sensors/1.8V -> /1.8V
- U1403 pad 10: /Voltage Sensors/1.8V -> /1.8V
- U1403 pad 14: /Voltage Sensors/1.8V -> /1.8V
- U1601 pad 11: -5V -> +5V
- U1701 pad 11: -5V -> +5V
- U1801 pad 11: -5V -> +5V
- U1901 pad 11: -5V -> +5V
- U2001 pad 11: -5V -> +5V
- U2101 pad 11: -5V -> +5V
- U2201 pad 11: -5V -> +5V
- U2301 pad 11: -5V -> +5V
- U2401 pad 11: -5V -> +5V
- U2501 pad 11: -5V -> +5V
- U2701 pad 1: Net-(R3407-Pad2) -> Net-(R2705-Pad2)
- U2701 pad 10: Net-(R3410-Pad1) -> Net-(R2712-Pad1)
- U2701 pad 11: Net-(Q3401-Pad1) -> Net-(Q2703-Pad1)
- U2701 pad 12: Net-(R3409-Pad1) -> Net-(R2711-Pad1)
- U2701 pad 13: Net-(Q3404-Pad1) -> Net-(Q2702-Pad1)
- U2701 pad 14: Net-(R3412-Pad1) -> Net-(R2710-Pad1)
- U2701 pad 15: Net-(Q3403-Pad1) -> Net-(Q2701-Pad1)
- U2701 pad 16: Net-(R3411-Pad1) -> Net-(R2709-Pad1)
- U2701 pad 3: Net-(R3408-Pad2) -> Net-(R2706-Pad2)
- U2701 pad 5: Net-(R3405-Pad2) -> Net-(R2707-Pad2)
- U2701 pad 7: Net-(R3406-Pad2) -> Net-(R2708-Pad2)
- U2701 pad 9: Net-(Q3402-Pad1) -> Net-(Q2704-Pad1)
- U2801 pad 1: Net-(R3507-Pad2) -> Net-(R2805-Pad2)
- U2801 pad 10: Net-(R3510-Pad1) -> Net-(R2812-Pad1)
- U2801 pad 11: Net-(Q3501-Pad1) -> Net-(Q2803-Pad1)
- U2801 pad 12: Net-(R3509-Pad1) -> Net-(R2811-Pad1)
- U2801 pad 13: Net-(Q3504-Pad1) -> Net-(Q2802-Pad1)
- U2801 pad 14: Net-(R3512-Pad1) -> Net-(R2810-Pad1)
- U2801 pad 15: Net-(Q3503-Pad1) -> Net-(Q2801-Pad1)
- U2801 pad 16: Net-(R3511-Pad1) -> Net-(R2809-Pad1)
- U2801 pad 3: Net-(R3508-Pad2) -> Net-(R2806-Pad2)
- U2801 pad 5: Net-(R3505-Pad2) -> Net-(R2807-Pad2)
- U2801 pad 7: Net-(R3506-Pad2) -> Net-(R2808-Pad2)
- U2801 pad 9: Net-(Q3502-Pad1) -> Net-(Q2804-Pad1)
- U2901 pad 1: Net-(R3607-Pad2) -> Net-(R2905-Pad2)
- U2901 pad 10: Net-(R3610-Pad1) -> Net-(R2912-Pad1)
- U2901 pad 11: Net-(Q3601-Pad1) -> Net-(Q2903-Pad1)
- U2901 pad 12: Net-(R3609-Pad1) -> Net-(R2911-Pad1)
- U2901 pad 13: Net-(Q3604-Pad1) -> Net-(Q2902-Pad1)
- U2901 pad 14: Net-(R3612-Pad1) -> Net-(R2910-Pad1)
- U2901 pad 15: Net-(Q3603-Pad1) -> Net-(Q2901-Pad1)
- U2901 pad 16: Net-(R3611-Pad1) -> Net-(R2909-Pad1)
- U2901 pad 3: Net-(R3608-Pad2) -> Net-(R2906-Pad2)
- U2901 pad 5: Net-(R3605-Pad2) -> Net-(R2907-Pad2)
- U2901 pad 7: Net-(R3606-Pad2) -> Net-(R2908-Pad2)
- U2901 pad 9: Net-(Q3602-Pad1) -> Net-(Q2904-Pad1)
- U3001 pad 1: Net-(R3707-Pad2) -> Net-(R3005-Pad2)
- U3001 pad 10: Net-(R3710-Pad1) -> Net-(R3012-Pad1)
- U3001 pad 11: Net-(Q3701-Pad1) -> Net-(Q3003-Pad1)
- U3001 pad 12: Net-(R3709-Pad1) -> Net-(R3011-Pad1)
- U3001 pad 13: Net-(Q3704-Pad1) -> Net-(Q3002-Pad1)
- U3001 pad 14: Net-(R3712-Pad1) -> Net-(R3010-Pad1)
- U3001 pad 15: Net-(Q3703-Pad1) -> Net-(Q3001-Pad1)
- U3001 pad 16: Net-(R3711-Pad1) -> Net-(R3009-Pad1)
- U3001 pad 3: Net-(R3708-Pad2) -> Net-(R3006-Pad2)
- U3001 pad 5: Net-(R3705-Pad2) -> Net-(R3007-Pad2)
- U3001 pad 7: Net-(R3706-Pad2) -> Net-(R3008-Pad2)
- U3001 pad 9: Net-(Q3702-Pad1) -> Net-(Q3004-Pad1)
- U301 pad 5: -5V -> +5V
- U302 pad 5: -5V -> +5V
- U304 pad 5: -5V -> +5V
- U305 pad 5: -5V -> +5V
- U503 pad 10: /Voltage Sensors/1.8V -> /1.8V
- U503 pad 14: /Voltage Sensors/1.8V -> /1.8V
- U603 pad 10: /Voltage Sensors/1.8V -> /1.8V
- U603 pad 14: /Voltage Sensors/1.8V -> /1.8V
- U703 pad 10: /Voltage Sensors/1.8V -> /1.8V
- U703 pad 14: /Voltage Sensors/1.8V -> /1.8V
- U803 pad 10: /Voltage Sensors/1.8V -> /1.8V
- U803 pad 14: /Voltage Sensors/1.8V -> /1.8V
- U903 pad 10: /Voltage Sensors/1.8V -> /1.8V
- U903 pad 14: /Voltage Sensors/1.8V -> /1.8V
Routing:
- net -5V: track 623.7 -> 0.00 mm, vias 22 -> 0
- net +5V: track 538.3 -> 1162.0 mm, vias 23 -> 46
- net /1.8V: track 0.00 -> 408.7 mm
- net /Voltage Sensors/1.8V: track 374.1 -> 0.00 mm
- net /2.2727V: track 0.00 -> 358.8 mm, vias 0 -> 2
- net /Temperature Sensors/2.2727V: track 355.3 -> 0.00 mm, vias 2 -> 0
- net /Voltage References/1.8V: track 34.6 -> 0.00 mm
- net /Voltage References/2.2727V: track 3.56 -> 0.00 mm
- net GND: track 1514.1 -> 1512.7 mm
- added copper zone on In1.Cu, net GND
Other:
- board size 242.8 x 149.9 mm -> 241.3 x 149.9 mm
- copper layers 2 -> 4
