File: BMS_20S/LM235_1_2.sch (KiCad schematic (older format))
At the start: 17 parts, among them U1001 LM324

Commit message: add current sense block to the schematic
Parts:
- renumbered C1001 to C1601, C1002 to C1602, R1001 to R1601, R1002 to R1602, R1003 to R1603, R1004 to R1604, R1005 to R1605, R1006 to R1606, R1007 to R1607, R1008 to R1608, R1009 to R1609, R1010 to R1610, R1011 to R1611, R1012 to R1612, R1013 to R1613, R1014 to R1614, U1001 to U1601

Commit message: rounded corners
Changed lines of the file:
@@
 $Descr User 7874 4725
 encoding utf-8
-Sheet 16 32
+Sheet 21 32
 Title ""
 Date ""
@@
 AR Path="/5EC24961/5EC7F6A7/5EA4C987" Ref="U?"  Part="5"
 AR Path="/5EC24961/5EC85226/5EA4C987" Ref="U?"  Part="5"
-F 0 "U2501" V 1075 3100 50  0000 C CNN
+F 0 "U2101" V 1075 3100 50  0000 C CNN
 F 1 "LM324" V 1166 3100 50  0000 C CNN
 F 2 "Package_SO:SOIC-14_3.9x8.7mm_P1.27mm" H 1400 2825 50  0001 C CNN
@@
 AR Path="/5EC24961/5EC7F6A7/5EC12A8F" Ref="R?"  Part="1"
 AR Path="/5EC24961/5EC85226/5EC12A8F" Ref="R?"  Part="1"
-F 0 "R2508" V 4400 1000 50  0000 C CNN
+F 0 "R2108" V 4400 1000 50  0000 C CNN
 F 1 "1K" V 4500 1000 50  0000 C CNN
 F 2 "Resistor_SMD:R_0805_2012Metric" V 4430 1000 50  0001 C CNN
@@
 AR Path="/5EC24961/5EC7F6A7/5EC12A91" Ref="#PWR?"  Part="1"
 AR Path="/5EC24961/5EC85226/5EC12A91" Ref="#PWR?"  Part="1"
-F 0 "#PWR02507" H 4300 850 50  0001 C CNN
+F 0 "#PWR02107" H 4300 850 50  0001 C CNN
 F 1 "+5V" H 4315 1173 50  0000 C CNN
 F 2 "" H 4300 1000 50  0001 C CNN
@@
 AR Path="/5EC24961/5EC7F6A7/5EC12A92" Ref="R?"  Part="1"
 AR Path="/5EC24961/5EC85226/5EC12A92" Ref="R?"  Part="1"
-F 0 "R2509" V 5700 1350 50  0000 C CNN
+F 0 "R2109" V 5700 1350 50  0000 C CNN
 F 1 "10K" V 5800 1250 50  0000 C CNN
 F 2 "Resistor_SMD:R_0805_2012Metric" V 5730 1250 50  0001 C CNN
@@
 AR Path="/5EC24961/5EC7F6A7/5EC12A93" Ref="R?"  Part="1"
 AR Path="/5EC24961/5EC85226/5EC12A93" Ref="R?"  Part="1"
-F 0 "R2510" V 5700 1250 50  0000 C CNN
+F 0 "R2110" V 5700 1250 50  0000 C CNN
 F 1 "10K" V 5800 1350 50  0000 C CNN
 F 2 "Resistor_SMD:R_0805_2012Metric" V 5730 1350 50  0001 C CNN
@@
 AR Path="/5EC24961/5EC7F6A7/5EC12A94" Ref="R?"  Part="1"
 AR Path="/5EC24961/5EC85226/5EC12A94" Ref="R?"  Part="1"
-F 0 "R2511" V 5700 1750 50  0000 C CNN
+F 0 "R2111" V 5700 1750 50  0000 C CNN
 F 1 "10K" V 5800 1650 50  0000 C CNN
 F 2 "Resistor_SMD:R_0805_2012Metric" V 5730 1650 50  0001 C CNN
@@
 AR Path="/5EC24961/5EC7F6A7/5EA5D0CB" Ref="R?"  Part="1"
 AR Path="/5EC24961/5EC85226/5EA5D0CB" Ref="R?"  Part="1"
-F 0 "R2512" V 5700 1650 50  0000 C CNN
+F 0 "R2112" V 5700 1650 50  0000 C CNN
 F 1 "10K" V 5800 1750 50  0000 C CNN
 F 2 "Resistor_SMD:R_0805_2012Metric" V 5730 1750 50  0001 C CNN
@@
 AR Path="/5EC24961/5EC7F6A7/5EA604DB" Ref="R?"  Part="1"
 AR Path="/5EC24961/5EC85226/5EA604DB" Ref="R?"  Part="1"
-F 0 "R2513" H 6100 1950 50  0000 C CNN
+F 0 "R2113" H 6100 1950 50  0000 C CNN
 F 1 "10K" V 6000 2000 50  0000 C CNN
 F 2 "Resistor_SMD:R_0805_2012Metric" V 5930 2000 50  0001 C CNN
@@
 AR Path="/5EC24961/5EC7F6A7/5EA61D0D" Ref="#PWR?"  Part="1"
 AR Path="/5EC24961/5EC85226/5EA61D0D" Ref="#PWR?"  Part="1"
-F 0 "#PWR02508" H 6000 1950 50  0001 C CNN
+F 0 "#PWR02108" H 6000 1950 50  0001 C CNN
 F 1 "GND" H 6005 2027 50  0000 C CNN
 F 2 "" H 6000 2200 50  0001 C CNN
@@
 AR Path="/5EC24961/5EC7F6A7/5EC12A98" Ref="R?"  Part="1"
 AR Path="/5EC24961/5EC85226/5EC12A98" Ref="R?"  Part="1"
-F 0 "R2514" V 6450 1100 50  0000 C CNN
+F 0 "R2114" V 6450 1100 50  0000 C CNN
 F 1 "10K" V 6350 1150 50  0000 C CNN
 F 2 "Resistor_SMD:R_0805_2012Metric" V 6280 1150 50  0001 C CNN
@@
 AR Path="/5EC24961/5EC7F6A7/5EC12A90" Ref="#PWR?"  Part="1"
 AR Path="/5EC24961/5EC85226/5EC12A90" Ref="#PWR?"  Part="1"
-F 0 "#PWR02503" H 1200 850 50  0001 C CNN
+F 0 "#PWR02103" H 1200 850 50  0001 C CNN
 F 1 "+5V" H 1215 1173 50  0000 C CNN
 F 2 "" H 1200 1000 50  0001 C CNN
@@
 AR Path="/5EC24961/5EC7F6A7/5EC12A8E" Ref="R?"  Part="1"
 AR Path="/5EC24961/5EC85226/5EC12A8E" Ref="R?"  Part="1"
-F 0 "R2501" V 1193 1000 50  0000 C CNN
+F 0 "R2101" V 1193 1000 50  0000 C CNN
 F 1 "1K" V 1284 1000 50  0000 C CNN
 F 2 "Resistor_SMD:R_0805_2012Metric" V 1330 1000 50  0001 C CNN
@@
 AR Path="/5EC24961/5EC7F6A7/5EC12A89" Ref="U?"  Part="1"
 AR Path="/5EC24961/5EC85226/5EC12A89" Ref="U?"  Part="1"
-F 0 "U2501" H 2050 1100 50  0000 C CNN
+F 0 "U2101" H 2050 1100 50  0000 C CNN
 F 1 "LM324" H 1950 1250 50  0000 C CNN
 F 2 "Package_SO:SOIC-14_3.9x8.7mm_P1.27mm" H 1950 975 50  0001 C CNN
@@
 AR Path="/5EC24961/5EC7F6A7/5EC12A99" Ref="R?"  Part="1"
 AR Path="/5EC24961/5EC85226/5EC12A99" Ref="R?"  Part="1"
-F 0 "R2502" V 2500 1250 50  0000 C CNN
+F 0 "R2102" V 2500 1250 50  0000 C CNN
 F 1 "10K" V 2700 1250 50  0000 C CNN
 F 2 "Resistor_SMD:R_0805_2012Metric" V 2630 1250 50  0001 C CNN
@@
 AR Path="/5EC24961/5EC7F6A7/5EACB844" Ref="R?"  Part="1"
 AR Path="/5EC24961/5EC85226/5EACB844" Ref="R?"  Part="1"
-F 0 "R2503" V 2600 1250 50  0000 C CNN
+F 0 "R2103" V 2600 1250 50  0000 C CNN
 F 1 "10K" V 2700 1350 50  0000 C CNN
 F 2 "Resistor_SMD:R_0805_2012Metric" V 2630 1350 50  0001 C CNN
@@
 AR Path="/5EC24961/5EC7F6A7/5EACE1A4" Ref="R?"  Part="1"
 AR Path="/5EC24961/5EC85226/5EACE1A4" Ref="R?"  Part="1"
-F 0 "R2504" V 2600 1750 50  0000 C CNN
+F 0 "R2104" V 2600 1750 50  0000 C CNN
 F 1 "10K" V 2700 1650 50  0000 C CNN
 F 2 "Resistor_SMD:R_0805_2012Metric" V 2630 1650 50  0001 C CNN
@@
 AR Path="/5EC24961/5EC7F6A7/5EACE7C9" Ref="R?"  Part="1"
 AR Path="/5EC24961/5EC85226/5EACE7C9" Ref="R?"  Part="1"
-F 0 "R2505" V 2550 1750 50  0000 C CNN
+F 0 "R2105" V 2550 1750 50  0000 C CNN
 F 1 "10K" V 2700 1750 50  0000 C CNN
 F 2 "Resistor_SMD:R_0805_2012Metric" V 2630 1750 50  0001 C CNN
@@
 AR Path="/5EC24961/5EC7F6A7/5EC12A9D" Ref="R?"  Part="1"
 AR Path="/5EC24961/5EC85226/5EC12A9D" Ref="R?"  Part="1"
-F 0 "R2506" H 3100 1950 50  0000 C CNN
+F 0 "R2106" H 3100 1950 50  0000 C CNN
 F 1 "10K" V 2900 2000 50  0000 C CNN
 F 2 "Resistor_SMD:R_0805_2012Metric" V 2830 2000 50  0001 C CNN
@@
 AR Path="/5EC24961/5EC7F6A7/5EAD8CC0" Ref="#PWR?"  Part="1"
 AR Path="/5EC24961/5EC85226/5EAD8CC0" Ref="#PWR?"  Part="1"
-F 0 "#PWR02506" H 2900 1950 50  0001 C CNN
+F 0 "#PWR02106" H 2900 1950 50  0001 C CNN
 F 1 "GND" H 2905 2027 50  0000 C CNN
 F 2 "" H 2900 2200 50  0001 C CNN
@@
 AR Path="/5EC24961/5EC7F6A7/5EADC7DB" Ref="R?"  Part="1"
 AR Path="/5EC24961/5EC85226/5EADC7DB" Ref="R?"  Part="1"
-F 0 "R2507" V 3150 1250 50  0000 C CNN
+F 0 "R2107" V 3150 1250 50  0000 C CNN
 F 1 "10K" V 3250 1150 50  0000 C CNN
 F 2 "Resistor_SMD:R_0805_2012Metric" V 3180 1150 50  0001 C CNN
@@
 AR Path="/5EC24961/5EC7F6A7/5EC12AA0" Ref="#PWR?"  Part="1"
 AR Path="/5EC24961/5EC85226/5EC12AA0" Ref="#PWR?"  Part="1"
-F 0 "#PWR02504" H 1800 2750 50  0001 C CNN
+F 0 "#PWR02104" H 1800 2750 50  0001 C CNN
 F 1 "+5V" H 1815 3073 50  0000 C CNN
 F 2 "" H 1800 2900 50  0001 C CNN
@@
 AR Path="/5EC24961/5EC7F6A7/5EC12AA1" Ref="#PWR?"  Part="1"
 AR Path="/5EC24961/5EC85226/5EC12AA1" Ref="#PWR?"  Part="1"
-F 0 "#PWR02501" H 1000 3000 50  0001 C CNN
+F 0 "#PWR02101" H 1000 3000 50  0001 C CNN
 F 1 "-5V" H 1015 3073 50  0000 C CNN
 F 2 "" H 1000 2900 50  0001 C CNN
@@
 AR Path="/5EC24961/5EC7F6A7/5EC12AA2" Ref="C?"  Part="1"
 AR Path="/5EC24961/5EC85226/5EC12AA2" Ref="C?"  Part="1"
-F 0 "C2502" H 1915 3296 50  0000 L CNN
+F 0 "C2102" H 1915 3296 50  0000 L CNN
 F 1 "100nF" H 1915 3205 50  0000 L CNN
 F 2 "Capacitor_SMD:C_0805_2012Metric" H 1838 3100 50  0001 C CNN
@@
 AR Path="/5EC24961/5EC7F6A7/5EC12AA3" Ref="C?"  Part="1"
 AR Path="/5EC24961/5EC85226/5EC12AA3" Ref="C?"  Part="1"
-F 0 "C2501" H 1115 3296 50  0000 L CNN
+F 0 "C2101" H 1115 3296 50  0000 L CNN
 F 1 "100nF" H 1115 3205 50  0000 L CNN
 F 2 "Capacitor_SMD:C_0805_2012Metric" H 1038 3100 50  0001 C CNN
@@
 AR Path="/5EC24961/5EC7F6A7/5EC12AA4" Ref="#PWR?"  Part="1"
 AR Path="/5EC24961/5EC85226/5EC12AA4" Ref="#PWR?"  Part="1"
-F 0 "#PWR02505" H 1800 3250 50  0001 C CNN
+F 0 "#PWR02105" H 1800 3250 50  0001 C CNN
 F 1 "GND" H 1805 3327 50  0000 C CNN
 F 2 "" H 1800 3500 50  0001 C CNN
@@
 AR Path="/5EC24961/5EC7F6A7/5EC12AA5" Ref="#PWR?"  Part="1"
 AR Path="/5EC24961/5EC85226/5EC12AA5" Ref="#PWR?"  Part="1"
-F 0 "#PWR02502" H 1000 3250 50  0001 C CNN
+F 0 "#PWR02102" H 1000 3250 50  0001 C CNN
 F 1 "GND" H 1005 3327 50  0000 C CNN
 F 2 "" H 1000 3500 50  0001 C CNN
@@
 AR Path="/5EC24961/5EC7F6A7/5EA4A09D" Ref="U?"  Part="2"
 AR Path="/5EC24961/5EC85226/5EA4A09D" Ref="U?"  Part="2"
-F 0 "U2501" H 5150 1100 50  0000 C CNN
+F 0 "U2101" H 5150 1100 50  0000 C CNN
 F 1 "LM324" H 5000 1250 50  0000 C CNN
 F 2 "Package_SO:SOIC-14_3.9x8.7mm_P1.27mm" H 5050 975 50  0001 C CNN
@@
 AR Path="/5EC24961/5EC7F6A7/5EC12A8C" Ref="U?"  Part="4"
 AR Path="/5EC24961/5EC85226/5EC12A8C" Ref="U?"  Part="4"
-F 0 "U2501" H 3350 1350 50  0000 C CNN
+F 0 "U2101" H 3350 1350 50  0000 C CNN
 F 1 "LM324" H 3250 1500 50  0000 C CNN
 F 2 "Package_SO:SOIC-14_3.9x8.7mm_P1.27mm" H 3250 1225 50  0001 C CNN
@@
 AR Path="/5EC24961/5EC7F6A7/5EA4B508" Ref="U?"  Part="3"
 AR Path="/5EC24961/5EC85226/5EA4B508" Ref="U?"  Part="3"
-F 0 "U2501" H 6450 1350 50  0000 C CNN
+F 0 "U2101" H 6450 1350 50  0000 C CNN
 F 1 "LM324" H 6300 1500 50  0000 C CNN
 F 2 "Package_SO:SOIC-14_3.9x8.7mm_P1.27mm" H 6350 1225 50  0001 C CNN
