File: TSAL/TSAL.kicad_pcb (KiCad board)
At the start: 2 copper layers, 100.1 x 100.1 mm, 100 parts, among them J1 Screw_Terminal_01x02, J2 Screw_Terminal_01x02, K1 RELAY_19.1x15.5mm, Q1 Si2302DS, Q2 IRF3205, Q3 IRF3205, U1 TLP290-4, U2 NE555, U3 TL431DBZ, U4 LM358, U5 MC34063, U6 TL431DBZ

Commit message: update TSAL
Parts:
- added G1: Logo_High_Voltage_Large, e-Power:Logo_High_Voltage_13.7x12.0mm_SilkS, F.Cu at (139.9, 79.1)
- added G2: Logo_UFRGS_Large, e-Power:Logo_UFRGS_14.7x8.0mm_SilkS, F.Cu at (201.7, 145.3)
- added G3: Logo_e-Power_Large, e-Power:Logo_e-Power_22.8x12.0mm_SilkS, F.Cu at (189.7, 125.5)
- added R51: ADJ, Resistor_SMD:R_0805_2012Metric, F.Cu at (150.6, 113.6)
- added TP11: GND, e-Power:TestPoint_Pad_D1.0mm, F.Cu at (185.9, 112.4)
- added TP12: +V, e-Power:TestPoint_Pad_D1.0mm, F.Cu at (143.9, 56.0)
- added TP13: GND, e-Power:TestPoint_Pad_D1.0mm, F.Cu at (188.3, 73.5)
- added TP14: -V, e-Power:TestPoint_Pad_D1.0mm, F.Cu at (143.9, 75.3)
- added TP15: GND, e-Power:TestPoint_Pad_D1.0mm, F.Cu at (213.4, 56.9)
- added TP16: GND, e-Power:TestPoint_Pad_D1.0mm, F.Cu at (205.9, 140.3)
- added TP17: +VIN, e-Power:TestPoint_Pad_D1.0mm, F.Cu at (135.1, 138.3)
- added TP18: RED, e-Power:TestPoint_Pad_D1.0mm, F.Cu at (184.7, 138.4)
- added TP19: +24V, e-Power:TestPoint_Pad_D1.0mm, F.Cu at (174.5, 138.4)
- added TP20: BLUE, e-Power:TestPoint_Pad_D1.0mm, F.Cu at (179.6, 138.4)
- added TP21: 12V, e-Power:TestPoint_Pad_D1.0mm, F.Cu at (163.6, 109.5)
- added TP22: GND, e-Power:TestPoint_Pad_D1.0mm, F.Cu at (166.1, 135.1)
- C1, C11, C12, C13, C4, C6, C7, C8, C9: footprint Capacitor_SMD:C_0805_2012Metric_Pad1.15x1.40mm_HandSolder -> Capacitor_SMD:C_0805_2012Metric
- H1: value +12V -> +VIN
- H4: value GND -> NC
- J1: value Screw_Terminal_01x02 -> Tractive System
- J2: value Screw_Terminal_01x02 -> Input Power
- L1: footprint Inductor_SMD:L_12x12mm_H6mm -> e-Power:L_12x12mm_H6mm
- R10, R11, R12, R13, R14, R15, R16, R17, R18, R19, R20, R21, R22, R23, R24, R25, R26, R27, R28, R29, R3, R30, R31, R32, R33, R34, R35, R36, R37, R38, R39, R4, R40, R41, R42, R43, R44, R45, R46, R47, R48, R49, R5, R50, R8, R9: footprint Resistor_SMD:R_0805_2012Metric_Pad1.15x1.40mm_HandSolder -> Resistor_SMD:R_0805_2012Metric
- TP8: value G -> GREEN
- U3, U6: value TL431DBZ -> TL431
- moved TP6 101.8 mm to (205.9, 137.6)
- moved C11 90.5 mm to (188.3, 89.3)
- moved R11 83.9 mm to (178.3, 96.5), turned to 270 degrees
- moved R9 69.2 mm to (182.3, 106.5), turned to 0 degrees
- moved R13 68.9 mm to (194.2, 108.0), turned to 180 degrees
- moved U2 67.3 mm to (188.4, 107.0)
- moved R8 65.1 mm to (194.2, 104.0), turned to 0 degrees
- moved C1 64.7 mm to (194.2, 110.1), turned to 180 degrees
- moved TP4 63.7 mm to (217.4, 56.9), turned to 0 degrees
- moved TP2 62.7 mm to (188.5, 112.4)
- moved R12 62.4 mm to (194.2, 106.0), turned to 180 degrees
- moved D5 61.3 mm to (182.4, 108.4), turned to 180 degrees
- moved C10 59.1 mm to (170.9, 118.2), turned to 270 degrees
- moved C2 57.2 mm to (194.3, 112.3), turned to 0 degrees
- moved J1 53.1 mm to (133.8, 62.8), turned to 270 degrees
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Connections:
- H1 pad 1: +12V -> Input_Power
- H4 pad 1: GND -> Net-(H4-Pad1)
- R1 pad 2: Net-(J1-Pad2) -> Net-(J1-Pad1)
- R6 pad 2: Net-(J1-Pad1) -> Net-(J1-Pad2)
- U1 pad 1: Net-(D3-Pad2) -> Net-(R42-Pad1)
- U1 pad 10: Net-(Q3-Pad1) -> Net-(R3-Pad2)
- U1 pad 16: Net-(R3-Pad2) -> Net-(Q3-Pad1)
- U1 pad 2: Net-(R7-Pad1) -> GND
- U1 pad 7: Net-(R42-Pad1) -> Net-(D3-Pad2)
- U1 pad 8: GND -> Net-(R7-Pad1)
Routing:
- net GND: track 54.9 -> 757.1 mm, vias 0 -> 14
- net +12V: track 57.6 -> 229.4 mm, vias 0 -> 6
- net Net-(C7-Pad2): track 0.00 -> 108.5 mm, vias 0 -> 2
- net Net-(D6-Pad3): track 0.00 -> 84.5 mm, vias 0 -> 4
- net Net-(C4-Pad2): track 0.00 -> 84.5 mm
- net (no net): track 78.9 -> 0.00 mm
- net Net-(Q2-Pad1): track 0.00 -> 65.9 mm, vias 0 -> 4
- net Net-(R14-Pad2): track 0.00 -> 62.0 mm, vias 0 -> 2
- net Net-(R11-Pad2): track 0.00 -> 49.9 mm
- net Net-(K1-Pad3): track 40.7 -> 90.4 mm, vias 1 -> 3
- net Net-(Q3-Pad1): track 0.00 -> 45.8 mm, vias 0 -> 2
- net +24V: track 33.0 -> 76.7 mm, vias 0 -> 2
- net Input_Power: track 0.00 -> 42.4 mm
- net Net-(C13-Pad2): track 0.00 -> 39.5 mm
- net Net-(D3-Pad2): track 0.00 -> 24.4 mm
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- added copper zone on F.Cu, net +12V
- added copper zone on F.Cu, net GND
- added copper zone on F.Cu, net Net-(D6-Pad3)
- added copper zone on F.Cu, net Net-(D6-Pad4)
Other:
- board text added: "-"
- board text added: "---------------"
- board text added: "-------------------"
- board text added: "TESTED ON"
- board text removed: "+24V"
- board text removed: "G"
- board text removed: "GND"
- board text removed: "Input Power"
- board text removed: "R"

Commit message: update tsal
Parts:
- moved U3 0.18 mm to (190.2, 80.8)
- moved U6 0.17 mm to (186.3, 80.8)
- turned R30 to 180 degrees
Connections:
- U3 pad 1: Net-(R14-Pad2) -> Net-(R14-Pad1)
- U3 pad 2: Net-(R14-Pad1) -> Net-(R14-Pad2)
- U6 pad 1: Net-(R29-Pad1) -> Net-(R30-Pad1)
- U6 pad 2: Net-(R30-Pad1) -> Net-(R29-Pad1)
Routing:
- net Net-(R29-Pad1): track 11.4 -> 8.54 mm, vias 2 -> 0
- net Net-(R30-Pad1): track 10.3 -> 11.9 mm
- net Net-(R14-Pad1): track 16.2 -> 14.9 mm
