File: TSAL/TSAL.sch (KiCad schematic (older format))
At the start: 60 parts, among them J1 Screw_Terminal_01x02, J2 Screw_Terminal_01x02, K1 RELAY_19.1x15.5mm, Q1 BC548, Q2 IRF3205, Q3 IRF3205, U1 MC34063AP, U2 TLP290-4, U3 LM555, U4 TL431DBZ, U5 TL431DBZ, U6 LM358

Commit message: update all circuits
Parts:
- removed C1: 100uF, e-Power:CP_Elec_10x10, symbol Device:CP
- removed C6: 100nF, Capacitor_SMD:C_0805_2012Metric_Pad1.15x1.40mm_HandSolder, symbol Device:C
- removed D3, D4: 1N5819, e-Power:DO-214AC, symbol Diode:1N5819
- removed Q1: BC548, Package_TO_SOT_SMD:SOT-23, symbol Transistor_BJT:BC548
- removed R10: 18K, Resistor_SMD:R_0805_2012Metric_Pad1.15x1.40mm_HandSolder, symbol Device:R
- removed R14: 220K, Resistor_SMD:R_0805_2012Metric_Pad1.15x1.40mm_HandSolder, symbol Device:R
- removed unit 2 of U2
- removed unit 3 of U2
- removed unit 4 of U2
- removed U3: LM555, Package_DIP:DIP-8_W7.62mm_LongPads, symbol Timer:LM555
- removed U4, U5: TL431DBZ, Package_TO_SOT_SMD:SOT-23, symbol Reference_Voltage:TL431DBZ
- added C11, C12, C13, C4: 100nF, Capacitor_SMD:C_0805_2012Metric_Pad1.15x1.40mm_HandSolder, symbol Device:C
- added C5: 220u, e-Power:CP_Elec_10x10, symbol Device:CP
- added D2, D7: SS54HF, e-Power:DO-214AC, symbol e-Power:D_SCH_1N5819
- added H1, H2, H3, H4: MountingHole_Pad, e-Power:MountingHole_3.2mm_M3_Pad_Via, symbol Mechanical:MountingHole_Pad
- added Q1: Si2302DS, Package_TO_SOT_SMD:SOT-23, symbol e-Power:Si2302DS
- added R12, R13, R32: 100K, Resistor_SMD:R_0805_2012Metric_Pad1.15x1.40mm_HandSolder, symbol Device:R
- added R17: 1R, Resistor_SMD:R_0805_2012Metric_Pad1.15x1.40mm_HandSolder, symbol Device:R
- added R18, R19, R20, R27, R28, R33, R34, R35, R39, R40, R41, R43, R44, R45, R46, R47, R48: 10R, Resistor_SMD:R_0805_2012Metric_Pad1.15x1.40mm_HandSolder, symbol Device:R
- added R24, R31, R49, R50: 10K, Resistor_SMD:R_0805_2012Metric_Pad1.15x1.40mm_HandSolder, symbol Device:R
- added TP1: 24V, e-Power:TestPoint_Pad_D1.0mm, symbol Connector:TestPoint
- added TP2: OUT, e-Power:TestPoint_Pad_D1.0mm, symbol Connector:TestPoint
- added TP3: Vref_R, e-Power:TestPoint_Pad_D1.0mm, symbol Connector:TestPoint
- added TP4: RS_R, e-Power:TestPoint_Pad_D1.0mm, symbol Connector:TestPoint
- added TP5: Vref_G, e-Power:TestPoint_Pad_D1.0mm, symbol Connector:TestPoint
- added TP6: RS_G, e-Power:TestPoint_Pad_D1.0mm, symbol Connector:TestPoint
- added TP7: 12V, e-Power:TestPoint_Pad_D1.0mm, symbol Connector:TestPoint
- added TP?: G, e-Power:TestPoint_Pad_D1.0mm, symbol Connector:TestPoint
- added unit 2 of U1
- added unit 3 of U1
- added unit 4 of U1
- added U2: NE555, Package_SO:SOIC-8_3.9x4.9mm_P1.27mm, symbol Timer:NE555
- added U3, U6: TL431DBZ, Package_TO_SOT_SMD:SOT-23, symbol Reference_Voltage:TL431DBZ
- C1: renamed from C4; LCSC (none) -> C49678; Voltage (none) -> 50V
- C10: value 470u -> 220u; LCSC (none) -> C311611
- C2: renamed from C5; footprint e-Power:CP_Elec_10x10 -> Capacitor_SMD:C_0805_2012Metric; LCSC (none) -> C28323; Voltage 16V -> 50V
- C3: value 100uF -> 220u; LCSC (none) -> C311611; Voltage 16V -> (none)
- C6: renamed from C2; LCSC (none) -> C53172; Voltage (none) -> 50V
- C7: LCSC (none) -> C49678; Voltage (none) -> 50V
- C8: value 100n -> 100nF; LCSC (none) -> C49678; Voltage (none) -> 50V
- C9: LCSC (none) -> C1710
- D4: renamed from D5; value LED -> LED GREEN; footprint LED_SMD:LED_0805_2012Metric -> LED_SMD:LED_0603_1608Metric; Color GREEN -> (none); LCSC (none) -> C72043; Size 5mm -> (none)
- D5: renamed from D6; value LED -> LED RED; footprint LED_SMD:LED_0805_2012Metric -> LED_SMD:LED_0603_1608Metric; Color RED -> (none); LCSC (none) -> C2286; Size 5mm -> (none)
- D8: value D_SCH_1N5819 -> SS54HF; footprint Diode_SMD:D_SOD-323_HandSoldering -> e-Power:DO-214AC; LCSC (none) -> C22452
- F1: LCSC (none) -> C182445
- FB1: LCSC (none) -> C1002
- J2: footprint Connector_Phoenix_GMSTB:PhoenixContact_GMSTBA_2,5_2-G_1x02_P7.50mm_Horizontal -> e-Power:TerminalBlock_Phoenix_MKDS-1,5-2_1x02_P5.08mm_Horizontal
- L1: value 170uH -> 100uH; footprint e-Power:L_10.4x10.4_H4.8 -> Inductor_SMD:L_12x12mm_H6mm; LCSC (none) -> C169389; Loops 50 TURNS -> (none)
- R10: renamed from R17; LCSC (none) -> C17513
- R11: renamed from R16; LCSC (none) -> C17513
- R14: renamed from R1; value 10K -> 1K; LCSC (none) -> C17513
- R15: renamed from R23; LCSC (none) -> C17513
- R16: renamed from R19; value 10K -> ADJ
- R21: LCSC (none) -> C17513
- R22: renamed from R2; value 0.68R -> 1R; LCSC (none) -> C25271
- R23: renamed from R7; LCSC (none) -> C17408
- R25: value 22R -> 100K; LCSC (none) -> C17513; Power 1W -> (none)
- R26: value 27R -> 10R; LCSC (none) -> C17415; Power 1W -> (none); Precision (none) -> 1%
- R29: renamed from R18; LCSC (none) -> C17513
- R3: renamed from R8; LCSC (none) -> C17414
- R30: renamed from R20; value 10K -> 1K; LCSC (none) -> C17513
- R36: renamed from R24; LCSC (none) -> C17513
- R37: renamed from R27; value 10K -> ADJ
- R38: renamed from R11; LCSC (none) -> C17513
- R4: renamed from R12; LCSC (none) -> C17513
- R42: renamed from R22; LCSC (none) -> C17513
- R5: renamed from R9; LCSC (none) -> C17414
- R8: renamed from R13; LCSC (none) -> C17414
- R9: renamed from R15; LCSC (none) -> C17513
- U1: renamed from U2; footprint e-Power:TLP290-4 -> e-Power:SOIC-16_4.55x10.3mm_P1.27mm(TLP290-4); LCSC (none) -> C39031
- U4: renamed from U6; LCSC (none) -> C7950
- U5: renamed from U1; footprint Package_DIP:DIP-8_W7.62mm -> Package_SO:SOIC-8_3.9x4.9mm_P1.27mm; LCSC (none) -> C32078
- renumbered D2 to D3, D7 to D6, R3 to R1, R5 to R2, R4 to R6, R6 to R7
Connections:
- wire segments 178 -> 284
Other:
- note added: "Vref = 1.25V\n"
- moved on the sheet: C1, C10, C2, C6, C7, C8, C9, D1, D3, D4, D5, D6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

Commit message: review
Parts:
- added TP10: GND, e-Power:TestPoint_Pad_D1.0mm, symbol Connector:TestPoint
- added TP9: 1.25V, e-Power:TestPoint_Pad_D1.0mm, symbol Connector:TestPoint
- C10, C3, C5: value 220u -> 220uF
- D6: footprint Connector_Phoenix_GMSTB:PhoenixContact_GMSTBA_2,5_4-G_1x04_P7.50mm_Horizontal -> e-Power:TerminalBlock_Phoenix_MKDS-1,5-4-5.08_1x04_P5.08mm_Horizontal
- H1: value MountingHole_Pad -> +12V
- H2, H3, H4: value MountingHole_Pad -> GND
- J1: footprint Connector_Phoenix_GMSTB:PhoenixContact_GMSTBA_2,5_2-G_1x02_P7.50mm_Horizontal -> e-Power:TerminalBlock_Phoenix_MKDS-1,5-2_1x02_P5.08mm_Horizontal
- Q2, Q3: footprint Package_TO_SOT_THT:TO-220-3_Horizontal_TabDown -> e-Power:TO-220-3_Horizontal_TabDown
- U5: value MC34063AP -> MC34063
- gave numbers to parts that had none: 1
Connections:
- net GND: now also TP10.1
- net at R31.2, R32.2, R38.2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: now also TP9.1
Changed lines of the file:
@@
 F 0 "J1" H 1118 725 50  0000 C CNN
 F 1 "Screw_Terminal_01x02" H 1118 816 50  0001 C CNN
-F 2 "Connector_Phoenix_GMSTB:PhoenixContact_GMSTBA_2,5_2-G_1x02_P7.50mm_Horizontal" H 1200 1050 50  0001 C CNN
+F 2 "e-Power:TerminalBlock_Phoenix_MKDS-1,5-2_1x02_P5.08mm_Horizontal" H 1200 1050 50  0001 C CNN
 F 3 "~" H 1200 1050 50  0001 C CNN
 F 4 "Tractive System Voltage" H 1118 816 50  0000 C CNN "Comment"
@@
 $EndComp
 $Comp
-L Regulator_Switching:MC34063AP U5
-U 1 1 5E38713E
-P 1700 4600
-F 0 "U5" H 1700 5067 50  0000 C CNN
-F 1 "MC34063AP" H 1700 4976 50  0000 C CNN
-F 2 "Package_SO:SOIC-8_3.9x4.9mm_P1.27mm" H 1750 4150 50  0001 L CNN
-F 3 "http://www.onsemi.com/pub_link/Collateral/MC34063A-D.PDF" H 2200 4500 50  0001 C CNN
-F 4 "C32078" H 1700 4600 50  0001 C CNN "LCSC"
-	1    1700 4600
-	1    0    0    -1
-$EndComp
-$Comp
 L Device:C C6
 U 1 1 5E3972FE
@@
 F 0 "Q2" H 9250 3000 50  0000 L CNN
 F 1 "IRF3205" H 9100 2900 50  0000 L CNN
-F 2 "Package_TO_SOT_THT:TO-220-3_Horizontal_TabDown" H 9650 2975 50  0001 L CIN
+F 2 "e-Power:TO-220-3_Horizontal_TabDown" H 9650 2975 50  0001 L CIN
 F 3 "http://www.irf.com/product-info/datasheets/data/irf3205.pdf" H 9400 3050 50  0001 L CNN
 	1    9400 3050
@@
 F 0 "D6" V 9791 2270 50  0000 R CNN
 F 1 "RGB LED" V 9700 2270 50  0000 R CNN
-F 2 "Connector_Phoenix_GMSTB:PhoenixContact_GMSTBA_2,5_4-G_1x04_P7.50mm_Horizontal" H 9700 2600 50  0001 C CNN
+F 2 "e-Power:TerminalBlock_Phoenix_MKDS-1,5-4-5.08_1x04_P5.08mm_Horizontal" H 9700 2600 50  0001 C CNN
 F 3 "~" H 9700 2600 50  0001 C CNN
 F 4 "50W" V 9609 2270 50  0000 R CNN "Power"
@@
 F 0 "Q3" H 9400 4800 50  0000 L CNN
 F 1 "IRF3205" H 9300 4700 50  0000 L CNN
-F 2 "Package_TO_SOT_THT:TO-220-3_Horizontal_TabDown" H 9850 4775 50  0001 L CIN
+F 2 "e-Power:TO-220-3_Horizontal_TabDown" H 9850 4775 50  0001 L CIN
 F 3 "http://www.irf.com/product-info/datasheets/data/irf3205.pdf" H 9600 4850 50  0001 L CNN
 	1    9600 4850
@@
 Text Notes 5750 5750 0    50   ~ 0
 DESABILITA O LED VERDE\n
-Text Notes 7650 2700 0    79   ~ 16
+Text Notes 7550 2750 0    79   ~ 16
 CONSTANT CURRENT SOURCE
 Text Notes 7650 6400 0    79   ~ 16
@@
 P 3850 6500
 F 0 "C10" H 3968 6546 50  0000 L CNN
-F 1 "220u" H 3968 6455 50  0000 L CNN
+F 1 "220uF" H 3968 6455 50  0000 L CNN
 F 2 "e-Power:CP_Elec_10x10" H 3888 6350 50  0001 C CNN
 F 3 "~" H 3850 6500 50  0001 C CNN
@@
 P 850 4550
 F 0 "C5" H 968 4596 50  0000 L CNN
-F 1 "220u" H 968 4505 50  0000 L CNN
+F 1 "220uF" H 968 4505 50  0000 L CNN
 F 2 "e-Power:CP_Elec_10x10" H 888 4400 50  0001 C CNN
 F 3 "~" H 850 4550 50  0001 C CNN
@@
 P 4150 4300
 F 0 "C3" H 4268 4346 50  0000 L CNN
-F 1 "220u" H 4268 4255 50  0000 L CNN
+F 1 "220uF" H 4268 4255 50  0000 L CNN
 F 2 "e-Power:CP_Elec_10x10" H 4188 4150 50  0001 C CNN
 F 3 "~" H 4150 4300 50  0001 C CNN
@@
 	3500 4900 3500 4800
 Wire Wire Line
-	2100 4900 3500 4900
+	2100 4900 2850 4900
 Connection ~ 3500 4900
 Wire Wire Line
@@
 P 4300 6600
 F 0 "H1" H 4350 6800 50  0000 R CNN
-F 1 "MountingHole_Pad" H 4400 6558 50  0001 L CNN
+F 1 "+12V" H 4400 6558 50  0001 L CNN
 F 2 "e-Power:MountingHole_3.2mm_M3_Pad_Via" H 4300 6600 50  0001 C CNN
 F 3 "~" H 4300 6600 50  0001 C CNN
@@
 P 4700 6600
 F 0 "H3" H 4650 6800 50  0000 L CNN
-F 1 "MountingHole_Pad" H 4800 6558 50  0001 L CNN
+F 1 "GND" H 4800 6558 50  0001 L CNN
 F 2 "e-Power:MountingHole_3.2mm_M3_Pad_Via" H 4700 6600 50  0001 C CNN
 F 3 "~" H 4700 6600 50  0001 C CNN
@@
 P 4900 6600
 F 0 "H4" H 4850 6800 50  0000 L CNN
-F 1 "MountingHole_Pad" H 5000 6558 50  0001 L CNN
+F 1 "GND" H 5000 6558 50  0001 L CNN
 F 2 "e-Power:MountingHole_3.2mm_M3_Pad_Via" H 4900 6600 50  0001 C CNN
 F 3 "~" H 4900 6600 50  0001 C CNN
@@
 P 4500 6600
 F 0 "H2" H 4450 6800 50  0000 L CNN
-F 1 "MountingHole_Pad" H 4600 6558 50  0001 L CNN
+F 1 "GND" H 4600 6558 50  0001 L CNN
 F 2 "e-Power:MountingHole_3.2mm_M3_Pad_Via" H 4500 6600 50  0001 C CNN
 F 3 "~" H 4500 6600 50  0001 C CNN
@@
 $EndComp
 $Comp
-L Connector:TestPoint TP?
+L Connector:TestPoint TP8
 U 1 1 5F4F05DE
 P 9800 3450
-F 0 "TP?" H 9858 3568 50  0000 L CNN
+F 0 "TP8" H 9858 3568 50  0000 L CNN
 F 1 "G" H 9858 3477 50  0000 L CNN
 F 2 "e-Power:TestPoint_Pad_D1.0mm" H 10000 3450 50  0001 C CNN
@@
 Wire Wire Line
 	9700 3450 9700 4650
+$Comp
+L Regulator_Switching:MC34063AP U5
+U 1 1 5E38713E
+P 1700 4600
+F 0 "U5" H 1700 5067 50  0000 C CNN
+F 1 "MC34063" H 1700 4976 50  0000 C CNN
+F 2 "Package_SO:SOIC-8_3.9x4.9mm_P1.27mm" H 1750 4150 50  0001 L CNN
+F 3 "http://www.onsemi.com/pub_link/Collateral/MC34063A-D.PDF" H 2200 4500 50  0001 C CNN
+F 4 "C32078" H 1700 4600 50  0001 C CNN "LCSC"
+	1    1700 4600
+	1    0    0    -1
+$EndComp
+$Comp
+L Connector:TestPoint TP10
+U 1 1 5F3A5548
+P 3800 5250
+F 0 "TP10" H 3858 5368 50  0000 L CNN
+F 1 "GND" H 3858 5277 50  0000 L CNN
+F 2 "e-Power:TestPoint_Pad_D1.0mm" H 4000 5250 50  0001 C CNN
+F 3 "~" H 4000 5250 50  0001 C CNN
+	1    3800 5250
+	1    0    0    -1
+$EndComp
+$Comp
+L power:GND #PWR0102
+U 1 1 5F3A61BD
+P 3800 5350
+F 0 "#PWR0102" H 3800 5100 50  0001 C CNN
+F 1 "GND" H 3805 5177 50  0000 C CNN
+F 2 "" H 3800 5350 50  0001 C CNN
+F 3 "" H 3800 5350 50  0001 C CNN
+	1    3800 5350
+	1    0    0    -1
+$EndComp
+Wire Wire Line
+	3800 5350 3800 5250
+$Comp
+L Connector:TestPoint TP9
+U 1 1 5F3BB24C
+P 2850 4850
+F 0 "TP9" H 2908 4968 50  0000 L CNN
+F 1 "1.25V" H 2908 4877 50  0000 L CNN
+F 2 "e-Power:TestPoint_Pad_D1.0mm" H 3050 4850 50  0001 C CNN
+F 3 "~" H 3050 4850 50  0001 C CNN
+	1    2850 4850
+	1    0    0    -1
+$EndComp
+Wire Wire Line
+	2850 4850 2850 4900
+Connection ~ 2850 4900
+Wire Wire Line
+	2850 4900 3500 4900
 $EndSCHEMATC

Commit message: update TSAL
Parts:
- added G1: Logo_High_Voltage_Large, e-Power:Logo_High_Voltage_13.7x12.0mm_SilkS, symbol e-Power:Logo_High_Voltage_Large
- added G2: Logo_UFRGS_Large, e-Power:Logo_UFRGS_14.7x8.0mm_SilkS, symbol e-Power:Logo_UFRGS_Large
- added G3: Logo_e-Power_Large, e-Power:Logo_e-Power_22.8x12.0mm_SilkS, symbol e-Power:Logo_e-Power_Large
- added R51: ADJ, Resistor_SMD:R_0805_2012Metric, symbol Device:R
- added TP11, TP13, TP15, TP16, TP22: GND, e-Power:TestPoint_Pad_D1.0mm, symbol Connector:TestPoint
- added TP12: +V, e-Power:TestPoint_Pad_D1.0mm, symbol Connector:TestPoint
- added TP14: -V, e-Power:TestPoint_Pad_D1.0mm, symbol Connector:TestPoint
- added TP17: +VIN, e-Power:TestPoint_Pad_D1.0mm, symbol Connector:TestPoint
- added TP18: RED, e-Power:TestPoint_Pad_D1.0mm, symbol Connector:TestPoint
- added TP19: +24V, e-Power:TestPoint_Pad_D1.0mm, symbol Connector:TestPoint
- added TP20: BLUE, e-Power:TestPoint_Pad_D1.0mm, symbol Connector:TestPoint
- added TP21: 12V, e-Power:TestPoint_Pad_D1.0mm, symbol Connector:TestPoint
- C1, C11, C12, C13, C4, C6, C7, C8, C9: footprint Capacitor_SMD:C_0805_2012Metric_Pad1.15x1.40mm_HandSolder -> Capacitor_SMD:C_0805_2012Metric
- H1: value +12V -> +VIN
- H4: value GND -> NC
- J1: value Screw_Terminal_01x02 -> Tractive System; Comment Tractive System Voltage -> (none)
- J2: value Screw_Terminal_01x02 -> Input Power
- L1: footprint Inductor_SMD:L_12x12mm_H6mm -> e-Power:L_12x12mm_H6mm
- R10, R11, R12, R13, R14, R15, R16, R17, R18, R19, R20, R21, R22, R23, R24, R25, R26, R27, R28, R29, R3, R30, R31, R32, R33, R34, R35, R36, R37, R38, R39, R4, R40, R41, R42, R43, R44, R45, R46, R47, R48, R49, R5, R50, R8, R9: footprint Resistor_SMD:R_0805_2012Metric_Pad1.15x1.40mm_HandSolder -> Resistor_SMD:R_0805_2012Metric
- TP8: value G -> GREEN
- U3, U6: value TL431DBZ -> TL431
Connections:
- net +12V: now also R51.2, TP21.1; no longer H1.1
- net +24V: now also TP19.1
- net GND: now also U1.2, TP11.1, TP13.1, TP15.1, TP16.1, TP22.1; no longer H4.1, U1.8
- net Input_Power: now also H1.1, TP17.1
- net at D3.2 (A): now also U1.7; no longer U1.1
- net at J1.1 (Pin_1): now also R1.2, TP12.1; no longer R6.2
- net at J1.2 (Pin_2): now also R6.2, TP14.1; no longer R1.2
- net at R7.1: now also U1.8; no longer U1.2
- net at R3.2, R5.2: now also U1.10; no longer U1.16
- net at D6.2 (BK): now also TP20.1
- net at D6.3 (RK), Q2.2 (D): now also TP18.1
- net at L1.1, R17.1, R22.1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: now also R51.1
- net at Q3.1 (G), R36.2: now also U1.16; no longer U1.10
- net at R42.1: now also U1.1; no longer U1.7
- no-connect marks 1 -> 2
Other:
- moved on the sheet: H1, J1, J2, U1A, U1D

Commit message: update tsal
Parts:
- removed U3, U6: TL431, Package_TO_SOT_SMD:SOT-23, symbol Reference_Voltage:TL431DBZ
- added U3, U6: TL431, Package_TO_SOT_SMD:SOT-23, symbol Reference_Voltage:TL432DBZ
Connections:
- net GND: now also U3.3 (A), U6.3 (A)
- net at R14.1, R16.2, TP3.1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: now also U3.1 (REF)
- net at R14.2, U1.13: now also U3.2 (K)
- net at R30.1, R37.2, TP5.1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: now also U6.1 (REF)
- net at R29.1, R30.2: now also U6.2 (K)
Changed lines of the file:
@@
 	10650 5050 10650 4950
-$Comp
-L Reference_Voltage:TL431DBZ U6
-U 1 1 5F71BCAC
-P 6850 4750
-F 0 "U6" V 6896 4681 50  0000 R CNN
-F 1 "TL431" V 6805 4681 50  0000 R CNN
-F 2 "Package_TO_SOT_SMD:SOT-23" H 6850 4600 50  0001 C CIN
-F 3 "http://www.ti.com/lit/ds/symlink/tl431.pdf" H 6850 4750 50  0001 C CIN
-F 4 "C190245" V 6850 4750 50  0001 C CNN "LCSC"
-	1    6850 4750
-	0    1    -1   0
-$EndComp
-$Comp
-L Reference_Voltage:TL431DBZ U3
-U 1 1 5F728B3A
-P 7350 3300
-F 0 "U3" V 7396 3231 50  0000 R CNN
-F 1 "TL431" V 7305 3231 50  0000 R CNN
-F 2 "Package_TO_SOT_SMD:SOT-23" H 7350 3150 50  0001 C CIN
-F 3 "http://www.ti.com/lit/ds/symlink/tl431.pdf" H 7350 3300 50  0001 C CIN
-F 4 "C190245" V 7350 3300 50  0001 C CNN "LCSC"
-	1    7350 3300
-	0    1    -1   0
-$EndComp
 $Comp
 L Timer:NE555 U2
@@
 	1    0    0    -1
 $EndComp
+$Comp
+L Reference_Voltage:TL432DBZ U3
+U 1 1 5F372C96
+P 7350 3300
+F 0 "U3" V 7396 3231 50  0000 R CNN
+F 1 "TL431" V 7305 3231 50  0000 R CNN
+F 2 "Package_TO_SOT_SMD:SOT-23" H 7350 3150 50  0001 C CIN
+F 3 "http://www.ti.com/lit/ds/symlink/tl431.pdf" H 7350 3300 50  0001 C CIN
+	1    7350 3300
+	0    1    -1   0
+$EndComp
+$Comp
+L Reference_Voltage:TL432DBZ U6
+U 1 1 5F37A9A8
+P 6850 4750
+F 0 "U6" V 6896 4681 50  0000 R CNN
+F 1 "TL431" V 6805 4681 50  0000 R CNN
+F 2 "Package_TO_SOT_SMD:SOT-23" H 6850 4600 50  0001 C CIN
+F 3 "http://www.ti.com/lit/ds/symlink/tl431.pdf" H 6850 4750 50  0001 C CIN
+	1    6850 4750
+	0    1    -1   0
+$EndComp
 $EndSCHEMATC

Commit message: TSAL temp management update
Parts:
- added F2, F3: Fuse, e-Power:FUSE_1206_3216Metric, symbol Device:Fuse
Connections:
- net at R1.2, TP12.1: now also F2.1; no longer J1.1 (Pin_1)
- net at R6.2, TP14.1: now also F3.2; no longer J1.2 (Pin_2)
- new net: F2.2, J1.1 (Pin_1)
- new net: F3.1, J1.2 (Pin_2)
Other:
- moved on the sheet: J1
Changed lines of the file:
@@
 L Connector:Screw_Terminal_01x02 J1
 U 1 1 5E2CCD12
-P 1200 1050
-F 0 "J1" H 1200 1150 50  0000 C CNN
-F 1 "Tractive System " H 1118 816 50  0001 C CNN
-F 2 "e-Power:TerminalBlock_Phoenix_MKDS-1,5-2_1x02_P5.08mm_Horizontal" H 1200 1050 50  0001 C CNN
-F 3 "~" H 1200 1050 50  0001 C CNN
-	1    1200 1050
+P 800 1050
+F 0 "J1" H 800 1150 50  0000 C CNN
+F 1 "Tractive System " H 718 816 50  0001 C CNN
+F 2 "e-Power:TerminalBlock_Phoenix_MKDS-1,5-2_1x02_P5.08mm_Horizontal" H 800 1050 50  0001 C CNN
+F 3 "~" H 800 1050 50  0001 C CNN
+	1    800  1050
 	-1   0    0    -1
 $EndComp
@@
 	0    1    -1   0
 $EndComp
+$Comp
+L Device:Fuse F3
+U 1 1 5F37DB3A
+P 1250 1150
+F 0 "F3" V 1050 1150 50  0000 C CNN
+F 1 "Fuse" V 1150 1150 50  0000 C CNN
+F 2 "e-Power:FUSE_1206_3216Metric" V 1180 1150 50  0001 C CNN
+F 3 "~" H 1250 1150 50  0001 C CNN
+F 4 "C182445" V 1250 1150 50  0001 C CNN "LCSC"
+	1    1250 1150
+	0    -1   -1   0
+$EndComp
+$Comp
+L Device:Fuse F2
+U 1 1 5F3800A4
+P 1250 1050
+F 0 "F2" V 1050 1050 50  0000 C CNN
+F 1 "Fuse" V 1150 1050 50  0000 C CNN
+F 2 "e-Power:FUSE_1206_3216Metric" V 1180 1050 50  0001 C CNN
+F 3 "~" H 1250 1050 50  0001 C CNN
+F 4 "C182445" V 1250 1050 50  0001 C CNN "LCSC"
+	1    1250 1050
+	0    1    1    0
+$EndComp
+Wire Wire Line
+	1000 1050 1100 1050
+Wire Wire Line
+	1000 1150 1100 1150
 $EndSCHEMATC

Commit message: update bms pcb
Parts:
- FB1: footprint e-Power:FB_0603_1608Metric -> e-Power:FB_0805_2012Metric
Changed lines of the file:
@@
 F 0 "FB1" V 2426 6300 50  0000 C CNN
 F 1 "Ferrite_Bead" V 2517 6300 50  0000 C CNN
-F 2 "e-Power:FB_0603_1608Metric" V 2630 6300 50  0001 C CNN
+F 2 "e-Power:FB_0805_2012Metric" V 2630 6300 50  0001 C CNN
 F 3 "~" H 2700 6300 50  0001 C CNN
 F 4 "C1002" V 2700 6300 50  0001 C CNN "LCSC"
