File: BMS_24S/BMS_24S.sch (KiCad schematic (older format))
At the start: 30 parts, among them J101 IN, J102 OUT, U101 74HC4051, U102 74HC4051, U103 74HC4051, U104 74HC4051, U105 74HC4051, U106 74HC4051, U107 74HC595, U108 74HC595, U109 74HC595

Commit message: update balancing circuit
Parts:
- C101, C102, C103, C104, C105, C106, C107, C108, C109: LCSC (none) -> C49678; Precision (none) -> 10%; Voltage (none) -> 50V
- H101, H102, H103, H104: footprint MountingHole:MountingHole_4.3mm_M4_Pad_Via -> e-Power:MountingHole_3.2mm_M3_Pad_Via
- R101, R102, R103, R104, R105, R106: LCSC (none) -> C17513; Power (none) -> 1/8W; Precision (none) -> 1%; Voltage (none) -> 150V
Connections:
- net labels added: T21, T22, T23, T24, T[17..24], V21, V22, V23, V24, V[17..24]
- net labels removed: T[17..20], V[17..20]
- wire segments 291 -> 311
- no-connect marks 15 -> 7

Commit message: updates made on BMS
Parts:
- removed J101: IN, e-Power:DSUB-9_Female_EdgeMount_P2.77mm, symbol e-Power:DB9_Female
- removed J102: OUT, e-Power:DSUB-9_Female_EdgeMount_P2.77mm, symbol e-Power:DB9_Female
- added C110, C111: 100nF, Capacitor_SMD:C_0805_2012Metric, symbol Device:C
- added R107, R108, R109, R110, R111, R112, R114, R116, R117, R118, R119, R120, R121, R122, R124, R126, R127, R128, R129, R130, R131, R132, R134, R136: 10K, Resistor_SMD:R_0805_2012Metric, symbol Device:R
- added R113, R115, R123, R125, R133, R135: 1K, Resistor_SMD:R_0805_2012Metric, symbol Device:R
- added U110, U111: LM324, Package_SO:SOIC-14_3.9x8.7mm_P1.27mm, symbol Amplifier_Operational:LM324
- renumbered C104 to C102, C102 to C103, C105 to C104, C103 to C105, R104 to R102, R102 to R103, R105 to R104, R103 to R105, U104 to U102, U102 to U103, U105 to U104, U103 to U105
Connections:
- net labels added: B21, B22, B23, B24, B[1..8], B[17..24], B[9..16], TOUT_1P, TOUT_2P, TOUT_3P, VOUT_1P, VOUT_2P, VOUT_3P
- wire segments 311 -> 478
- no-connect marks 7 -> 3
Other:
- note added: "(VS_1/5)*3.5\n"
- note added: "0.00V ~~ 2.94V\n"
- note added: "0.00V ~~ 4.20V\n"
- note removed: "0.000V ~~ 16.500V\n"

Commit message: update all circuits
Parts:
- added TP1: B1, e-Power:TestPoint_Pad_D1.0mm, symbol Connector:TestPoint
- added TP10: B10, e-Power:TestPoint_Pad_D1.0mm, symbol Connector:TestPoint
- added TP11: B11, e-Power:TestPoint_Pad_D1.0mm, symbol Connector:TestPoint
- added TP12: B12, e-Power:TestPoint_Pad_D1.0mm, symbol Connector:TestPoint
- added TP13: B13, e-Power:TestPoint_Pad_D1.0mm, symbol Connector:TestPoint
- added TP14: B14, e-Power:TestPoint_Pad_D1.0mm, symbol Connector:TestPoint
- added TP15: B15, e-Power:TestPoint_Pad_D1.0mm, symbol Connector:TestPoint
- added TP16: B16, e-Power:TestPoint_Pad_D1.0mm, symbol Connector:TestPoint
- added TP17: B17, e-Power:TestPoint_Pad_D1.0mm, symbol Connector:TestPoint
- added TP18: B18, e-Power:TestPoint_Pad_D1.0mm, symbol Connector:TestPoint
- added TP19: B19, e-Power:TestPoint_Pad_D1.0mm, symbol Connector:TestPoint
- added TP2: B2, e-Power:TestPoint_Pad_D1.0mm, symbol Connector:TestPoint
- added TP20: B20, e-Power:TestPoint_Pad_D1.0mm, symbol Connector:TestPoint
- added TP21: B21, e-Power:TestPoint_Pad_D1.0mm, symbol Connector:TestPoint
- added TP22: B22, e-Power:TestPoint_Pad_D1.0mm, symbol Connector:TestPoint
- added TP23: B23, e-Power:TestPoint_Pad_D1.0mm, symbol Connector:TestPoint
- added TP24: B24, e-Power:TestPoint_Pad_D1.0mm, symbol Connector:TestPoint
- added TP25: GND, e-Power:TestPoint_Pad_D1.0mm, symbol Connector:TestPoint
- added TP3: B3, e-Power:TestPoint_Pad_D1.0mm, symbol Connector:TestPoint
- added TP4: B4, e-Power:TestPoint_Pad_D1.0mm, symbol Connector:TestPoint
- added TP5: B5, e-Power:TestPoint_Pad_D1.0mm, symbol Connector:TestPoint
- added TP6: B6, e-Power:TestPoint_Pad_D1.0mm, symbol Connector:TestPoint
- added TP7: B7, e-Power:TestPoint_Pad_D1.0mm, symbol Connector:TestPoint
- added TP8: B8, e-Power:TestPoint_Pad_D1.0mm, symbol Connector:TestPoint
- added TP9: B9, e-Power:TestPoint_Pad_D1.0mm, symbol Connector:TestPoint

Commit message: get BSPD
Parts:
- added unit 4 of U110
- added unit 4 of U111
- R107, R108, R109, R110, R111, R112, R114, R116, R117, R118, R119, R120, R121, R122, R124, R126, R127, R128, R129, R130, R131, R132, R134, R136: LCSC C17513 -> C17414
- U101, U102, U103, U104, U105, U106: LCSC (none) -> C9386
- U107, U108, U109: LCSC (none) -> C5947
- U110, U111: LCSC (none) -> C71035
Connections:
- wire segments 478 -> 486
- no-connect marks 3 -> 5

Commit message: update bms pcb
Parts:
- H101, H102, H103, H104: value MountingHole_Pad -> GND
- renumbered TP1 to TP101, TP2 to TP102, TP3 to TP103, TP4 to TP104, TP5 to TP105, TP6 to TP106, TP7 to TP107, TP8 to TP108, TP9 to TP109, TP10 to TP110, TP11 to TP111, TP12 to TP112, TP13 to TP113, TP14 to TP114, TP15 to TP115, TP16 to TP116, TP17 to TP117, TP18 to TP118, TP19 to TP119, TP20 to TP120, TP21 to TP121, TP22 to TP122, TP23 to TP123, TP24 to TP124, TP25 to TP125
Other:
- note added: "Generates +12V, +5V"
- note removed: "Generates +12V, +5V \nand -5V from INPUT"

Commit message: update BMS
Connections:
- wire segments 486 -> 477
- no-connect marks 5 -> 9
Changed lines of the file:
@@
 0.00V ~~ 4.20V\n
 $Comp
-L power:GND #PWR0129
-U 1 1 5EEFA243
-P 15100 4600
-F 0 "#PWR0129" H 15100 4350 50  0001 C CNN
-F 1 "GND" H 15105 4427 50  0000 C CNN
-F 2 "" H 15100 4600 50  0001 C CNN
-F 3 "" H 15100 4600 50  0001 C CNN
-	1    15100 4600
-	1    0    0    -1
-$EndComp
-$Comp
 L Mechanical:MountingHole_Pad H101
 U 1 1 5EEFB35E
@@
 	1    0    0    -1
 $EndComp
-Wire Wire Line
-	14950 4400 14950 4500
-Wire Wire Line
-	14700 4500 14950 4500
-Wire Wire Line
-	14700 4400 14700 4500
-Connection ~ 14950 4500
-Wire Wire Line
-	14950 4500 15100 4500
-Wire Wire Line
-	15500 4500 15500 4400
-Wire Wire Line
-	15250 4400 15250 4500
-Connection ~ 15250 4500
-Wire Wire Line
-	15250 4500 15500 4500
-Wire Wire Line
-	15100 4600 15100 4500
-Connection ~ 15100 4500
-Wire Wire Line
-	15100 4500 15250 4500
 Text Label 14800 2700 2    50   ~ 0
 BMS_ERROR
@@
 	5450 10900 5450 10700
 NoConn ~ 6150 10800
+NoConn ~ 14700 4400
+NoConn ~ 14950 4400
+NoConn ~ 15250 4400
+NoConn ~ 15500 4400
 Wire Bus Line
 	3950 5450 3950 6150

Commit message: melhorias feitas no BMS
Parts:
- added C112: 10uF, Capacitor_SMD:C_0805_2012Metric, symbol Device:C
- added C113: 100nF, Capacitor_SMD:C_0805_2012Metric, symbol Device:C
Connections:
- wire segments 477 -> 485
Other:
- moved on the sheet: C107, C108, C109, TP101, TP102, TP103, TP104, TP105, TP106, TP107, TP108, TP109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

Commit message: updates made on BMS
Parts:
- added C105, C116, C117, C119, C120, C121, C122: 100nF, Capacitor_SMD:C_0805_2012Metric, symbol Device:C
- added C109, C110: 12pF, Capacitor_SMD:C_0805_2012Metric, symbol Device:C
- added C111, C112: 100pF, Capacitor_SMD:C_0805_2012Metric, symbol Device:C
- added C123, C124, C127: 10uF, Capacitor_SMD:C_0805_2012Metric, symbol Device:C
- added D101, D102, D103, D104, D105, D106, D107, D108: LED, e-Power:LED_0805_1.15x1.40mm_HandSolder, symbol Device:LED
- added FB101: Ferrite_Bead, e-Power:FB_0805_2012Metric, symbol Device:Ferrite_Bead
- added G101: Logo_UFRGS_Large, e-Power:Logo_UFRGS_22.0x12.0mm_SilkS, symbol e-Power:Logo_UFRGS_Large
- added G102: Logo_e-Power_Large, e-Power:Logo_e-Power_22.8x12.0mm_SilkS, symbol e-Power:Logo_e-Power_Large
- added J101: Conn_01x08_Male, e-Power:Molex_Mini-Fit_Jr_2x04_P4.20mm_Horizontal, symbol Connector:Conn_01x08_Male
- added J102: ST-LINK, Connector_PinHeader_2.54mm:PinHeader_1x05_P2.54mm_Vertical, symbol Connector:Conn_01x05_Male
- added Q101: MMBT5401, Package_TO_SOT_SMD:SOT-23, symbol Transistor_BJT:MMBT3904
- added R103, R126, R127, R128, R129, R130, R131, R132, R133: 1K, Resistor_SMD:R_0805_2012Metric, symbol Device:R
- added R104, R109: 10K, Resistor_SMD:R_0805_2012Metric, symbol Device:R
- added R110: 100R, Resistor_SMD:R_0805_2012Metric, symbol Device:R
- added R111, R112: 10R, Resistor_SMD:R_0805_2012Metric, symbol Device:R
- added SW101: SW_Push, Button_Switch_SMD:SW_Push_1P1T_NO_6x6mm_H9.5mm, symbol Switch:SW_Push
- added TP126, TP132: VCC, e-Power:TestPoint_Pad_D1.0mm, symbol Connector:TestPoint
- added TP127, TP133, TP138: GND, e-Power:TestPoint_Pad_D1.0mm, symbol Connector:TestPoint
- added TP128: CAN_L, e-Power:TestPoint_Pad_D1.0mm, symbol Connector:TestPoint
- added TP129: CAN_H, e-Power:TestPoint_Pad_D1.0mm, symbol Connector:TestPoint
- added TP130: CAN_GND, e-Power:TestPoint_Pad_D1.0mm, symbol Connector:TestPoint
- added TP131: ~ERROR, e-Power:TestPoint_Pad_D1.0mm, symbol Connector:TestPoint
- added TP134: T_SWCLK, e-Power:TestPoint_Pad_D1.0mm, symbol Connector:TestPoint
- added TP135: 3.3V, e-Power:TestPoint_Pad_D1.0mm, symbol Connector:TestPoint
- added TP136: NRST, e-Power:TestPoint_Pad_D1.0mm, symbol Connector:TestPoint
- added TP137: T_SWDIO, e-Power:TestPoint_Pad_D1.0mm, symbol Connector:TestPoint
- added U108: STM32G431CBTx, Package_QFP:LQFP-48_7x7mm_P0.5mm, symbol e-Power:STM32G431CBTx
- added U110: MCP2558FD-xSN, Package_SO:SOIC-8_3.9x4.9mm_P1.27mm, symbol Interface_CAN_LIN:MCP2558FD-xSN
- added Y101: 24MHz, Crystal:Crystal_HC52-6mm_Vertical, symbol Device:Crystal
- added Y102: 32.768KHz, Crystal:Crystal_HC52-6mm_Vertical, symbol Device:Crystal
- renumbered C105 to C106, C106 to C107, C107 to C108, C108 to C113, C112 to C114, C113 to C115, C109 to C118, C110 to C125, C111 to C126, R103 to R105, R104 to R106, R105 to R107, R106 to R108, R107 to R113, R108 to R114, R109 to R115, R110 to R116, R111 to R117, R112 to R118, R113 to R119, R114 to R120, R115 to R121, R116 to R122, R117 to R123, R118 to R124, R119 to R125, R120 to R134, R121 to R135, R122 to R136, R123 to R137, R124 to R138, R125 to R139, R126 to R140, R127 to R141, R128 to R142, R129 to R143, R130 to R144, R131 to R145, R132 to R146, R133 to R147, R134 to R148, R135 to R149, R136 to R150, U108 to U109, U109 to U111, U110 to U112, U111 to U113
Connections:
- net labels added: +3.3V, BOOT0, C_ERROR, ERROR_TRIG, NRST, PB3, RX, S, TX, T_ERROR, T_SWCLK, T_SWDIO, VDDA, V_ERROR, ~ERROR
- net labels removed: BMS_ERROR
- wire segments 485 -> 636
- no-connect marks 9 -> 12
Other:
- note added: "Gen. +12V, +5V, +3.3V"
- note removed: "Generates +12V, +5V"
