File: BMS_24S/current_sensor.sch (KiCad schematic (older format))
At the start: 11 parts, among them J3201 Current_Conn, J3202 BSPD_Conn, J3203 jumper, U3201 LM324

Commit message: update balancing circuit
Parts:
- C3101: renamed from C3201; LCSC (none) -> C49678; Precision (none) -> 10%; Voltage (none) -> 50V
- C3102: renamed from C3202; LCSC (none) -> C49678; Precision (none) -> 10%; Voltage (none) -> 50V
- J3103: renamed from J3203; footprint (none) -> Connector_PinSocket_2.54mm:PinSocket_1x02_P2.54mm_Vertical
- R3101: renamed from R3201; LCSC (none) -> C17414; Power (none) -> 1/8W; Voltage (none) -> 150V
- R3102: renamed from R3202; LCSC (none) -> C17414; Power (none) -> 1/8W; Voltage (none) -> 150V
- R3103: renamed from R3203; LCSC (none) -> C17414; Power (none) -> 1/8W; Voltage (none) -> 150V
- R3104: renamed from R3204; LCSC (none) -> C17414; Power (none) -> 1/8W; Voltage (none) -> 150V
- renumbered J3201 to J3101, J3202 to J3102, JP3201 to JP3101, U3201 to U3101
Changed lines of the file:
@@
 $Descr User 8268 5827
 encoding utf-8
-Sheet 32 32
+Sheet 31 31
 Title ""
 Date ""
@@
 $EndDescr
 $Comp
-L Connector:Conn_01x04_Male J3201
+L Connector:Conn_01x04_Male J3101
 U 1 1 5F3568F3
 P 3000 1700
-F 0 "J3201" H 3000 1300 50  0000 C CNN
+F 0 "J3101" H 3000 1300 50  0000 C CNN
 F 1 "Current_Conn" H 3000 1400 50  0000 C CNN
 F 2 "Connector_PinHeader_2.54mm:PinHeader_1x04_P2.54mm_Horizontal" H 3000 1700 50  0001 C CNN
@@
 AR Path="/5EC24961/5EC7F6A7/5F36FFAB" Ref="U?"  Part="1"
 AR Path="/5EC24961/5EC85226/5F36FFAB" Ref="U?"  Part="1"
-AR Path="/5F3561B0/5F36FFAB" Ref="U3201"  Part="1"
-F 0 "U3201" H 4900 1750 50  0000 C CNN
+AR Path="/5F3561B0/5F36FFAB" Ref="U3101"  Part="1"
+F 0 "U3101" H 4900 1750 50  0000 C CNN
 F 1 "LM324" H 4800 1900 50  0000 C CNN
 F 2 "Package_SO:SOIC-14_3.9x8.7mm_P1.27mm" H 4800 1625 50  0001 C CNN
@@
 Connection ~ 5150 1900
 $Comp
-L power:+5V #PWR03204
+L power:+5V #PWR03104
 U 1 1 5F3710A8
 P 5250 3250
-F 0 "#PWR03204" H 5250 3100 50  0001 C CNN
+F 0 "#PWR03104" H 5250 3100 50  0001 C CNN
 F 1 "+5V" H 5265 3423 50  0000 C CNN
 F 2 "" H 5250 3250 50  0001 C CNN
@@
 $EndComp
 $Comp
-L power:-5V #PWR03203
+L power:-5V #PWR03103
 U 1 1 5F371489
 P 4450 3450
-F 0 "#PWR03203" H 4450 3550 50  0001 C CNN
+F 0 "#PWR03103" H 4450 3550 50  0001 C CNN
 F 1 "-5V" H 4465 3623 50  0000 C CNN
 F 2 "" H 4450 3450 50  0001 C CNN
@@
 5.000V
 $Comp
-L power:GND #PWR03201
+L power:GND #PWR03101
 U 1 1 5F372131
 P 3600 1900
-F 0 "#PWR03201" H 3600 1650 50  0001 C CNN
+F 0 "#PWR03101" H 3600 1650 50  0001 C CNN
 F 1 "GND" H 3605 1727 50  0000 C CNN
 F 2 "" H 3600 1900 50  0001 C CNN
@@
 AR Path="/5EC24961/5EC7F6A7/5F3748A9" Ref="U?"  Part="1"
 AR Path="/5EC24961/5EC85226/5F3748A9" Ref="U?"  Part="1"
-AR Path="/5F3561B0/5F3748A9" Ref="U3201"  Part="5"
-F 0 "U3201" V 4950 3450 50  0000 C CNN
+AR Path="/5F3561B0/5F3748A9" Ref="U3101"  Part="5"
+F 0 "U3101" V 4950 3450 50  0000 C CNN
 F 1 "LM324" V 4850 3450 50  0000 C CNN
 F 2 "Package_SO:SOIC-14_3.9x8.7mm_P1.27mm" H 4850 3175 50  0001 C CNN
@@
 AR Path="/5EC24961/5EC7F6A7/5F37C448" Ref="C?"  Part="1"
 AR Path="/5EC24961/5EC85226/5F37C448" Ref="C?"  Part="1"
-AR Path="/5F3561B0/5F37C448" Ref="C3201"  Part="1"
-F 0 "C3201" H 4315 3646 50  0000 L CNN
+AR Path="/5F3561B0/5F37C448" Ref="C3101"  Part="1"
+F 0 "C3101" H 4315 3646 50  0000 L CNN
 F 1 "100nF" H 4315 3555 50  0000 L CNN
 F 2 "Capacitor_SMD:C_0805_2012Metric" H 4238 3450 50  0001 C CNN
-F 3 "~" H 4200 3600 50  0001 C CNN
+F 3 "https://datasheet.lcsc.com/szlcsc/YAGEO-CC0805KRX7R9BB104_C49678.pdf" H 4200 3600 50  0001 C CNN
+F 4 "C49678" H 4200 3600 50  0001 C CNN "LCSC"
+F 5 "10%" H 4200 3600 50  0001 C CNN "Precision"
+F 6 "50V" H 4200 3600 50  0001 C CNN "Voltage"
 	1    4200 3600
 	-1   0    0    -1
 $EndComp
 $Comp
-L power:GND #PWR03202
+L power:GND #PWR03102
 U 1 1 5F37C9E9
 P 4200 3850
-F 0 "#PWR03202" H 4200 3600 50  0001 C CNN
+F 0 "#PWR03102" H 4200 3600 50  0001 C CNN
 F 1 "GND" H 4205 3677 50  0000 C CNN
 F 2 "" H 4200 3850 50  0001 C CNN
@@
 $EndComp
 $Comp
-L power:GND #PWR03205
+L power:GND #PWR03105
 U 1 1 5F37CD3B
 P 5450 3850
-F 0 "#PWR03205" H 5450 3600 50  0001 C CNN
+F 0 "#PWR03105" H 5450 3600 50  0001 C CNN
 F 1 "GND" H 5455 3677 50  0000 C CNN
 F 2 "" H 5450 3850 50  0001 C CNN
@@
 AR Path="/5EC24961/5EC7F6A7/5F37D4F6" Ref="C?"  Part="1"
 AR Path="/5EC24961/5EC85226/5F37D4F6" Ref="C?"  Part="1"
-AR Path="/5F3561B0/5F37D4F6" Ref="C3202"  Part="1"
-F 0 "C3202" H 5565 3646 50  0000 L CNN
+AR Path="/5F3561B0/5F37D4F6" Ref="C3102"  Part="1"
+F 0 "C3102" H 5565 3646 50  0000 L CNN
 F 1 "100nF" H 5565 3555 50  0000 L CNN
 F 2 "Capacitor_SMD:C_0805_2012Metric" H 5488 3450 50  0001 C CNN
-F 3 "~" H 5450 3600 50  0001 C CNN
+F 3 "https://datasheet.lcsc.com/szlcsc/YAGEO-CC0805KRX7R9BB104_C49678.pdf" H 5450 3600 50  0001 C CNN
+F 4 "C49678" H 5450 3600 50  0001 C CNN "LCSC"
+F 5 "10%" H 5450 3600 50  0001 C CNN "Precision"
+F 6 "50V" H 5450 3600 50  0001 C CNN "Voltage"
 	1    5450 3600
 	1    0    0    -1
@@
 Connection ~ 5250 3350
 $Comp
-L Connector:Conn_01x02_Female J3203
+L Connector:Conn_01x02_Female J3103
 U 1 1 5F391983
 P 3700 1300
-F 0 "J3203" V 3850 1300 50  0000 R CNN
+F 0 "J3103" V 3850 1300 50  0000 R CNN
 F 1 "jumper" V 3750 1350 50  0000 R CNN
-F 2 "" H 3700 1300 50  0001 C CNN
+F 2 "Connector_PinSocket_2.54mm:PinSocket_1x02_P2.54mm_Vertical" H 3700 1300 50  0001 C CNN
 F 3 "~" H 3700 1300 50  0001 C CNN
 	1    3700 1300
@@
 	3800 1500 3800 1600
 $Comp
-L e-Power:Jumper_0805 JP3201
+L e-Power:Jumper_0805 JP3101
 U 1 1 5F395F0C
 P 4100 1400
-F 0 "JP3201" V 4350 1400 50  0000 C CNN
+F 0 "JP3101" V 4350 1400 50  0000 C CNN
 F 1 "jumper" V 4250 1400 50  0000 C CNN
 F 2 "e-Power:zero_ohm_resistor_0805" H 4100 1275 50  0001 C CNN
@@
 AR Path="/5EC24961/5EC7F6A7/5F186021" Ref="U?"  Part="1"
 AR Path="/5EC24961/5EC85226/5F186021" Ref="U?"  Part="1"
-AR Path="/5F3561B0/5F186021" Ref="U3201"  Part="2"
-F 0 "U3201" H 4900 2300 50  0000 C CNN
+AR Path="/5F3561B0/5F186021" Ref="U3101"  Part="2"
+F 0 "U3101" H 4900 2300 50  0000 C CNN
 F 1 "LM324" H 4800 2450 50  0000 C CNN
 F 2 "Package_SO:SOIC-14_3.9x8.7mm_P1.27mm" H 4800 2175 50  0001 C CNN
@@
 Connection ~ 5150 2450
 $Comp
-L Connector:Conn_01x04_Male J3202
+L Connector:Conn_01x04_Male J3102
 U 1 1 5F189870
 P 3000 2700
-F 0 "J3202" H 3000 2300 50  0000 C CNN
+F 0 "J3102" H 3000 2300 50  0000 C CNN
 F 1 "BSPD_Conn" H 3000 2400 50  0000 C CNN
 F 2 "Connector_PinHeader_2.54mm:PinHeader_1x04_P2.54mm_Horizontal" H 3000 2700 50  0001 C CNN
@@
 AR Path="/5EC24961/5EC7F6A7/5F1961F4" Ref="U?"  Part="1"
 AR Path="/5EC24961/5EC85226/5F1961F4" Ref="U?"  Part="1"
-AR Path="/5F3561B0/5F1961F4" Ref="U3201"  Part="3"
-F 0 "U3201" H 6800 1850 50  0000 C CNN
+AR Path="/5F3561B0/5F1961F4" Ref="U3101"  Part="3"
+F 0 "U3101" H 6800 1850 50  0000 C CNN
 F 1 "LM324" H 6700 2000 50  0000 C CNN
 F 2 "Package_SO:SOIC-14_3.9x8.7mm_P1.27mm" H 6700 1725 50  0001 C CNN
@@
 AR Path="/5EC24961/5EC7F6A7/5F19D869" Ref="R?"  Part="1"
 AR Path="/5EC24961/5EC85226/5F19D869" Ref="R?"  Part="1"
-AR Path="/5F3561B0/5F19D869" Ref="R3201"  Part="1"
-F 0 "R3201" V 6050 1900 50  0000 C CNN
+AR Path="/5F3561B0/5F19D869" Ref="R3101"  Part="1"
+F 0 "R3101" V 6050 1900 50  0000 C CNN
 F 1 "10K" V 6150 1900 50  0000 C CNN
 F 2 "Resistor_SMD:R_0805_2012Metric" V 6080 1900 50  0001 C CNN
 F 3 "~" H 6150 1900 50  0001 C CNN
 F 4 "1%" V 5950 1900 50  0000 C CNN "Precision"
+F 5 "C17414" H 6150 1900 50  0001 C CNN "LCSC"
+F 6 "1/8W" H 6150 1900 50  0001 C CNN "Power"
+F 7 "150V" H 6150 1900 50  0001 C CNN "Voltage"
 	1    6150 1900
 	0    1    1    0
@@
 AR Path="/5EC24961/5EC7F6A7/5F19E141" Ref="R?"  Part="1"
 AR Path="/5EC24961/5EC85226/5F19E141" Ref="R?"  Part="1"
-AR Path="/5F3561B0/5F19E141" Ref="R3202"  Part="1"
-F 0 "R3202" V 6250 2100 50  0000 C CNN
+AR Path="/5F3561B0/5F19E141" Ref="R3102"  Part="1"
+F 0 "R3102" V 6250 2100 50  0000 C CNN
 F 1 "10K" V 6150 2100 50  0000 C CNN
 F 2 "Resistor_SMD:R_0805_2012Metric" V 6080 2100 50  0001 C CNN
 F 3 "~" H 6150 2100 50  0001 C CNN
 F 4 "1%" V 6350 2100 50  0000 C CNN "Precision"
+F 5 "C17414" H 6150 2100 50  0001 C CNN "LCSC"
+F 6 "1/8W" H 6150 2100 50  0001 C CNN "Power"
+F 7 "150V" H 6150 2100 50  0001 C CNN "Voltage"
 	1    6150 2100
 	0    1    1    0
@@
 AR Path="/5EC24961/5EC7F6A7/5F19E3C2" Ref="R?"  Part="1"
 AR Path="/5EC24961/5EC85226/5F19E3C2" Ref="R?"  Part="1"
-AR Path="/5F3561B0/5F19E3C2" Ref="R3203"  Part="1"
-F 0 "R3203" H 6150 2400 50  0000 C CNN
+AR Path="/5F3561B0/5F19E3C2" Ref="R3103"  Part="1"
+F 0 "R3103" H 6150 2400 50  0000 C CNN
 F 1 "10K" V 6350 2350 50  0000 C CNN
 F 2 "Resistor_SMD:R_0805_2012Metric" V 6280 2350 50  0001 C CNN
 F 3 "~" H 6350 2350 50  0001 C CNN
 F 4 "1%" H 6200 2300 50  0000 C CNN "Precision"
+F 5 "C17414" H 6350 2350 50  0001 C CNN "LCSC"
+F 6 "1/8W" H 6350 2350 50  0001 C CNN "Power"
+F 7 "150V" H 6350 2350 50  0001 C CNN "Voltage"
 	1    6350 2350
 	-1   0    0    1
@@
 AR Path="/5EC24961/5EC7F6A7/5F19EB05" Ref="R?"  Part="1"
 AR Path="/5EC24961/5EC85226/5F19EB05" Ref="R?"  Part="1"
-AR Path="/5F3561B0/5F19EB05" Ref="R3204"  Part="1"
-F 0 "R3204" V 6800 1650 50  0000 C CNN
+AR Path="/5F3561B0/5F19EB05" Ref="R3104"  Part="1"
+F 0 "R3104" V 6800 1650 50  0000 C CNN
 F 1 "10K" V 6700 1650 50  0000 C CNN
 F 2 "Resistor_SMD:R_0805_2012Metric" V 6630 1650 50  0001 C CNN
 F 3 "~" H 6700 1650 50  0001 C CNN
 F 4 "1%" V 6900 1650 50  0000 C CNN "Precision"
+F 5 "C17414" H 6700 1650 50  0001 C CNN "LCSC"
+F 6 "1/8W" H 6700 1650 50  0001 C CNN "Power"
+F 7 "150V" H 6700 1650 50  0001 C CNN "Voltage"
 	1    6700 1650
 	0    -1   -1   0
 $EndComp
 $Comp
-L power:GND #PWR03206
+L power:GND #PWR03106
 U 1 1 5F1A5F0B
 P 6350 2550
-F 0 "#PWR03206" H 6350 2300 50  0001 C CNN
+F 0 "#PWR03106" H 6350 2300 50  0001 C CNN
 F 1 "GND" H 6355 2377 50  0000 C CNN
 F 2 "" H 6350 2550 50  0001 C CNN

Commit message: updates made on BMS
Parts:
- removed J3103: jumper, Connector_PinSocket_2.54mm:PinSocket_1x02_P2.54mm_Vertical, symbol Connector:Conn_01x02_Female
- removed JP3101: jumper, e-Power:zero_ohm_resistor_0805, symbol e-Power:Jumper_0805
- added JP3101: Jumper, Jumper:SolderJumper-2_P1.3mm_Open_TrianglePad1.0x1.5mm, symbol Device:Jumper
- added R3105: 0R, Resistor_SMD:R_0805_2012Metric, symbol Device:R
- renumbered J3101 to J3102, J3102 to J3103, R3104 to R3101, R3101 to R3102, R3102 to R3103, R3103 to R3104
Connections:
- wire segments 57 -> 54
Changed lines of the file:
@@
 $EndDescr
 $Comp
-L Connector:Conn_01x04_Male J3101
+L Connector:Conn_01x04_Male J3102
 U 1 1 5F3568F3
 P 3000 1700
-F 0 "J3101" H 3000 1300 50  0000 C CNN
+F 0 "J3102" H 3000 1300 50  0000 C CNN
 F 1 "Current_Conn" H 3000 1400 50  0000 C CNN
 F 2 "Connector_PinHeader_2.54mm:PinHeader_1x04_P2.54mm_Horizontal" H 3000 1700 50  0001 C CNN
@@
 Connection ~ 5150 1900
 $Comp
-L power:+5V #PWR03104
+L power:+5V #PWR03103
 U 1 1 5F3710A8
 P 5250 3250
-F 0 "#PWR03104" H 5250 3100 50  0001 C CNN
+F 0 "#PWR03103" H 5250 3100 50  0001 C CNN
 F 1 "+5V" H 5265 3423 50  0000 C CNN
 F 2 "" H 5250 3250 50  0001 C CNN
@@
 $EndComp
 $Comp
-L power:-5V #PWR03103
+L power:-5V #PWR03104
 U 1 1 5F371489
 P 4450 3450
-F 0 "#PWR03103" H 4450 3550 50  0001 C CNN
+F 0 "#PWR03104" H 4450 3550 50  0001 C CNN
 F 1 "-5V" H 4465 3623 50  0000 C CNN
 F 2 "" H 4450 3450 50  0001 C CNN
@@
 	-1   0    0    1
 $EndComp
-Text HLabel 4200 1600 2    50   Input ~ 0
+Text HLabel 4700 1600 2    50   Input ~ 0
 5.000V
 $Comp
@@
 $EndComp
 $Comp
-L power:GND #PWR03102
+L power:GND #PWR03105
 U 1 1 5F37C9E9
 P 4200 3850
-F 0 "#PWR03102" H 4200 3600 50  0001 C CNN
+F 0 "#PWR03105" H 4200 3600 50  0001 C CNN
 F 1 "GND" H 4205 3677 50  0000 C CNN
 F 2 "" H 4200 3850 50  0001 C CNN
@@
 $EndComp
 $Comp
-L power:GND #PWR03105
+L power:GND #PWR03106
 U 1 1 5F37CD3B
 P 5450 3850
-F 0 "#PWR03105" H 5450 3600 50  0001 C CNN
+F 0 "#PWR03106" H 5450 3600 50  0001 C CNN
 F 1 "GND" H 5455 3677 50  0000 C CNN
 F 2 "" H 5450 3850 50  0001 C CNN
@@
 Wire Wire Line
 	5450 3850 5450 3750
+Text HLabel 5550 3350 2    50   Input ~ 0
++5V
 Text HLabel 4100 3350 0    50   Input ~ 0
-+5V
-Text HLabel 5550 3350 2    50   Input ~ 0
 -5V
 Wire Wire Line
@@
 	5250 3350 5450 3350
 Connection ~ 5250 3350
-$Comp
-L Connector:Conn_01x02_Female J3103
-U 1 1 5F391983
-P 3700 1300
-F 0 "J3103" V 3850 1300 50  0000 R CNN
-F 1 "jumper" V 3750 1350 50  0000 R CNN
-F 2 "Connector_PinSocket_2.54mm:PinSocket_1x02_P2.54mm_Vertical" H 3700 1300 50  0001 C CNN
-F 3 "~" H 3700 1300 50  0001 C CNN
-	1    3700 1300
-	0    -1   -1   0
-$EndComp
-Wire Wire Line
-	3700 1600 3700 1500
-Wire Wire Line
-	3200 1600 3700 1600
-Wire Wire Line
-	3800 1500 3800 1600
-$Comp
-L e-Power:Jumper_0805 JP3101
-U 1 1 5F395F0C
-P 4100 1400
-F 0 "JP3101" V 4350 1400 50  0000 C CNN
-F 1 "jumper" V 4250 1400 50  0000 C CNN
-F 2 "e-Power:zero_ohm_resistor_0805" H 4100 1275 50  0001 C CNN
-F 3 "" H 4100 1400 50  0001 C CNN
-	1    4100 1400
-	0    -1   -1   0
-$EndComp
-Wire Wire Line
-	3800 1600 4100 1600
-Wire Wire Line
-	4100 1500 4100 1600
-Connection ~ 4100 1600
-Wire Wire Line
-	4100 1600 4200 1600
 $Comp
 L e-Power:LM324 U?
@@
 Connection ~ 5150 2450
 $Comp
-L Connector:Conn_01x04_Male J3102
+L Connector:Conn_01x04_Male J3103
 U 1 1 5F189870
 P 3000 2700
-F 0 "J3102" H 3000 2300 50  0000 C CNN
+F 0 "J3103" H 3000 2300 50  0000 C CNN
 F 1 "BSPD_Conn" H 3000 2400 50  0000 C CNN
 F 2 "Connector_PinHeader_2.54mm:PinHeader_1x04_P2.54mm_Horizontal" H 3000 2700 50  0001 C CNN
@@
 AR Path="/5EC24961/5EC7F6A7/5F19D869" Ref="R?"  Part="1"
 AR Path="/5EC24961/5EC85226/5F19D869" Ref="R?"  Part="1"
-AR Path="/5F3561B0/5F19D869" Ref="R3101"  Part="1"
-F 0 "R3101" V 6050 1900 50  0000 C CNN
+AR Path="/5F3561B0/5F19D869" Ref="R3102"  Part="1"
+F 0 "R3102" V 6050 1900 50  0000 C CNN
 F 1 "10K" V 6150 1900 50  0000 C CNN
 F 2 "Resistor_SMD:R_0805_2012Metric" V 6080 1900 50  0001 C CNN
@@
 AR Path="/5EC24961/5EC7F6A7/5F19E141" Ref="R?"  Part="1"
 AR Path="/5EC24961/5EC85226/5F19E141" Ref="R?"  Part="1"
-AR Path="/5F3561B0/5F19E141" Ref="R3102"  Part="1"
-F 0 "R3102" V 6250 2100 50  0000 C CNN
+AR Path="/5F3561B0/5F19E141" Ref="R3103"  Part="1"
+F 0 "R3103" V 6250 2100 50  0000 C CNN
 F 1 "10K" V 6150 2100 50  0000 C CNN
 F 2 "Resistor_SMD:R_0805_2012Metric" V 6080 2100 50  0001 C CNN
@@
 AR Path="/5EC24961/5EC7F6A7/5F19E3C2" Ref="R?"  Part="1"
 AR Path="/5EC24961/5EC85226/5F19E3C2" Ref="R?"  Part="1"
-AR Path="/5F3561B0/5F19E3C2" Ref="R3103"  Part="1"
-F 0 "R3103" H 6150 2400 50  0000 C CNN
+AR Path="/5F3561B0/5F19E3C2" Ref="R3104"  Part="1"
+F 0 "R3104" H 6150 2400 50  0000 C CNN
 F 1 "10K" V 6350 2350 50  0000 C CNN
 F 2 "Resistor_SMD:R_0805_2012Metric" V 6280 2350 50  0001 C CNN
@@
 AR Path="/5EC24961/5EC7F6A7/5F19EB05" Ref="R?"  Part="1"
 AR Path="/5EC24961/5EC85226/5F19EB05" Ref="R?"  Part="1"
-AR Path="/5F3561B0/5F19EB05" Ref="R3104"  Part="1"
-F 0 "R3104" V 6800 1650 50  0000 C CNN
+AR Path="/5F3561B0/5F19EB05" Ref="R3101"  Part="1"
+F 0 "R3101" V 6800 1650 50  0000 C CNN
 F 1 "10K" V 6700 1650 50  0000 C CNN
 F 2 "Resistor_SMD:R_0805_2012Metric" V 6630 1650 50  0001 C CNN
@@
 $EndComp
 $Comp
-L power:GND #PWR03106
+L power:GND #PWR03102
 U 1 1 5F1A5F0B
 P 6350 2550
-F 0 "#PWR03106" H 6350 2300 50  0001 C CNN
+F 0 "#PWR03102" H 6350 2300 50  0001 C CNN
 F 1 "GND" H 6355 2377 50  0000 C CNN
 F 2 "" H 6350 2550 50  0001 C CNN
@@
 Wire Wire Line
 	5850 2100 6000 2100
+$Comp
+L Device:Jumper JP3101
+U 1 1 629BB045
+P 3900 1600
+F 0 "JP3101" H 3900 1864 50  0000 C CNN
+F 1 "Jumper" H 3900 1773 50  0000 C CNN
+F 2 "Jumper:SolderJumper-2_P1.3mm_Open_TrianglePad1.0x1.5mm" H 3900 1600 50  0001 C CNN
+F 3 "~" H 3900 1600 50  0001 C CNN
+	1    3900 1600
+	1    0    0    -1
+$EndComp
+Wire Wire Line
+	4700 1600 4600 1600
+Wire Wire Line
+	4300 1600 4200 1600
+Wire Wire Line
+	3600 1600 3200 1600
+$Comp
+L Device:R R?
+U 1 1 629BD18A
+P 4450 1600
+AR Path="/5EA47040/629BD18A" Ref="R?"  Part="1"
+AR Path="/5EA471BF/629BD18A" Ref="R?"  Part="1"
+AR Path="/5EEF4361/629BD18A" Ref="R?"  Part="1"
+AR Path="/5EEF524D/629BD18A" Ref="R?"  Part="1"
+AR Path="/5EC044AE/5EC054C7/629BD18A" Ref="R?"  Part="1"
+AR Path="/5EC044AE/5EC39151/629BD18A" Ref="R?"  Part="1"
+AR Path="/5EC24961/5EC054C7/629BD18A" Ref="R?"  Part="1"
+AR Path="/5EC24961/5EC3A225/629BD18A" Ref="R?"  Part="1"
+AR Path="/5EC24961/5EC4031A/629BD18A" Ref="R?"  Part="1"
+AR Path="/5EC24961/5EC462FD/629BD18A" Ref="R?"  Part="1"
+AR Path="/5EC24961/5EC4BDFE/629BD18A" Ref="R?"  Part="1"
+AR Path="/5EC24961/5EC51A1F/629BD18A" Ref="R?"  Part="1"
+AR Path="/5EC24961/5EC574F6/629BD18A" Ref="R?"  Part="1"
+AR Path="/5EC24961/5EC5D2D3/629BD18A" Ref="R?"  Part="1"
+AR Path="/5EC24961/5EC62E5E/629BD18A" Ref="R?"  Part="1"
+AR Path="/5EC24961/5EC6897D/629BD18A" Ref="R?"  Part="1"
+AR Path="/5EC24961/5EC6E4EA/629BD18A" Ref="R?"  Part="1"
+AR Path="/5EC24961/5EC74033/629BD18A" Ref="R?"  Part="1"
+AR Path="/5EC24961/5EC79B70/629BD18A" Ref="R?"  Part="1"
+AR Path="/5EC24961/5EC7F6A7/629BD18A" Ref="R?"  Part="1"
+AR Path="/5EC24961/5EC85226/629BD18A" Ref="R?"  Part="1"
+AR Path="/5F3561B0/629BD18A" Ref="R3105"  Part="1"
+F 0 "R3105" V 4350 1600 50  0000 C CNN
+F 1 "0R" V 4450 1600 50  0000 C CNN
+F 2 "Resistor_SMD:R_0805_2012Metric" V 4380 1600 50  0001 C CNN
+F 3 "~" H 4450 1600 50  0001 C CNN
+F 4 "1%" V 4250 1600 50  0001 C CNN "Precision"
+F 5 "C17414" H 4450 1600 50  0001 C CNN "LCSC"
+F 6 "1/8W" H 4450 1600 50  0001 C CNN "Power"
+F 7 "150V" H 4450 1600 50  0001 C CNN "Voltage"
+	1    4450 1600
+	0    1    1    0
+$EndComp
 $EndSCHEMATC
