File: BMS_24S/voltage_1_2.sch (KiCad schematic (older format))
At the start: 30 parts, among them U501 TS1851ILT, U502 TS1851ILT, U503 TLP290-4

Commit message: update balancing circuit
Parts:
- C501: LCSC (none) -> C49678; Precision (none) -> 10%; Voltage (none) -> 50V
- JP501, JP502, JP503, JP504: LCSC (none) -> C17477; Power (none) -> 1/8W; Precision (none) -> 1%; Voltage (none) -> 150V
- R501, R502, R503, R504, R505, R506, R507, R508, R509, R510, R511, R512, R513, R514, R515, R516: LCSC (none) -> C17513; Power (none) -> 1/8W; Precision (none) -> 1%; Voltage (none) -> 150V

Commit message: updates made on BMS
Parts:
- removed JP503: 0R, e-Power:zero_ohm_resistor_0805, symbol e-Power:Jumper_0805
- added C502, C503: 100nF, Capacitor_SMD:C_0805_2012Metric, symbol Device:C
- renumbered D503 to D502, D505 to D503, D502 to D504, D504 to D505, JP502 to JP501, JP504 to JP503, JP501 to JP504, R503 to R501, R505 to R502, R507 to R503, R509 to R504, R501 to R505, R511 to R506, R515 to R507, R516 to R508, R504 to R509, R506 to R510, R508 to R511, R510 to R512, R502 to R513, R512 to R514, R513 to R515, R514 to R516, U503 to U502, U502 to U503
Connections:
- net GND: now also C502.2, C503.2
- net V_01: now also C503.1
- net V_02: now also C502.1

Commit message: update bms pcb
Parts:
- D501, D502, D503, D504, D505, D506: LCSC (none) -> C9808
- renumbered JP503 to JP502, JP504 to JP503

Commit message: updates made on bms, almost done
Parts:
- JP501, JP502, JP503: LCSC C17477 -> (none)
- U502: LCSC (none) -> C39031
Changed lines of the file:
@@
 $Descr User 7087 6299
 encoding utf-8
-Sheet 16 31
+Sheet 8 31
 Title ""
 Date "2020-04-26"
@@
 F 2 "e-Power:SOIC-16_4.55x10.3mm_P1.27mm(TLP290-4)" H 4450 2050 50  0001 L CIN
 F 3 "https://toshiba.semicon-storage.com/info/docget.jsp?did=12855&prodName=TLP290-4" H 5325 2250 50  0001 L CNN
+F 4 "C39031" H 5300 2250 50  0001 C CNN "LCSC"
 	1    5300 2250
 	1    0    0    -1
@@
 F 2 "e-Power:SOIC-16_4.55x10.3mm_P1.27mm(TLP290-4)" H 4450 2450 50  0001 L CIN
 F 3 "https://toshiba.semicon-storage.com/info/docget.jsp?did=12855&prodName=TLP290-4" H 5325 2650 50  0001 L CNN
+F 4 "C39031" H 5300 2650 50  0001 C CNN "LCSC"
 	2    5300 2650
 	1    0    0    -1
@@
 F 2 "e-Power:SOIC-16_4.55x10.3mm_P1.27mm(TLP290-4)" H 4450 3400 50  0001 L CIN
 F 3 "https://toshiba.semicon-storage.com/info/docget.jsp?did=12855&prodName=TLP290-4" H 5325 3600 50  0001 L CNN
+F 4 "C39031" H 5300 3600 50  0001 C CNN "LCSC"
 	3    5300 3600
 	1    0    0    -1
@@
 F 2 "e-Power:SOIC-16_4.55x10.3mm_P1.27mm(TLP290-4)" H 4450 3800 50  0001 L CIN
 F 3 "https://toshiba.semicon-storage.com/info/docget.jsp?did=12855&prodName=TLP290-4" H 5325 4000 50  0001 L CNN
+F 4 "C39031" H 5300 4000 50  0001 C CNN "LCSC"
 	4    5300 4000
 	1    0    0    -1
@@
 F 2 "e-Power:zero_ohm_resistor_0805" H 4500 1525 50  0001 C CNN
 F 3 "~" H 4500 1650 50  0001 C CNN
-F 4 "C17477" H 4500 1650 50  0001 C CNN "LCSC"
+F 4 "" H 4500 1650 50  0001 C CNN "LCSC"
 F 5 "1/8W" H 4500 1650 50  0001 C CNN "Power"
 F 6 "1%" H 4500 1650 50  0001 C CNN "Precision"
@@
 F 2 "e-Power:zero_ohm_resistor_0805" H 4100 3925 50  0001 C CNN
 F 3 "~" H 4100 4050 50  0001 C CNN
-F 4 "C17477" H 4100 4050 50  0001 C CNN "LCSC"
+F 4 "" H 4100 4050 50  0001 C CNN "LCSC"
 F 5 "1/8W" H 4100 4050 50  0001 C CNN "Power"
 F 6 "1%" H 4100 4050 50  0001 C CNN "Precision"
@@
 F 2 "e-Power:zero_ohm_resistor_0805" H 6150 3725 50  0001 C CNN
 F 3 "~" H 6150 3850 50  0001 C CNN
-F 4 "C17477" H 6150 3850 50  0001 C CNN "LCSC"
+F 4 "" H 6150 3850 50  0001 C CNN "LCSC"
 F 5 "1/8W" H 6150 3850 50  0001 C CNN "Power"
 F 6 "1%" H 6150 3850 50  0001 C CNN "Precision"
