File: BMS_24S/LM235_1_2_3_4.sch (KiCad schematic (older format))
At the start: 6 parts, among them U2001 LM324

Commit message: updates made on BMS
Parts:
- renumbered R2003 to R2002, R2002 to R2003

Commit message: get BSPD
Parts:
- U2001: LCSC (none) -> C71035
Changed lines of the file:
@@
 $Descr User 7874 4725
 encoding utf-8
-Sheet 20 31
+Sheet 23 31
 Title ""
 Date ""
@@
 F 2 "Package_SO:SOIC-14_3.9x8.7mm_P1.27mm" H 1400 2825 50  0001 C CNN
 F 3 "http://www.ti.com/lit/ds/symlink/lm2902-n.pdf" H 1450 3300 50  0001 C CNN
+F 4 "C71035" H 1400 3100 50  0001 C CNN "LCSC"
 	5    1400 3100
 	0    1    1    0
@@
 F 2 "Package_SO:SOIC-14_3.9x8.7mm_P1.27mm" H 1950 975 50  0001 C CNN
 F 3 "http://www.ti.com/lit/ds/symlink/lm2902-n.pdf" H 2000 1450 50  0001 C CNN
+F 4 "C71035" H 1950 1250 50  0001 C CNN "LCSC"
 	1    1950 1250
 	1    0    0    -1
@@
 F 2 "Package_SO:SOIC-14_3.9x8.7mm_P1.27mm" H 1950 1675 50  0001 C CNN
 F 3 "http://www.ti.com/lit/ds/symlink/lm2902-n.pdf" H 2000 2150 50  0001 C CNN
+F 4 "C71035" H 1950 1950 50  0001 C CNN "LCSC"
 	2    1950 1950
 	1    0    0    -1
@@
 F 2 "Package_SO:SOIC-14_3.9x8.7mm_P1.27mm" H 3850 975 50  0001 C CNN
 F 3 "http://www.ti.com/lit/ds/symlink/lm2902-n.pdf" H 3900 1450 50  0001 C CNN
+F 4 "C71035" H 3850 1250 50  0001 C CNN "LCSC"
 	3    3850 1250
 	1    0    0    -1
@@
 F 2 "Package_SO:SOIC-14_3.9x8.7mm_P1.27mm" H 3850 1675 50  0001 C CNN
 F 3 "http://www.ti.com/lit/ds/symlink/lm2902-n.pdf" H 3900 2150 50  0001 C CNN
+F 4 "C71035" H 3850 1950 50  0001 C CNN "LCSC"
 	4    3850 1950
 	1    0    0    -1

Commit message: layout final bms temp
Changed lines of the file:
@@
 AR Path="/5EC24961/5F67B671/5EA4C987" Ref="U2201"  Part="5"
 AR Path="/5EC24961/5F6A1F0B/5EA4C987" Ref="U2301"  Part="5"
-F 0 "U2301" V 1075 3100 50  0000 C CNN
+F 0 "U2001" V 1075 3100 50  0000 C CNN
 F 1 "LM324" V 1166 3100 50  0000 C CNN
 F 2 "Package_SO:SOIC-14_3.9x8.7mm_P1.27mm" H 1400 2825 50  0001 C CNN
@@
 AR Path="/5EC24961/5F67B671/5EC12A8F" Ref="R2203"  Part="1"
 AR Path="/5EC24961/5F6A1F0B/5EC12A8F" Ref="R2303"  Part="1"
-F 0 "R2303" V 1300 1700 50  0000 C CNN
+F 0 "R2003" V 1300 1700 50  0000 C CNN
 F 1 "1K" V 1400 1700 50  0000 C CNN
 F 2 "Resistor_SMD:R_0805_2012Metric" V 1330 1700 50  0001 C CNN
@@
 AR Path="/5EC24961/5F67B671/5EC12A91" Ref="#PWR02203"  Part="1"
 AR Path="/5EC24961/5F6A1F0B/5EC12A91" Ref="#PWR02303"  Part="1"
-F 0 "#PWR02303" H 1200 1550 50  0001 C CNN
+F 0 "#PWR02003" H 1200 1550 50  0001 C CNN
 F 1 "+5V" H 1215 1873 50  0000 C CNN
 F 2 "" H 1200 1700 50  0001 C CNN
@@
 AR Path="/5EC24961/5F67B671/5EC12A90" Ref="#PWR02201"  Part="1"
 AR Path="/5EC24961/5F6A1F0B/5EC12A90" Ref="#PWR02301"  Part="1"
-F 0 "#PWR02301" H 1200 850 50  0001 C CNN
+F 0 "#PWR02001" H 1200 850 50  0001 C CNN
 F 1 "+5V" H 1215 1173 50  0000 C CNN
 F 2 "" H 1200 1000 50  0001 C CNN
@@
 AR Path="/5EC24961/5F67B671/5EC12A8E" Ref="R2201"  Part="1"
 AR Path="/5EC24961/5F6A1F0B/5EC12A8E" Ref="R2301"  Part="1"
-F 0 "R2301" V 1300 1000 50  0000 C CNN
+F 0 "R2001" V 1300 1000 50  0000 C CNN
 F 1 "1K" V 1400 1000 50  0000 C CNN
 F 2 "Resistor_SMD:R_0805_2012Metric" V 1330 1000 50  0001 C CNN
@@
 AR Path="/5EC24961/5F67B671/5EC12A89" Ref="U2201"  Part="1"
 AR Path="/5EC24961/5F6A1F0B/5EC12A89" Ref="U2301"  Part="1"
-F 0 "U2301" H 2050 1100 50  0000 C CNN
+F 0 "U2001" H 2050 1100 50  0000 C CNN
 F 1 "LM324" H 1950 1250 50  0000 C CNN
 F 2 "Package_SO:SOIC-14_3.9x8.7mm_P1.27mm" H 1950 975 50  0001 C CNN
@@
 AR Path="/5EC24961/5F67B671/5EC12AA0" Ref="#PWR02205"  Part="1"
 AR Path="/5EC24961/5F6A1F0B/5EC12AA0" Ref="#PWR02305"  Part="1"
-F 0 "#PWR02305" H 1800 2750 50  0001 C CNN
+F 0 "#PWR02005" H 1800 2750 50  0001 C CNN
 F 1 "+5V" H 1815 3073 50  0000 C CNN
 F 2 "" H 1800 2900 50  0001 C CNN
@@
 AR Path="/5EC24961/5F67B671/5EC12AA2" Ref="C2201"  Part="1"
 AR Path="/5EC24961/5F6A1F0B/5EC12AA2" Ref="C2301"  Part="1"
-F 0 "C2301" H 1915 3296 50  0000 L CNN
+F 0 "C2001" H 1915 3296 50  0000 L CNN
 F 1 "100nF" H 1915 3205 50  0000 L CNN
 F 2 "Capacitor_SMD:C_0805_2012Metric" H 1838 3100 50  0001 C CNN
@@
 AR Path="/5EC24961/5F67B671/5EC12AA4" Ref="#PWR02207"  Part="1"
 AR Path="/5EC24961/5F6A1F0B/5EC12AA4" Ref="#PWR02307"  Part="1"
-F 0 "#PWR02307" H 1800 3250 50  0001 C CNN
+F 0 "#PWR02007" H 1800 3250 50  0001 C CNN
 F 1 "GND" H 1805 3327 50  0000 C CNN
 F 2 "" H 1800 3500 50  0001 C CNN
@@
 AR Path="/5EC24961/5F67B671/5EC12AA5" Ref="#PWR02206"  Part="1"
 AR Path="/5EC24961/5F6A1F0B/5EC12AA5" Ref="#PWR02306"  Part="1"
-F 0 "#PWR02306" H 1000 3250 50  0001 C CNN
+F 0 "#PWR02006" H 1000 3250 50  0001 C CNN
 F 1 "GND" H 1005 3327 50  0000 C CNN
 F 2 "" H 1000 3500 50  0001 C CNN
@@
 AR Path="/5EC24961/5F67B671/5EA4A09D" Ref="U2201"  Part="2"
 AR Path="/5EC24961/5F6A1F0B/5EA4A09D" Ref="U2301"  Part="2"
-F 0 "U2301" H 2050 1800 50  0000 C CNN
+F 0 "U2001" H 2050 1800 50  0000 C CNN
 F 1 "LM324" H 1900 1950 50  0000 C CNN
 F 2 "Package_SO:SOIC-14_3.9x8.7mm_P1.27mm" H 1950 1675 50  0001 C CNN
@@
 AR Path="/5EC24961/5F67B671/5F5E9DCD" Ref="R2204"  Part="1"
 AR Path="/5EC24961/5F6A1F0B/5F5E9DCD" Ref="R2304"  Part="1"
-F 0 "R2304" V 3200 1700 50  0000 C CNN
+F 0 "R2004" V 3200 1700 50  0000 C CNN
 F 1 "1K" V 3300 1700 50  0000 C CNN
 F 2 "Resistor_SMD:R_0805_2012Metric" V 3230 1700 50  0001 C CNN
@@
 AR Path="/5EC24961/5F67B671/5F5E9DD7" Ref="#PWR02204"  Part="1"
 AR Path="/5EC24961/5F6A1F0B/5F5E9DD7" Ref="#PWR02304"  Part="1"
-F 0 "#PWR02304" H 3100 1550 50  0001 C CNN
+F 0 "#PWR02004" H 3100 1550 50  0001 C CNN
 F 1 "+5V" H 3115 1873 50  0000 C CNN
 F 2 "" H 3100 1700 50  0001 C CNN
@@
 AR Path="/5EC24961/5F67B671/5F5E9DF4" Ref="#PWR02202"  Part="1"
 AR Path="/5EC24961/5F6A1F0B/5F5E9DF4" Ref="#PWR02302"  Part="1"
-F 0 "#PWR02302" H 3100 850 50  0001 C CNN
+F 0 "#PWR02002" H 3100 850 50  0001 C CNN
 F 1 "+5V" H 3115 1173 50  0000 C CNN
 F 2 "" H 3100 1000 50  0001 C CNN
@@
 AR Path="/5EC24961/5F67B671/5F5E9E02" Ref="R2202"  Part="1"
 AR Path="/5EC24961/5F6A1F0B/5F5E9E02" Ref="R2302"  Part="1"
-F 0 "R2302" V 3200 1000 50  0000 C CNN
+F 0 "R2002" V 3200 1000 50  0000 C CNN
 F 1 "1K" V 3300 1000 50  0000 C CNN
 F 2 "Resistor_SMD:R_0805_2012Metric" V 3230 1000 50  0001 C CNN
@@
 AR Path="/5EC24961/5F67B671/5F5E9E0E" Ref="U2201"  Part="3"
 AR Path="/5EC24961/5F6A1F0B/5F5E9E0E" Ref="U2301"  Part="3"
-F 0 "U2301" H 3950 1100 50  0000 C CNN
+F 0 "U2001" H 3950 1100 50  0000 C CNN
 F 1 "LM324" H 3850 1250 50  0000 C CNN
 F 2 "Package_SO:SOIC-14_3.9x8.7mm_P1.27mm" H 3850 975 50  0001 C CNN
@@
 AR Path="/5EC24961/5F67B671/5F5E9E1B" Ref="U2201"  Part="4"
 AR Path="/5EC24961/5F6A1F0B/5F5E9E1B" Ref="U2301"  Part="4"
-F 0 "U2301" H 3950 1800 50  0000 C CNN
+F 0 "U2001" H 3950 1800 50  0000 C CNN
 F 1 "LM324" H 3800 1950 50  0000 C CNN
 F 2 "Package_SO:SOIC-14_3.9x8.7mm_P1.27mm" H 3850 1675 50  0001 C CNN
