File: UFRGS-PILL/UFRGS PILL.sch (KiCad schematic (older format))
At the start: 38 parts, among them J1 ST-LINK, J2 USB_B_Micro, J3 CONN_01x20, J4 CONN_01x20, SW1 SW_Push, U1 AZ1117-3.3, U2 STM32G431CBTx, Y1 24MHz, Y2 32K768Hz

Commit message: backup AIL
Parts:
- SW1: footprint e-Power:SW_Push_1P1T_NO_6x6mm_H9.5mm -> e-Power:SW_SPST_CK_8.0x2.5x3.65mm
Changed lines of the file:
@@
 F 0 "SW1" H 7850 2435 50  0000 C CNN
 F 1 "SW_Push" H 7850 2344 50  0000 C CNN
-F 2 "e-Power:SW_Push_1P1T_NO_6x6mm_H9.5mm" H 7850 2350 50  0001 C CNN
+F 2 "e-Power:SW_SPST_CK_8.0x2.5x3.65mm" H 7850 2350 50  0001 C CNN
 F 3 "~" H 7850 2350 50  0001 C CNN
 	1    7850 2150
