File: UFRGS-PILL/UFRGS PILL.kicad_pcb (KiCad board)
At the start: 2 copper layers, 56.6 x 21.3 mm, 38 parts, among them J1 ST-LINK, J2 USB_B_Micro, J3 CONN_01x20, J4 CONN_01x20, SW1 SW_Push, U1 AZ1117-3.3, U2 STM32G431CBTx, Y1 24MHz, Y2 32K768Hz

Commit message: backup AIL
Parts:
- SW1: footprint e-Power:SW_Push_1P1T_NO_6x6mm_H9.5mm -> e-Power:SW_SPST_CK_8.0x2.5x3.65mm
- moved SW1 1.02 mm to (114.8, 47.2)
Routing:
- net NRST: track 77.4 -> 65.7 mm
- net +3V3: track 101.4 -> 98.1 mm
- net VDDA: track 26.8 -> 23.8 mm
- net T_SWCLK: track 39.4 -> 37.6 mm
- net USB_DM: track 39.3 -> 37.8 mm
- net Net-(C15-Pad1): track 14.7 -> 14.0 mm
- net PB9: track 27.7 -> 27.1 mm
Other:
- outline, holes or cut-outs redrawn

Commit message: generate gerbers and add powertrain pcbs
Parts:
- added C1: 100nF, Capacitor_SMD:C_0805_2012Metric_Pad1.15x1.40mm_HandSolder, B.Cu at (121.9, 48.3)
- added SW1: SW_Push, e-Power:SW_SPST_CK_8.0x2.5x3.65mm, F.Cu at (119.9, 47.2)
- renumbered C15 to C10, C1 to C11, C2 to C12, C3 to C13, C6 to C14, C7 to C15, C9 to C16, C11 to C2, C12 to C3, C13 to C4, C4 to C5, C5 to C6, C8 to C7, C10 to C8, C14 to C9, J3 to J2, J4 to J3, J2 to J4, R8 to R2, R2 to R3, SW1 to SW2
Routing:
- net NRST: track 65.7 -> 92.6 mm, vias 3 -> 7
- net PA10: track 6.72 -> 32.1 mm, vias 0 -> 2
- net +3V3: track 98.1 -> 94.4 mm
- net GND: track 234.5 -> 236.8 mm
Other:
- board text removed: "03/2020"

Commit message: add small option panel board
Parts:
- added G***: LOGO, e-Power:Logo_UFRGS_11.0x6.0mm_SilkS, B.Cu at (132.8, 52.1)
- added G***: e-Power_12.4x6.0mm, e-Power:Logo_e-Power_12.4x6.0mm_SilkS, B.Cu at (132.7, 44.5)
- moved C2 1.27 mm to (111.3, 51.6)
Routing:
- net NRST: track 92.6 -> 95.5 mm
- net GND: track 236.8 -> 235.1 mm
Other:
- board text added: "3V3"
- board text added: "5V"
- board text added: "A1"
- board text added: "A10"
- board text added: "A15"
- board text added: "A2"
- board text added: "A3"
- board text added: "A4"
- board text added: "A5"
- board text added: "A6"
- board text added: "A7"
- board text added: "A8"
- board text added: "A9"
- board text added: "B0"
- board text added: "B1"
- board text added: "B10"
- board text added: "B11"
- board text added: "B12"
- board text added: "B13"
- board text added: "B14"
- board text added: "B15"
- board text added: "B2"
- board text added: "CLK"
- board text added: "DIO"
- board text added: "GND"
- board text added: "PB3"
- board text added: "PB4"
- board text added: "PB5"
- board text added: "USB"
- board text added: "VDDA"
- board text added: "VIN"
- board text added: "~RST"
