File: Main ECU/Main ECU.sch (KiCad schematic (older format))
At the start: 42 parts, among them J1 Screw_Terminal_01x06, J2 Screw_Terminal_01x02, U1 LM317_3PinPackage, U2 UFRGS_PILL, U3 MCP2558FD-xSN, U4 LM358

Commit message: Layout Main ECU and Layout Luz de Freio
Parts:
- added G1: Logo_UFRGS_Large, e-Power:Logo_UFRGS_14.7x8.0mm_SilkS, symbol e-Power:Logo_UFRGS_Large
- added G2: Logo_e-Power_Large, e-Power:Logo_e-Power_16.5x8.0mm_SilkS, symbol e-Power:Logo_e-Power_Large
- added H1, H2, H3, H4: MountingHole_Pad, e-Power:MountingHole_3.2mm_M3_Pad_Via, symbol Mechanical:MountingHole_Pad
- C1, C2: footprint (none) -> e-Power:CP_Elec_10x10
- C3: footprint (none) -> Capacitor_SMD:C_0805_2012Metric
- J1: footprint (none) -> Connector_Phoenix_MSTB:PhoenixContact_MSTBA_2,5_6-G-5,08_1x06_P5.08mm_Horizontal
- J2: footprint (none) -> e-Power:TerminalBlock_Phoenix_MKDS-1,5-2_1x02_P5.08mm_Horizontal_3D
- R1, R10, R11, R12, R13, R14, R15, R16, R17, R18, R19, R2, R20, R21, R3, R4, R5, R6, R7, R8, R9: footprint Resistor_SMD:R_0805_2012Metric_Pad1.15x1.40mm_HandSolder -> Resistor_SMD:R_0805_2012Metric
- TP1, TP2: footprint (none) -> e-Power:TestPoint_Pad_D1.0mm
- U1: footprint (none) -> e-Power:TO-220-3_Horizontal_TabDown
- U4: footprint (none) -> Package_SO:SOIC-8_3.9x4.9mm_P1.27mm
Connections:
- net Out_DC: now also U2.14 (PA15)
- no-connect marks 25 -> 24

Commit message: Layout Fixes and CAN Connector Added
Parts:
- added C21: 100nF, Capacitor_SMD:C_0805_2012Metric, symbol Device:C
- added J4: CAN_2, e-Power:Molex_Mini-Fit_Jr_2x04_P4.20mm_Horizontal, symbol Connector:Screw_Terminal_01x08
- added J5: CAN_1, e-Power:Molex_Mini-Fit_Jr_2x04_P4.20mm_Horizontal, symbol Connector:Screw_Terminal_01x08
- FB1: footprint e-Power:FB_0603_1608Metric -> e-Power:FB_0805_2012Metric
Connections:
- net BUCK-BOOST KiCad/12V is gone; now on net +12V: D1.2 (A)
- net +12V: now also J4.1 (Pin_1), J4.7 (Pin_7), J5.1 (Pin_1), J5.7 (Pin_7)
- net +5V: now also C21.1
- net GND: now also C21.2, J4.2 (Pin_2), J4.5 (Pin_5), J4.8 (Pin_8), J5.2 (Pin_2), J5.5 (Pin_5), J5.8 (Pin_8)
- net CAN_L: now reaches R12.2, U3.6 (CANL)
- net CAN_L: now also J4.3 (Pin_3), J5.3 (Pin_3)
- net CAN_H: now reaches R15.1, U3.7 (CANH)
- net CAN_H: now also J4.4 (Pin_4), J5.4 (Pin_4)
- new net: J4.6 (Pin_6), J5.6 (Pin_6)
- no-connect marks 24 -> 28
Changed lines of the file:
@@
 L power:GND #PWR015
 U 1 1 5F522D07
-P 9475 5400
-F 0 "#PWR015" H 9475 5150 50  0001 C CNN
-F 1 "GND" H 9480 5227 50  0000 C CNN
-F 2 "" H 9475 5400 50  0001 C CNN
-F 3 "" H 9475 5400 50  0001 C CNN
-	1    9475 5400
+P 9475 5275
+F 0 "#PWR015" H 9475 5025 50  0001 C CNN
+F 1 "GND" H 9480 5102 50  0000 C CNN
+F 2 "" H 9475 5275 50  0001 C CNN
+F 3 "" H 9475 5275 50  0001 C CNN
+	1    9475 5275
 	-1   0    0    1
 $EndComp
@@
 F 0 "FB1" V 4901 1025 50  0000 C CNN
 F 1 "Ferrite_Bead_0603" V 4992 1025 50  0000 C CNN
-F 2 "e-Power:FB_0603_1608Metric" V 4925 1200 50  0001 C CNN
+F 2 "e-Power:FB_0805_2012Metric" V 4925 1200 50  0001 C CNN
 F 3 "" H 5175 1025 50  0001 C CNN
 	1    5175 1025
@@
 	1    0    0    -1
 $EndComp
+NoConn ~ 10675 975
+NoConn ~ 10400 975
+NoConn ~ 10100 975
+NoConn ~ 9800 975
+$Comp
+L Device:C C?
+U 1 1 5F59F125
+P 11000 6150
+AR Path="/5F37241F/5F59F125" Ref="C?"  Part="1"
+AR Path="/5F59F125" Ref="C21"  Part="1"
+F 0 "C21" H 11250 6150 50  0000 C CNN
+F 1 "100nF" H 11200 6075 50  0000 C CNN
+F 2 "Capacitor_SMD:C_0805_2012Metric" H 11038 6000 50  0001 C CNN
+F 3 "~" H 11000 6150 50  0001 C CNN
+	1    11000 6150
+	-1   0    0    1
+$EndComp
+$Comp
+L power:GND #PWR0101
+U 1 1 5F5A19EA
+P 11000 6000
+F 0 "#PWR0101" H 11000 5750 50  0001 C CNN
+F 1 "GND" H 11005 5827 50  0000 C CNN
+F 2 "" H 11000 6000 50  0001 C CNN
+F 3 "" H 11000 6000 50  0001 C CNN
+	1    11000 6000
+	-1   0    0    1
+$EndComp
+$Comp
+L power:+5V #PWR0102
+U 1 1 5F5A1DA5
+P 11000 6300
+F 0 "#PWR0102" H 11000 6150 50  0001 C CNN
+F 1 "+5V" H 11015 6473 50  0000 C CNN
+F 2 "" H 11000 6300 50  0001 C CNN
+F 3 "" H 11000 6300 50  0001 C CNN
+	1    11000 6300
+	-1   0    0    1
+$EndComp
+$Comp
+L Connector:Screw_Terminal_01x08 J5
+U 1 1 5F671F01
+P 10450 4300
+F 0 "J5" H 10425 4850 50  0000 L CNN
+F 1 "CAN_1" H 10400 4750 50  0000 L CNN
+F 2 "e-Power:Molex_Mini-Fit_Jr_2x04_P4.20mm_Horizontal" H 10450 4300 50  0001 C CNN
+F 3 "~" H 10450 4300 50  0001 C CNN
+	1    10450 4300
+	1    0    0    -1
+$EndComp
+$Comp
+L Connector:Screw_Terminal_01x08 J4
+U 1 1 5F673072
+P 9250 4300
+F 0 "J4" H 9350 4825 50  0000 C CNN
+F 1 "CAN_2" H 9300 4725 50  0000 C CNN
+F 2 "e-Power:Molex_Mini-Fit_Jr_2x04_P4.20mm_Horizontal" H 9250 4300 50  0001 C CNN
+F 3 "~" H 9250 4300 50  0001 C CNN
+	1    9250 4300
+	-1   0    0    -1
+$EndComp
+Wire Wire Line
+	10250 4600 9450 4600
+Wire Wire Line
+	9450 4500 10250 4500
+Wire Wire Line
+	10250 4400 9450 4400
+Wire Wire Line
+	9450 4300 10250 4300
+Wire Wire Line
+	10250 4200 9450 4200
+Wire Wire Line
+	9450 4100 10250 4100
+Wire Wire Line
+	10250 4000 9500 4000
+$Comp
+L power:GND #PWR053
+U 1 1 5F6A0444
+P 9500 4700
+F 0 "#PWR053" H 9500 4450 50  0001 C CNN
+F 1 "GND" H 9505 4527 50  0000 C CNN
+F 2 "" H 9500 4700 50  0001 C CNN
+F 3 "" H 9500 4700 50  0001 C CNN
+	1    9500 4700
+	1    0    0    -1
+$EndComp
+Wire Wire Line
+	9450 4700 9500 4700
+Connection ~ 9500 4700
+Wire Wire Line
+	9500 4700 10250 4700
+Text Label 9650 4700 0    50   ~ 0
+GND
+Text Label 9650 4100 0    50   ~ 0
+GND
+Text Label 9650 4000 0    50   ~ 0
+VCC
+Text Label 9650 4600 0    50   ~ 0
+VCC
+Text Label 9650 4200 0    50   ~ 0
+CAN_L
+Text Label 9650 4300 0    50   ~ 0
+CAN_H
+Text Label 9650 4400 0    50   ~ 0
+CAN_GND
+$Comp
+L power:+12V #PWR052
+U 1 1 5F6AC105
+P 9500 4000
+F 0 "#PWR052" H 9500 3850 50  0001 C CNN
+F 1 "+12V" H 9500 4175 50  0000 C CNN
+F 2 "" H 9500 4000 50  0001 C CNN
+F 3 "" H 9500 4000 50  0001 C CNN
+	1    9500 4000
+	1    0    0    -1
+$EndComp
+Connection ~ 9500 4000
+Wire Wire Line
+	9500 4000 9450 4000
+Text Label 8850 5375 0    50   ~ 0
+CAN_L
+Text Label 8850 6275 0    50   ~ 0
+CAN_H
+Text Label 9475 5300 0    50   ~ 0
+CAN_GND
+Wire Wire Line
+	9475 5275 9475 5400
+Text Label 3575 1025 0    50   ~ 0
+VCC
 $EndSCHEMATC
