File: SET-RESET/SET-RESET.sch (KiCad schematic (older format))
At the start: 103 parts, among them J1 BMS, J2 BSPD, J3 IMD, J4 IMD_SHTDNW, J5 BMS_SHTDNW, J6 BSPD_SHTDNW, J7 Led's paineis, J8 voltage supply, K1 RELAY_19.1x15.5mm, K2 RELAY_19.1x15.5mm, K3 RELAY_19.1x15.5mm, K4 RELAY_19.1x15.5mm, K5 RELAY_19.1x15.5mm, K6 RELAY_19.1x15.5mm, Q1 BC557, Q10 BC548, Q11 BC548, Q12 BC557, Q13 BC548, Q14 BC548, Q15 BC557, Q16 BC548, Q17 BC548, Q18 BC557, Q2 BC557, Q3 BC557, Q4 Si2302DS, Q5 Si2302DS, Q6 Si2302DS, Q7 BC548, Q8 BC548, Q9 BC548, U1 TLP290-4

Commit message: Rev. B - BSPD and Rev. B - Set/Reset
Parts:
- removed G1: e-Power_12.4x6.0mm_Copper, e-Power:e-Power_16.5x8.0mm_Copper, symbol e-Power:e-Power_12.4x6.0mm_Copper
- removed G2: UFRGS_1_11.0x6.0mm_Copper, e-Power:ESD-Logo_8.9x8mm_Copper, symbol e-Power:UFRGS_1_11.0x6.0mm_Copper
- removed G3: ST Logo, e-Power:ST_6.5x4.1mm_Copper, symbol e-Power:e-Power_12.4x6.0mm_Copper
- removed G4: UFRGS_1_14.7x8.0mm_Copper, e-Power:UFRGS_14.7x8.0mm_Copper, symbol e-Power:UFRGS_1_14.7x8.0mm_Copper
- added G1: Logo_e-Power_Large, e-Power:Logo_e-Power_16.5x8.0mm_SilkS, symbol e-Power:Logo_e-Power_Large
- added G2: Logo_UFRGS_Large, e-Power:Logo_UFRGS_14.7x8.0mm_SilkS, symbol e-Power:Logo_UFRGS_Large
- added G_BMS1: G_BMS, e-Power:TestPoint_Pad_D1.0mm, symbol Connector:TestPoint
- added G_BSPD1: G_BSPD, e-Power:TestPoint_Pad_D1.0mm, symbol Connector:TestPoint
- added G_IMD1: G_IMD, e-Power:TestPoint_Pad_D1.0mm, symbol Connector:TestPoint
- added H1, H2, H3, H4: MountingHole_Pad, e-Power:MountingHole_3.2mm_M3_Pad_Via, symbol Mechanical:MountingHole_Pad
- added R_BMS1: R_BMS, e-Power:TestPoint_Pad_D1.0mm, symbol Connector:TestPoint
- added R_BSPD1: R_BSPD, e-Power:TestPoint_Pad_D1.0mm, symbol Connector:TestPoint
- added R_IMD1: R_IMD, e-Power:TestPoint_Pad_D1.0mm, symbol Connector:TestPoint
- added TP1: GND, e-Power:TestPoint_Pad_D1.0mm, symbol Connector:TestPoint
- added TP2: +12V, e-Power:TestPoint_Pad_D1.0mm, symbol Connector:TestPoint
- C5: value 470uF -> 220uF
- J1, J2, J3, J4, J5, J6, J8, SET/RESET1: footprint Connector_Phoenix_GMSTB:PhoenixContact_GMSTBA_2,5_2-G_1x02_P7.50mm_Horizontal -> e-Power:TerminalBlock_Phoenix_MKDS-1,5-2_1x02_P5.08mm_Horizontal
Connections:
- net +12V: now also TP2.1; no longer D6.2 (A), J8.2 (Pin_2)
- net GND: now also H2.1, H3.1, H4.1, TP1.1
- net ledGREEN_BMS: now also G_BMS1.1
- net ledGREEN_BSPD: now also G_BSPD1.1
- net ledGREEN_IMD: now also G_IMD1.1
- net ledRED_BMS: now also R_BMS1.1
- net ledRED_BSPD: now also R_BSPD1.1
- net ledRED_IMD: now also R_IMD1.1
- new net Input_Power: D6.2 (A), H1.1, J8.2 (Pin_2)
Other:
- moved on the sheet: C1, C2, C3, C4, C5, D6, F1, FB1, J7, J8, R10, R11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

Commit message: Set/Reset Rev. C
Parts:
- removed D1, D2, D3: 1N5819, e-Power:DO-41_SMD, symbol Diode:1N5819
- removed G_BMS1: G_BMS, e-Power:TestPoint_Pad_D1.0mm, symbol Connector:TestPoint
- removed G_BSPD1: G_BSPD, e-Power:TestPoint_Pad_D1.0mm, symbol Connector:TestPoint
- removed G_IMD1: G_IMD, e-Power:TestPoint_Pad_D1.0mm, symbol Connector:TestPoint
- removed Q1, Q12, Q15, Q18, Q2, Q3: BC557, Package_TO_SOT_SMD:SOT-23, symbol Transistor_BJT:BC557
- removed Q10, Q11, Q13, Q14, Q16, Q17, Q7, Q8, Q9: BC548, Package_TO_SOT_SMD:SOT-23, symbol Transistor_BJT:BC548
- removed R40, R41, R42, R43, R44, R45, R46, R47, R48: 1K, Resistor_SMD:R_1206_3216Metric, symbol Device:R
- removed R_BMS1: R_BMS, e-Power:TestPoint_Pad_D1.0mm, symbol Connector:TestPoint
- removed R_BSPD1: R_BSPD, e-Power:TestPoint_Pad_D1.0mm, symbol Connector:TestPoint
- removed R_IMD1: R_IMD, e-Power:TestPoint_Pad_D1.0mm, symbol Connector:TestPoint
- added D1, D2, D3: SS54HF, e-Power:DO-214AC, symbol e-Power:1N5819
- added Q1, Q10, Q11, Q12, Q13, Q14, Q15, Q2, Q3: MMBT5551, Package_TO_SOT_SMD:SOT-23, symbol Transistor_BJT:MMBT3904
- added Q16, Q17, Q18, Q7, Q8, Q9: MMBT5551, Package_TO_SOT_SMD:SOT-23, symbol Transistor_BJT:MMBTA92
- added TP10: +VIN, e-Power:TestPoint_Pad_D1.0mm, symbol Connector:TestPoint
- added TP11: GND, e-Power:TestPoint_Pad_D1.0mm, symbol Connector:TestPoint
- added TP3: ERROR_BMS, e-Power:TestPoint_Pad_D1.0mm, symbol Connector:TestPoint
- added TP4: ERROR_IMD, e-Power:TestPoint_Pad_D1.0mm, symbol Connector:TestPoint
- added TP5: ERROR_BSPD, e-Power:TestPoint_Pad_D1.0mm, symbol Connector:TestPoint
- added TP6: IMD_SHTDNW, e-Power:TestPoint_Pad_D1.0mm, symbol Connector:TestPoint
- added TP7: Led_BSPD, e-Power:TestPoint_Pad_D1.0mm, symbol Connector:TestPoint
- added TP8: Led_IMD, e-Power:TestPoint_Pad_D1.0mm, symbol Connector:TestPoint
- added TP9: Led_BMS, e-Power:TestPoint_Pad_D1.0mm, symbol Connector:TestPoint
- C1, C5: footprint Capacitor_SMD:CP_Elec_4x5.3 -> Capacitor_SMD:CP_Elec_8x10
- C2, C3, C4: footprint Capacitor_SMD:C_0603_1608Metric_Pad1.05x0.95mm_HandSolder -> Capacitor_SMD:C_0805_2012Metric
- D6: value 1N5819 -> SS54HF; footprint e-Power:DO-41_SMD -> e-Power:DO-214AC
- FB1: footprint e-Power:FB_0603_1608Metric -> e-Power:FB_0805_2012Metric
- R1, R10, R11, R12, R13, R14, R15, R16, R17, R18, R19, R2, R20, R21, R22, R23, R24, R25, R26, R27, R28, R29, R3, R30, R31, R32, R33, R34, R35, R36, R37, R38, R39, R4, R5, R6, R7, R8, R9: footprint Resistor_SMD:R_1206_3216Metric -> Resistor_SMD:R_0805_2012Metric
- U1: footprint e-Power:TLP290-4 -> e-Power:SOIC-16_4.55x10.3mm_P1.27mm(TLP290-4)
- renumbered D10 to RED3
Connections:
- net ledRED_BMS is gone; now on net led_BMS: J7.2 (Pin_2)
- net ledRED_BSPD is gone; now on net led_BSPD: J7.3 (Pin_3)
- net ledRED_IMD is gone; now on net led_IMD: J7.1 (Pin_1)
- net +12V: now also D1.1 (K), D2.1 (K), D3.1 (K), Q16.2 (E), Q17.2 (E), Q18.2 (E), Q7.2 (E), Q8.2 (E), Q9.2 (E)
- net GND: now also Q1.2 (E), Q10.2 (E), Q11.2 (E), Q12.2 (E), Q13.2 (E), Q14.2 (E), Q15.2 (E), Q2.2 (E), Q3.2 (E), TP11.1
- net Input_Power: now also TP10.1
- net at R1.1: now also Q7.1 (B)
- net at R1.2, R16.2: now also Q3.3 (C)
- net at K1.1, U1.16: now also Q7.3 (C)
- net at R17.2, R2.2: now also Q1.3 (C)
- net at R13.1: now also Q1.1 (B), TP3.1
- net at R2.1: now also Q8.1 (B)
- net at K2.1, U1.14: now also Q8.3 (C)
- net at R3.1: now also Q9.1 (B)
- net at R18.2, R3.2: now also Q2.3 (C)
- net at K3.1, U1.12: now also Q9.3 (C)
- net at R15.1: now also Q3.1 (B), TP4.1
- net at R19.1: now also Q11.1 (B)
- net at K1.5, K4.5, Q4.3 (D)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: now also D1.2 (A)
- net at R14.1: now also Q2.1 (B), TP5.1
- net at R22.2, R23.2: now also Q14.3 (C)
- net at R21.2: now also Q14.1 (B)
- net at R23.1: now also Q17.1 (B)
- net led_IMD: now reaches R24.1
- net led_IMD: now also Q17.3 (C), TP8.1
- net at R26.1: now also Q12.1 (B)
- net at K2.5, K5.5, Q5.3 (D)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: now also D2.2 (A)
- net at R29.2, R30.1: now also Q15.3 (C)
- net at R30.2: now also Q18.1 (B)
- net led_BMS: now reaches R31.1
- net led_BMS: now also Q18.3 (C), TP9.1
- net at R28.1: now also Q15.1 (B)
- net at R33.1: now also Q10.1 (B)
- net at K3.5, K6.5, Q6.3 (D)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: now also D3.2 (A)
- net at R36.2, R37.1: now also Q13.3 (C)
- net at R37.2: now also Q16.1 (B)
- net led_BSPD: now reaches R38.1
- net led_BSPD: now also Q16.3 (C), TP7.1
- net at R35.2: now also Q13.1 (B)
- net ledGREEN_BMS: no longer names the net of D5.2 (A), R27.2
- net ledGREEN_BMS: now also Q12.3 (C); no longer J7.5 (Pin_5)
- net ledGREEN_BSPD: no longer names the net of D4.2 (A), R34.2
- net ledGREEN_BSPD: now also Q10.3 (C); no longer J7.6 (Pin_6)
- net ledGREEN_IMD: no longer names the net of D8.2 (A), R20.2
- net ledGREEN_IMD: now also Q11.3 (C); no longer J7.4 (Pin_4)
Other:
- moved on the sheet: F1, TP1

Commit message: att set/reset and ail 07/09/2020
Parts:
- removed J7: Led's paineis, Connector_PinHeader_1.27mm:PinHeader_1x08_P1.27mm_Vertical, symbol Connector:Screw_Terminal_01x08
- removed TP6: IMD_SHTDNW, e-Power:TestPoint_Pad_D1.0mm, symbol Connector:TestPoint
- added J10, J11, J7, J9: Painel, e-Power:TerminalBlock_Phoenix_MKDS-1,5-2_1x02_P5.08mm_Horizontal, symbol Connector:Screw_Terminal_01x02
- added Q19, Q20, Q21: MMBT5551, Package_TO_SOT_SMD:SOT-23, symbol Transistor_BJT:MMBT3904
- added R40, R41, R42: 1K, Resistor_SMD:R_0805_2012Metric, symbol Device:R
- renumbered H3 to GND1, H2 to NC1, H4 to NC2, H1 to Vin+1
Connections:
- net +12V: now also R40.1, R41.1, R42.1
- net GND: now also J11.1 (Pin_1), Q19.2 (E), Q20.2 (E), Q21.2 (E); no longer NC1.1, NC2.1
- net led_BMS: now also J7.2 (Pin_2), Q20.1 (B)
- net led_BSPD: now also J9.1 (Pin_1), Q19.1 (B)
- net led_IMD: now also J7.1 (Pin_1), Q21.1 (B)
- new net: J9.2 (Pin_2), Q19.3 (C), R40.2
- new net: J10.1 (Pin_1), Q20.3 (C), R41.2
- new net: J10.2 (Pin_2), Q21.3 (C), R42.2
- no-connect marks 7 -> 9
Other:
- moved on the sheet: C1, C2, C3, C4, C5, D6, F1, FB1, GND1, J8, NC1, NC2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
