File: Shutdown/AIL.sch (KiCad schematic (older format))
At the start: 36 parts

Commit message: update shutdown
Parts:
- F? (x2): symbol e-Power:Fuse_1206 -> Shutdown-rescue:Fuse_1206-e-Power
- G?: symbol e-Power:Logo_UFRGS_Large -> Shutdown-rescue:Logo_UFRGS_Large-e-Power
- G?: symbol e-Power:Logo_e-Power_Large -> Shutdown-rescue:Logo_e-Power_Large-e-Power
Connections:
- net TS+ renamed HV_+
Changed lines of the file:
@@
 EESchema Schematic File Version 4
-LIBS:Shutdown-cache
 EELAYER 30 0
 EELAYER END
 $Descr A4 11693 8268
 encoding utf-8
-Sheet 1 43
+Sheet 4 43
 Title "AIL"
 Date "2020-17-07"
@@
 Connection ~ 6900 5400
 $Comp
-L e-Power:Fuse_1206 F?
+L Shutdown-rescue:Fuse_1206-e-Power F?
 U 1 1 5F14FB8F
 P 4050 2050
@@
 $EndComp
 $Comp
-L e-Power:Fuse_1206 F?
+L Shutdown-rescue:Fuse_1206-e-Power F?
 U 1 1 5F150096
 P 4050 2150
@@
 NoConn ~ 8600 5000
 $Comp
-L e-Power:Logo_UFRGS_Large G?
+L Shutdown-rescue:Logo_UFRGS_Large-e-Power G?
 U 1 1 5F5590C7
 P 7900 2700
@@
 $EndComp
 $Comp
-L e-Power:Logo_e-Power_Large G?
+L Shutdown-rescue:Logo_e-Power_Large-e-Power G?
 U 1 1 5F559F30
 P 7900 2300
@@
 	1    0    0    -1
 $EndComp
+Text HLabel 4275 2050 1    50   Input ~ 0
+HV_+
+Text HLabel 4275 2150 3    50   Input ~ 0
+HV_-
 $EndSCHEMATC
