File: Shutdown/BMS_24S.sch (KiCad schematic (older format))
At the start: 186 parts

Commit message: update shutdown
Parts:
- G? (x2): symbol e-Power:Logo_UFRGS_Large -> Shutdown-rescue:Logo_UFRGS_Large-e-Power
- G?: symbol e-Power:Logo_e-Power_Large -> Shutdown-rescue:Logo_e-Power_Large-e-Power
Changed lines of the file:
@@
 EESchema Schematic File Version 4
-LIBS:Shutdown-cache
 EELAYER 30 0
 EELAYER END
 $Descr A3 16535 11693
 encoding utf-8
-Sheet 12 43
+Sheet 11 43
 Title ""
 Date ""
@@
 	15000 6300 15350 6300
 $Comp
-L e-Power:Logo_UFRGS_Large G?
+L Shutdown-rescue:Logo_UFRGS_Large-e-Power G?
 U 1 1 62BF7C1B
 P 10900 10100
@@
 $EndComp
 $Comp
-L e-Power:Logo_e-Power_Large G?
+L Shutdown-rescue:Logo_e-Power_Large-e-Power G?
 U 1 1 62BF88DC
 P 10900 9650
@@
 $EndComp
 $Comp
-L e-Power:Logo_UFRGS_Large G?
+L Shutdown-rescue:Logo_UFRGS_Large-e-Power G?
 U 1 1 6038A412
 P 10900 10650
@@
 Wire Bus Line
 	3900 1200 3900 1900
+Text HLabel 15400 6100 1    50   Input ~ 0
+CAN_L
+Text HLabel 15375 6500 3    50   Input ~ 0
+CAN_H
 $EndSCHEMATC
