File: Shutdown/BSPD.sch (KiCad schematic (older format))
At the start: 103 parts

Commit message: update shutdown
Parts:
- D? (x2): symbol e-Power:LED -> Shutdown-rescue:LED-e-Power
- D? (x2): symbol e-Power:1N5819 -> Shutdown-rescue:1N5819-e-Power
- G?: symbol e-Power:Logo_UFRGS_Large -> Shutdown-rescue:Logo_UFRGS_Large-e-Power
- G?: symbol e-Power:Logo_e-Power_Large -> Shutdown-rescue:Logo_e-Power_Large-e-Power
Changed lines of the file:
@@
 EESchema Schematic File Version 4
-LIBS:Shutdown-cache
 EELAYER 30 0
 EELAYER END
@@
 	7100 4350 7250 4350
 $Comp
-L e-Power:LED D?
+L Shutdown-rescue:LED-e-Power D?
 U 1 1 5EF511BA
 P 6700 4900
@@
 Input_Power
 $Comp
-L e-Power:LED D?
+L Shutdown-rescue:LED-e-Power D?
 U 1 1 5F337AD6
 P 9300 4900
@@
 $EndComp
 $Comp
-L e-Power:1N5819 D?
+L Shutdown-rescue:1N5819-e-Power D?
 U 1 1 5F358A00
 P 4750 6700
+AR Path="/5F358A00" Ref="D?"  Part="1"
+AR Path="/5F7F3E0E/5F358A00" Ref="D?"  Part="1"
 F 0 "D?" H 4750 6484 50  0000 C CNN
 F 1 "1N5819" H 4750 6575 50  0000 C CNN
@@
 	4900 4150 4950 4150
 $Comp
-L e-Power:1N5819 D?
+L Shutdown-rescue:1N5819-e-Power D?
 U 1 1 5F368B0A
 P 5100 4150
+AR Path="/5F368B0A" Ref="D?"  Part="1"
+AR Path="/5F7F3E0E/5F368B0A" Ref="D?"  Part="1"
 F 0 "D?" H 5100 4400 50  0000 C CNN
 F 1 "1N5819" H 5100 4300 50  0000 C CNN
@@
 Connection ~ 3450 4900
 $Comp
-L e-Power:Logo_UFRGS_Large G?
+L Shutdown-rescue:Logo_UFRGS_Large-e-Power G?
 U 1 1 5F60255C
 P 10600 850
@@
 $EndComp
 $Comp
-L e-Power:Logo_e-Power_Large G?
+L Shutdown-rescue:Logo_e-Power_Large-e-Power G?
 U 1 1 5F602D9E
 P 10600 1350
@@
 	4100 7050 4300 7050
 Connection ~ 4100 7050
+Text HLabel 7175 4350 1    50   Input ~ 0
+Out_BSPD
 $EndSCHEMATC
