File: Shutdown/BUCK-BOOST KiCad.sch (KiCad schematic (older format))
At the start: 96 parts

Commit message: update shutdown
Parts:
- D? (x3): symbol e-Power:D_SCH_SS54HF -> Shutdown-rescue:D_SCH_SS54HF-e-Power
- D? (x2): symbol e-Power:LED -> Shutdown-rescue:LED-e-Power
- FB?: symbol e-Power:Ferrite_Bead_0603 -> Shutdown-rescue:Ferrite_Bead_0603-e-Power
- L? (x5): symbol e-Power:INDUCTOR_PWR -> Shutdown-rescue:INDUCTOR_PWR-e-Power
- U?: symbol e-Power:LM2577S-ADJ -> Shutdown-rescue:LM2577S-ADJ-e-Power
Changed lines of the file:
@@
 EESchema Schematic File Version 4
-LIBS:Shutdown-cache
 EELAYER 30 0
 EELAYER END
 $Descr A4 11693 8268
 encoding utf-8
-Sheet 2 43
+Sheet 7 43
 Title "BUCK-BOOST 12V"
 Date "2020-05-10"
@@
 $EndComp
 $Comp
-L e-Power:D_SCH_SS54HF D?
+L Shutdown-rescue:D_SCH_SS54HF-e-Power D?
 U 1 1 5EB8B647
 P 3550 1675
@@
 	4500 1675 4850 1675
 $Comp
-L e-Power:D_SCH_SS54HF D?
+L Shutdown-rescue:D_SCH_SS54HF-e-Power D?
 U 1 1 5EB9411D
 P 6000 2125
@@
 	6000 2275 6000 2375
 $Comp
-L e-Power:INDUCTOR_PWR L?
+L Shutdown-rescue:INDUCTOR_PWR-e-Power L?
 U 1 1 5EB9596B
 P 6350 1875
@@
 $EndComp
 $Comp
-L e-Power:INDUCTOR_PWR L?
+L Shutdown-rescue:INDUCTOR_PWR-e-Power L?
 U 1 1 5EBB83D9
 P 1425 3875
@@
 	1725 3875 1675 3875
 $Comp
-L e-Power:D_SCH_SS54HF D?
+L Shutdown-rescue:D_SCH_SS54HF-e-Power D?
 U 1 1 5EBBB940
 P 1975 3875
@@
 $EndComp
 $Comp
-L e-Power:LM2577S-ADJ U?
+L Shutdown-rescue:LM2577S-ADJ-e-Power U?
 U 1 1 5EBB381F
 P 1425 4375
@@
 	8025 2625 8025 2575
 $Comp
-L e-Power:LED D?
+L Shutdown-rescue:LED-e-Power D?
 U 1 1 5EE0B68D
 P 8025 2425
@@
 	4000 4625 4000 4575
 $Comp
-L e-Power:LED D?
+L Shutdown-rescue:LED-e-Power D?
 U 1 1 5EE26E5D
 P 4000 4425
@@
 Connection ~ 4000 3875
 $Comp
-L e-Power:INDUCTOR_PWR L?
+L Shutdown-rescue:INDUCTOR_PWR-e-Power L?
 U 1 1 5F3769B1
 P 7250 1875
@@
 $EndComp
 $Comp
-L e-Power:Ferrite_Bead_0603 FB?
+L Shutdown-rescue:Ferrite_Bead_0603-e-Power FB?
 U 1 1 5F388AA4
 P 3200 1675
@@
 Input_Voltage_Cells
 $Comp
-L e-Power:INDUCTOR_PWR L?
+L Shutdown-rescue:INDUCTOR_PWR-e-Power L?
 U 1 1 5F3C9968
 P 3450 3875
@@
 $EndComp
 $Comp
-L e-Power:INDUCTOR_PWR L?
+L Shutdown-rescue:INDUCTOR_PWR-e-Power L?
 U 1 1 5F3EAA4E
 P 4100 1675
