File: Shutdown/Diferencial.sch (KiCad schematic (older format))
At the start: 113 parts

Commit message: update shutdown
Parts:
- D?: symbol e-Power:LED -> Shutdown-rescue:LED-e-Power
- D?: symbol e-Power:D_SCH_SS54HF -> Shutdown-rescue:D_SCH_SS54HF-e-Power
- D?: symbol e-Power:SS54HF -> Shutdown-rescue:SS54HF-e-Power
- G?: symbol e-Power:Logo_UFRGS_Large -> Shutdown-rescue:Logo_UFRGS_Large-e-Power
- G?: symbol e-Power:Logo_e-Power_Large -> Shutdown-rescue:Logo_e-Power_Large-e-Power
- K?: symbol e-Power:RELAY_19.1x15.5mm -> Shutdown-rescue:RELAY_19.1x15.5mm-e-Power
- U?: symbol e-Power:UFRGS_PILL -> Shutdown-rescue:UFRGS_PILL-e-Power
Connections:
- net In_ACCS_1: now reaches J?.3 (Pin_3), R?.1, R?.1, R?.2
- net In_ACCS_2: now reaches J?.3 (Pin_3), R?.1, R?.1, R?.2
- net Buzzer_Out: now reaches J?.1 (Pin_1), K?.1, R?.2
- net In_Brake_Sensor_1: now reaches J?.3 (Pin_3), R?.1, R?.1, R?.2
- net Out_Brake_Light: now reaches J?.1 (Pin_1), Q?.3 (C)
- net In_Brake_Pedal_2: now reaches J?.3 (Pin_3), R?.1, R?.1, R?.2
Changed lines of the file:
@@
 EESchema Schematic File Version 4
-LIBS:Shutdown-cache
 EELAYER 30 0
 EELAYER END
 $Descr A3 16535 11693
 encoding utf-8
-Sheet 43 43
+Sheet 42 43
 Title "Diferencial Board"
 Date "2020-08-06"
@@
 $EndComp
 $Comp
-L e-Power:UFRGS_PILL U?
+L Shutdown-rescue:UFRGS_PILL-e-Power U?
 U 1 1 5ECDC53F
 P 11250 4125
@@
 Connection ~ 6575 4775
 $Comp
-L e-Power:LED D?
+L Shutdown-rescue:LED-e-Power D?
 U 1 1 5F15AABA
 P 8925 9750
@@
 $EndComp
 $Comp
-L e-Power:RELAY_19.1x15.5mm K?
+L Shutdown-rescue:RELAY_19.1x15.5mm-e-Power K?
 U 1 1 5F1FE295
 P 8725 8800
@@
 $EndComp
 $Comp
-L e-Power:D_SCH_SS54HF D?
+L Shutdown-rescue:D_SCH_SS54HF-e-Power D?
 U 1 1 5F36ACFB
 P 7850 8800
@@
 $EndComp
 $Comp
-L e-Power:Logo_UFRGS_Large G?
+L Shutdown-rescue:Logo_UFRGS_Large-e-Power G?
 U 1 1 5F37D1F5
 P 15650 875
@@
 $EndComp
 $Comp
-L e-Power:Logo_e-Power_Large G?
+L Shutdown-rescue:Logo_e-Power_Large-e-Power G?
 U 1 1 5F37FB8E
 P 15650 1375
@@
 $EndComp
 $Comp
-L e-Power:SS54HF D?
+L Shutdown-rescue:SS54HF-e-Power D?
 U 1 1 5F4E4A0E
 P 11825 8525
@@
 	1    0    0    -1
 $EndComp
+Text HLabel 1150 1400 3    50   Input ~ 0
+In_ACCS_1
+Text HLabel 1500 2800 1    50   Input ~ 0
+In_ACCS_2
+Text HLabel 1400 4525 3    50   Input ~ 0
+In_Brake_Sensor_1
+Text HLabel 1475 6025 3    50   Input ~ 0
+In_Brake_Pedal_2
+Text HLabel 14525 6950 2    50   Input ~ 0
+Out_Brake_Light
+Text HLabel 9150 9225 1    50   Input ~ 0
+Buzzer_Out
+Text HLabel 2300 9775 2    50   Input ~ 0
+CAN_H
+Text HLabel 2300 9875 2    50   Input ~ 0
+CAN_L
 $EndSCHEMATC
