File: Shutdown/LM235_1_2_3_4.sch (KiCad schematic (older format))
At the start: 6 parts, among them U2001 LM324

Commit message: update shutdown
Parts:
- U2001: symbol e-Power:LM324 -> Shutdown-rescue:LM324-e-Power
Changed lines of the file:
@@
 EESchema Schematic File Version 4
-LIBS:Shutdown-cache
 EELAYER 30 0
 EELAYER END
@@
 $EndDescr
 $Comp
-L e-Power:LM324 U?
+L Shutdown-rescue:LM324-e-Power U?
 U 5 1 5EA4C987
 P 1400 3100
@@
 TS_1
 $Comp
-L e-Power:LM324 U?
+L Shutdown-rescue:LM324-e-Power U?
 U 1 1 5EC12A89
 P 1950 1250
@@
 	1800 3400 1800 3500
 $Comp
-L e-Power:LM324 U?
+L Shutdown-rescue:LM324-e-Power U?
 U 2 1 5EA4A09D
 P 1950 1950
@@
 TS_3
 $Comp
-L e-Power:LM324 U?
+L Shutdown-rescue:LM324-e-Power U?
 U 3 1 5F5E9E0E
 P 3850 1250
@@
 T3
 $Comp
-L e-Power:LM324 U?
+L Shutdown-rescue:LM324-e-Power U?
 U 4 1 5F5E9E1B
 P 3850 1950
