File: Shutdown/Luz de Freio.sch (KiCad schematic (older format))
At the start: 62 parts

Commit message: update shutdown
Parts:
- D? (x2): symbol e-Power:SS54HF -> Shutdown-rescue:SS54HF-e-Power
- G?: symbol e-Power:Logo_e-Power_Large -> Shutdown-rescue:Logo_e-Power_Large-e-Power
- G?: symbol e-Power:Logo_UFRGS_Large -> Shutdown-rescue:Logo_UFRGS_Large-e-Power
- K?: symbol e-Power:RELAY_19.1x15.5mm -> Shutdown-rescue:RELAY_19.1x15.5mm-e-Power
- L?: symbol e-Power:INDUCTOR_PWR -> Shutdown-rescue:INDUCTOR_PWR-e-Power
- Q?: symbol e-Power:Si2302DS -> Shutdown-rescue:Si2302DS-e-Power
Connections:
- net In_Brake_ON_OFF: now reaches J?.2 (Pin_2), R?.2, R?.2
Changed lines of the file:
@@
 EESchema Schematic File Version 4
-LIBS:Shutdown-cache
 EELAYER 30 0
 EELAYER END
 $Descr A4 11693 8268
 encoding utf-8
-Sheet 1 43
+Sheet 10 43
 Title "Luz de Freio"
 Date ""
@@
 $EndComp
 $Comp
-L e-Power:RELAY_19.1x15.5mm K?
+L Shutdown-rescue:RELAY_19.1x15.5mm-e-Power K?
 U 1 1 5F0862CF
 P 5500 1450
@@
 $EndComp
 $Comp
-L e-Power:INDUCTOR_PWR L?
+L Shutdown-rescue:INDUCTOR_PWR-e-Power L?
 U 1 1 5F081938
 P 2700 6050
@@
 	2875 6900 3700 6900
 $Comp
-L e-Power:Logo_e-Power_Large G?
+L Shutdown-rescue:Logo_e-Power_Large-e-Power G?
 U 1 1 5F3E273D
 P 975 800
@@
 $EndComp
 $Comp
-L e-Power:Logo_UFRGS_Large G?
+L Shutdown-rescue:Logo_UFRGS_Large-e-Power G?
 U 1 1 5F3E3C29
 P 1875 775
@@
 $EndComp
 $Comp
-L e-Power:Si2302DS Q?
+L Shutdown-rescue:Si2302DS-e-Power Q?
 U 1 1 5F4C2749
 P 4750 2050
@@
 	7800 2225 7800 2700
 $Comp
-L e-Power:SS54HF D?
+L Shutdown-rescue:SS54HF-e-Power D?
 U 1 1 5F5C0FB4
 P 4850 1450
@@
 Connection ~ 10925 6300
 $Comp
-L e-Power:SS54HF D?
+L Shutdown-rescue:SS54HF-e-Power D?
 U 1 1 5F5E50A2
 P 6325 5750
@@
 Wire Wire Line
 	7975 4300 7975 4350
+Text HLabel 3100 2050 3    50   Input ~ 0
+In_Brake_ON_OFF
 $EndSCHEMATC
