File: Shutdown/TSAL.sch (KiCad schematic (older format))
At the start: 123 parts

Commit message: update shutdown
Parts:
- D? (x3): symbol e-Power:D_SCH_1N5819 -> Shutdown-rescue:D_SCH_1N5819-e-Power
- G?: symbol e-Power:Logo_High_Voltage_Large -> Shutdown-rescue:Logo_High_Voltage_Large-e-Power
- G?: symbol e-Power:Logo_UFRGS_Large -> Shutdown-rescue:Logo_UFRGS_Large-e-Power
- G?: symbol e-Power:Logo_e-Power_Large -> Shutdown-rescue:Logo_e-Power_Large-e-Power
- K?: symbol e-Power:RELAY_19.1x15.5mm -> Shutdown-rescue:RELAY_19.1x15.5mm-e-Power
- L?: symbol e-Power:INDUCTOR_PWR -> Shutdown-rescue:INDUCTOR_PWR-e-Power
- Q?: symbol e-Power:Si2302DS -> Shutdown-rescue:Si2302DS-e-Power
Changed lines of the file:
@@
 EESchema Schematic File Version 4
-LIBS:Shutdown-cache
 EELAYER 30 0
 EELAYER END
@@
 $EndComp
 $Comp
-L e-Power:INDUCTOR_PWR L?
+L Shutdown-rescue:INDUCTOR_PWR-e-Power L?
 U 1 1 5F085F28
 P 2650 4050
@@
 $EndComp
 $Comp
-L e-Power:D_SCH_1N5819 D?
+L Shutdown-rescue:D_SCH_1N5819-e-Power D?
 U 1 1 5F0B5787
 P 1850 6300
@@
 Input_Power
 $Comp
-L e-Power:RELAY_19.1x15.5mm K?
+L Shutdown-rescue:RELAY_19.1x15.5mm-e-Power K?
 U 1 1 5F11030F
 P 4650 1350
@@
 $EndComp
 $Comp
-L e-Power:D_SCH_1N5819 D?
+L Shutdown-rescue:D_SCH_1N5819-e-Power D?
 U 1 1 5F486FD6
 P 3250 4050
@@
 $EndComp
 $Comp
-L e-Power:D_SCH_1N5819 D?
+L Shutdown-rescue:D_SCH_1N5819-e-Power D?
 U 1 1 5F487A9C
 P 4150 1350
@@
 	4550 1800 4550 4100
 $Comp
-L e-Power:Si2302DS Q?
+L Shutdown-rescue:Si2302DS-e-Power Q?
 U 1 1 60C7FE8D
 P 4050 1950
@@
 $EndComp
 $Comp
-L e-Power:Logo_High_Voltage_Large G?
+L Shutdown-rescue:Logo_High_Voltage_Large-e-Power G?
 U 1 1 5F45B899
 P 1500 3000
@@
 $EndComp
 $Comp
-L e-Power:Logo_UFRGS_Large G?
+L Shutdown-rescue:Logo_UFRGS_Large-e-Power G?
 U 1 1 5F9561DD
 P 2400 3000
@@
 $EndComp
 $Comp
-L e-Power:Logo_e-Power_Large G?
+L Shutdown-rescue:Logo_e-Power_Large-e-Power G?
 U 1 1 5F95A5B2
 P 3250 3050
@@
 Text HLabel 1050 1150 3    50   Input ~ 0
 HV-
+Text HLabel 1300 7050 1    50   Input ~ 0
+Input_Power
 $EndSCHEMATC
