File: Shutdown/balancing_01.sch (KiCad schematic (older format))
At the start: 65 parts, among them Q2501 Si2302DS, Q2502 Si2302DS, Q2503 Si2302DS, Q2504 Si2302DS, U2501 TLP290-4

Commit message: update shutdown
Parts:
- D2501, D2502, D2503, D2504: symbol e-Power:LED -> Shutdown-rescue:LED-e-Power
- Q2501, Q2502, Q2503, Q2504: symbol e-Power:Si2302DS -> Shutdown-rescue:Si2302DS-e-Power
Changed lines of the file:
@@
 EESchema Schematic File Version 4
-LIBS:Shutdown-cache
 EELAYER 30 0
 EELAYER END
@@
 	3100 600  3200 600
 $Comp
-L e-Power:LED D2503
+L Shutdown-rescue:LED-e-Power D2503
 U 1 1 5EEF5CEC
 P 6150 3100
@@
 Connection ~ 5900 2950
 $Comp
-L e-Power:LED D2504
+L Shutdown-rescue:LED-e-Power D2504
 U 1 1 5EEF5CEE
 P 6150 4100
@@
 Connection ~ 5900 3950
 $Comp
-L e-Power:LED D2502
+L Shutdown-rescue:LED-e-Power D2502
 U 1 1 5F454CCC
 P 6150 2100
@@
 Connection ~ 5900 1950
 $Comp
-L e-Power:LED D2501
+L Shutdown-rescue:LED-e-Power D2501
 U 1 1 5F46A117
 P 6150 1100
@@
 	4500 3950 4300 3950
 $Comp
-L e-Power:Si2302DS Q2501
+L Shutdown-rescue:Si2302DS-e-Power Q2501
 U 1 1 5F341634
 P 5000 1200
@@
 $EndComp
 $Comp
-L e-Power:Si2302DS Q2502
+L Shutdown-rescue:Si2302DS-e-Power Q2502
 U 1 1 5F34235C
 P 5000 2200
@@
 $EndComp
 $Comp
-L e-Power:Si2302DS Q2503
+L Shutdown-rescue:Si2302DS-e-Power Q2503
 U 1 1 5F3428FA
 P 5000 3200
@@
 $EndComp
 $Comp
-L e-Power:Si2302DS Q2504
+L Shutdown-rescue:Si2302DS-e-Power Q2504
 U 1 1 5F3433A2
 P 5000 4200
