File: Shutdown/current_sensor.sch (KiCad schematic (older format))
At the start: 10 parts, among them U3101 LM324

Commit message: update shutdown
Parts:
- U3101: symbol e-Power:LM324 -> Shutdown-rescue:LM324-e-Power
Changed lines of the file:
@@
 EESchema Schematic File Version 4
-LIBS:Shutdown-cache
 EELAYER 30 0
 EELAYER END
@@
 VIOUT
 $Comp
-L e-Power:LM324 U?
+L Shutdown-rescue:LM324-e-Power U?
 U 1 1 5F36FFAB
 P 4800 1900
@@
 AR Path="/5EC24961/5EC85226/5F36FFAB" Ref="U?"  Part="1"
 AR Path="/5F3561B0/5F36FFAB" Ref="U3101"  Part="1"
+AR Path="/5F805AC0/5F3561B0/5F36FFAB" Ref="U?"  Part="1"
 F 0 "U?" H 4900 1750 50  0000 C CNN
 F 1 "LM324" H 4800 1900 50  0000 C CNN
@@
 	4450 2000 4450 2150
 $Comp
-L e-Power:LM324 U?
+L Shutdown-rescue:LM324-e-Power U?
 U 5 1 5F3748A9
 P 4850 3450
@@
 AR Path="/5EC24961/5EC85226/5F3748A9" Ref="U?"  Part="1"
 AR Path="/5F3561B0/5F3748A9" Ref="U3101"  Part="5"
+AR Path="/5F805AC0/5F3561B0/5F3748A9" Ref="U?"  Part="5"
 F 0 "U?" V 4950 3450 50  0000 C CNN
 F 1 "LM324" V 4850 3450 50  0000 C CNN
@@
 AR Path="/5EC24961/5EC85226/5F37D4F6" Ref="C?"  Part="1"
 AR Path="/5F3561B0/5F37D4F6" Ref="C3101"  Part="1"
+AR Path="/5F805AC0/5F3561B0/5F37D4F6" Ref="C?"  Part="1"
 F 0 "C?" H 5565 3646 50  0000 L CNN
 F 1 "100nF" H 5565 3555 50  0000 L CNN
@@
 Connection ~ 5250 3350
 $Comp
-L e-Power:LM324 U?
+L Shutdown-rescue:LM324-e-Power U?
 U 2 1 5F186021
 P 4800 2450
@@
 AR Path="/5EC24961/5EC85226/5F186021" Ref="U?"  Part="1"
 AR Path="/5F3561B0/5F186021" Ref="U3101"  Part="2"
+AR Path="/5F805AC0/5F3561B0/5F186021" Ref="U?"  Part="2"
 F 0 "U?" H 4900 2300 50  0000 C CNN
 F 1 "LM324" H 4800 2450 50  0000 C CNN
@@
 	3200 2600 3700 2600
 $Comp
-L e-Power:LM324 U?
+L Shutdown-rescue:LM324-e-Power U?
 U 3 1 5F1961F4
 P 6700 2000
@@
 AR Path="/5EC24961/5EC85226/5F1961F4" Ref="U?"  Part="1"
 AR Path="/5F3561B0/5F1961F4" Ref="U3101"  Part="3"
+AR Path="/5F805AC0/5F3561B0/5F1961F4" Ref="U?"  Part="3"
 F 0 "U?" H 6800 1850 50  0000 C CNN
 F 1 "LM324" H 6700 2000 50  0000 C CNN
@@
 AR Path="/5EC24961/5EC85226/5F19D869" Ref="R?"  Part="1"
 AR Path="/5F3561B0/5F19D869" Ref="R3103"  Part="1"
+AR Path="/5F805AC0/5F3561B0/5F19D869" Ref="R?"  Part="1"
 F 0 "R?" V 6050 1900 50  0000 C CNN
 F 1 "10K" V 6150 1900 50  0000 C CNN
@@
 AR Path="/5EC24961/5EC85226/5F19E141" Ref="R?"  Part="1"
 AR Path="/5F3561B0/5F19E141" Ref="R3104"  Part="1"
+AR Path="/5F805AC0/5F3561B0/5F19E141" Ref="R?"  Part="1"
 F 0 "R?" V 6250 2100 50  0000 C CNN
 F 1 "10K" V 6150 2100 50  0000 C CNN
@@
 AR Path="/5EC24961/5EC85226/5F19E3C2" Ref="R?"  Part="1"
 AR Path="/5F3561B0/5F19E3C2" Ref="R3105"  Part="1"
+AR Path="/5F805AC0/5F3561B0/5F19E3C2" Ref="R?"  Part="1"
 F 0 "R?" H 6150 2400 50  0000 C CNN
 F 1 "10K" V 6350 2350 50  0000 C CNN
@@
 AR Path="/5EC24961/5EC85226/5F19EB05" Ref="R?"  Part="1"
 AR Path="/5F3561B0/5F19EB05" Ref="R3102"  Part="1"
+AR Path="/5F805AC0/5F3561B0/5F19EB05" Ref="R?"  Part="1"
 F 0 "R?" V 6800 1650 50  0000 C CNN
 F 1 "10K" V 6700 1650 50  0000 C CNN
@@
 AR Path="/5EC24961/5EC85226/629BD18A" Ref="R?"  Part="1"
 AR Path="/5F3561B0/629BD18A" Ref="R3101"  Part="1"
+AR Path="/5F805AC0/5F3561B0/629BD18A" Ref="R?"  Part="1"
 F 0 "R?" V 4350 1600 50  0000 C CNN
 F 1 "0R" V 4450 1600 50  0000 C CNN
@@
 $EndComp
 $Comp
-L e-Power:LM324 U?
+L Shutdown-rescue:LM324-e-Power U?
 U 4 1 5F58B9DC
 P 6700 3200
@@
 AR Path="/5EC24961/5EC85226/5F58B9DC" Ref="U?"  Part="1"
 AR Path="/5F3561B0/5F58B9DC" Ref="U3101"  Part="4"
+AR Path="/5F805AC0/5F3561B0/5F58B9DC" Ref="U?"  Part="4"
 F 0 "U?" H 6800 3050 50  0000 C CNN
 F 1 "LM324" H 6700 3200 50  0000 C CNN
