File: Shutdown/voltage_references.sch (KiCad schematic (older format))
At the start: 55 parts

Commit message: update shutdown
Parts:
- U? (x5): symbol e-Power:LM324 -> Shutdown-rescue:LM324-e-Power
- U? (x2): symbol e-Power:TL431 -> Shutdown-rescue:TL431-e-Power
Changed lines of the file:
@@
 EESchema Schematic File Version 4
-LIBS:Shutdown-cache
 EELAYER 30 0
 EELAYER END
@@
 1.8V
 $Comp
-L e-Power:LM324 U?
+L Shutdown-rescue:LM324-e-Power U?
 U 1 1 5EAE9BFA
 P 2300 2000
@@
 $EndComp
 $Comp
-L e-Power:LM324 U?
+L Shutdown-rescue:LM324-e-Power U?
 U 2 1 5EAEB674
 P 2300 1000
@@
 $EndComp
 $Comp
-L e-Power:LM324 U?
+L Shutdown-rescue:LM324-e-Power U?
 U 3 1 5EAECE19
 P 5100 1950
@@
 $EndComp
 $Comp
-L e-Power:LM324 U?
+L Shutdown-rescue:LM324-e-Power U?
 U 5 1 5EAEE4D6
 P 2250 3200
@@
 	5450 1600 5450 1650
 $Comp
-L e-Power:LM324 U?
+L Shutdown-rescue:LM324-e-Power U?
 U 4 1 5EAEDF43
 P 6800 2050
@@
 AR Path="/5ED9340F/5FB7FD92" Ref="TP?"  Part="1"
 AR Path="/5EC1D7DE/5FB7FD92" Ref="TP205"  Part="1"
+AR Path="/5F805AC0/5EC1D7DE/5FB7FD92" Ref="TP?"  Part="1"
 F 0 "TP?" H 2850 2650 50  0000 L CNN
 F 1 "2.2727V" H 2550 2500 50  0000 L CNN
@@
 AR Path="/5ED9340F/5FB877AE" Ref="TP?"  Part="1"
 AR Path="/5EC1D7DE/5FB877AE" Ref="TP201"  Part="1"
+AR Path="/5F805AC0/5EC1D7DE/5FB877AE" Ref="TP?"  Part="1"
 F 0 "TP?" H 3000 1100 50  0000 L CNN
 F 1 "1.8V" H 3000 1200 50  0000 L CNN
@@
 AR Path="/5ED9340F/5FB88B6A" Ref="TP?"  Part="1"
 AR Path="/5EC1D7DE/5FB88B6A" Ref="TP202"  Part="1"
+AR Path="/5F805AC0/5EC1D7DE/5FB88B6A" Ref="TP?"  Part="1"
 F 0 "TP?" H 5500 1350 50  0000 L CNN
 F 1 "5.000V" H 5500 1450 50  0000 L CNN
@@
 AR Path="/5ED9340F/5FB89627" Ref="TP?"  Part="1"
 AR Path="/5EC1D7DE/5FB89627" Ref="TP204"  Part="1"
+AR Path="/5F805AC0/5EC1D7DE/5FB89627" Ref="TP?"  Part="1"
 F 0 "TP?" H 6800 1550 50  0000 L CNN
 F 1 "0.850V" V 7050 1750 50  0000 L CNN
@@
 $EndComp
 $Comp
-L e-Power:TL431 U?
+L Shutdown-rescue:TL431-e-Power U?
 U 1 1 5FBA715A
 P 3400 1250
@@
 $EndComp
 $Comp
-L e-Power:TL431 U?
+L Shutdown-rescue:TL431-e-Power U?
 U 1 1 5FBA816C
 P 4100 2150
@@
 AR Path="/5ED9340F/5FC6D345" Ref="TP?"  Part="1"
 AR Path="/5EC1D7DE/5FC6D345" Ref="TP203"  Part="1"
+AR Path="/5F805AC0/5EC1D7DE/5FC6D345" Ref="TP?"  Part="1"
 F 0 "TP?" H 4700 1550 50  0000 L CNN
 F 1 "GND" H 4800 1450 50  0000 L CNN
