File: boards_unified/baseline.kicad_pcb (KiCad board)
At the start: 2 copper layers, 388 x 444 mm, 128 parts

Commit message: add small option panel board
Other:
- board text added: "Eco1.User is for rounting out 2.54mm"
- board text removed: "CMTS IS FOR ROUTING OUT"
