File: Luz de Freio/Luz de Freio.kicad_pcb (KiCad board)
At the start: 2 copper layers, 100.1 x 43.7 mm, 61 parts, among them J1 Screw_Terminal_01x02, J2 Screw_Terminal_01x02, K1 RELAY_19.1x15.5mm, Q1 Si2302DS, Q2 IRF3205, U1 MC34063AP, U2 TL431DBZ, U3 LM358

Commit message: Changed Tracks Width
Parts:
- moved TP4 0.92 mm to (198.4, 107.7)
Routing:
- net GND: track 276.4 -> 282.4 mm
- net Net-(D3-Pad3): track 34.5 -> 33.5 mm

Commit message: generate gerbers for brake light
Other:
- board text added: "> A. Araújo"
- board text removed: ">A. Araújo"
Changed lines of the file:
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@@
-(kicad_pcb (version 20171130) (host pcbnew "(5.1.4)-1")
+(kicad_pcb (version 20171130) (host pcbnew "(5.1.5)-3")
   (general
     (thickness 1.6)
@@
   )
   (setup
-    (last_trace_width 1)
+    (last_trace_width 0.25)
     (user_trace_width 0.3)
     (user_trace_width 0.4)
@@
       (outputformat 1)
       (mirror false)
-      (drillshape 1)
+      (drillshape 0)
       (scaleselection 1)
-      (outputdirectory ""))
+      (outputdirectory "GERBERS/"))
   )
   (net 0 "")
@@
     (effects (font (size 1.5 1.5) (thickness 0.3)) (justify left))
   )
-  (gr_text ">A. Araújo" (at 139 129.775 90) (layer F.SilkS)
+  (gr_text "> A. Araújo" (at 139 129.775 90) (layer F.SilkS)
     (effects (font (size 1.5 1.5) (thickness 0.3)) (justify left))
   )

Commit message: placa fdcan
Parts:
- moved G2 5.28 mm to (165.1, 99.0)
- moved G1 3.37 mm to (149.9, 99.1)
Changed lines of the file:
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@@
-(kicad_pcb (version 20171130) (host pcbnew "(5.1.5)-3")
+(kicad_pcb (version 20171130) (host pcbnew "(5.1.8)-1")
   (general
     (thickness 1.6)
@@
     (38 B.Mask user)
     (39 F.Mask user)
-    (40 Dwgs.User user)
+    (40 Dwgs.User user hide)
     (41 Cmts.User user)
     (42 Eco1.User user)
@@
     (fp_line (start 6.223 2.6) (end 7.493 2.6) (layer F.SilkS) (width 0.12))
     (fp_line (start 1.123 2.6) (end 3.937 2.6) (layer F.SilkS) (width 0.12))
-    (fp_text user %R (at 0 -3.048 90) (layer F.Fab)
-      (effects (font (size 1 1) (thickness 0.15)))
-    )
     (fp_line (start 8 -5.71) (end -3 -5.71) (layer F.CrtYd) (width 0.05))
     (fp_line (start 8 5.1) (end 8 -5.71) (layer F.CrtYd) (width 0.05))
@@
     (fp_circle (center 5.127 0) (end 6.627 0) (layer F.Fab) (width 0.1))
     (fp_circle (center 0 0) (end 1.5 0) (layer F.Fab) (width 0.1))
+    (fp_text user %R (at 0 -3.048 90) (layer F.Fab)
+      (effects (font (size 1 1) (thickness 0.15)))
+    )
     (fp_arc (start 0 0) (end -0.684 1.535) (angle -25) (layer F.SilkS) (width 0.12))
     (fp_arc (start 0 0) (end -1.535 -0.684) (angle -48) (layer F.SilkS) (width 0.12))
@@
     (fp_line (start 6.223 2.6) (end 7.493 2.6) (layer F.SilkS) (width 0.12))
     (fp_line (start 1.123 2.6) (end 3.937 2.6) (layer F.SilkS) (width 0.12))
-    (fp_text user %R (at 0 -3.048) (layer F.Fab)
-      (effects (font (size 1 1) (thickness 0.15)))
-    )
     (fp_line (start 8 -5.71) (end -3 -5.71) (layer F.CrtYd) (width 0.05))
     (fp_line (start 8 5.1) (end 8 -5.71) (layer F.CrtYd) (width 0.05))
@@
     (fp_circle (center 5.127 0) (end 6.627 0) (layer F.Fab) (width 0.1))
     (fp_circle (center 0 0) (end 1.5 0) (layer F.Fab) (width 0.1))
+    (fp_text user %R (at 0 -3.048) (layer F.Fab)
+      (effects (font (size 1 1) (thickness 0.15)))
+    )
     (fp_arc (start 0 0) (end -0.684 1.535) (angle -25) (layer F.SilkS) (width 0.12))
     (fp_arc (start 0 0) (end -1.535 -0.684) (angle -48) (layer F.SilkS) (width 0.12))
@@
     (fp_line (start 6.223 2.6) (end 7.493 2.6) (layer F.SilkS) (width 0.12))
     (fp_line (start 1.123 2.6) (end 3.937 2.6) (layer F.SilkS) (width 0.12))
-    (fp_text user %R (at 0 -3.048) (layer F.Fab)
-      (effects (font (size 1 1) (thickness 0.15)))
-    )
     (fp_line (start 8 -5.71) (end -3 -5.71) (layer F.CrtYd) (width 0.05))
     (fp_line (start 8 5.1) (end 8 -5.71) (layer F.CrtYd) (width 0.05))
@@
     (fp_circle (center 5.127 0) (end 6.627 0) (layer F.Fab) (width 0.1))
     (fp_circle (center 0 0) (end 1.5 0) (layer F.Fab) (width 0.1))
+    (fp_text user %R (at 0 -3.048) (layer F.Fab)
+      (effects (font (size 1 1) (thickness 0.15)))
+    )
     (fp_arc (start 0 0) (end -0.684 1.535) (angle -25) (layer F.SilkS) (width 0.12))
     (fp_arc (start 0 0) (end -1.535 -0.684) (angle -48) (layer F.SilkS) (width 0.12))
@@
       (effects (font (size 1 1) (thickness 0.15)))
     )
-    (fp_text user %R (at 0 0 90) (layer F.Fab)
-      (effects (font (size 0.5 0.5) (thickness 0.08)))
-    )
     (fp_line (start 1.85 0.95) (end -1.85 0.95) (layer F.CrtYd) (width 0.05))
     (fp_line (start 1.85 -0.95) (end 1.85 0.95) (layer F.CrtYd) (width 0.05))
@@
     (fp_line (start -1 -0.6) (end 1 -0.6) (layer F.Fab) (width 0.1))
     (fp_line (start -1 0.6) (end -1 -0.6) (layer F.Fab) (width 0.1))
+    (fp_text user %R (at 0 0 90) (layer F.Fab)
+      (effects (font (size 0.5 0.5) (thickness 0.08)))
+    )
     (pad 2 smd roundrect (at 1.025 0 90) (size 1.15 1.4) (layers F.Cu F.Paste F.Mask) (roundrect_rratio 0.217391)
       (net 29 "Net-(R14-Pad1)"))
@@
     (fp_text value 10K (at 0 1.65 90) (layer F.Fab)
       (effects (font (size 1 1) (thickness 0.15)))
-    )
-    (fp_text user %R (at 0 0 90) (layer F.Fab)
-      (effects (font (size 0.5 0.5) (thickness 0.08)))
     )
     (fp_line (start 1.85 0.95) (end -1.85 0.95) (layer F.CrtYd) (width 0.05))
@@
     (fp_line (start -1 -0.6) (end 1 -0.6) (layer F.Fab) (width 0.1))
     (fp_line (start -1 0.6) (end -1 -0.6) (layer F.Fab) (width 0.1))
+    (fp_text user %R (at 0 0 90) (layer F.Fab)
+      (effects (font (size 0.5 0.5) (thickness 0.08)))
+    )
     (pad 2 smd roundrect (at 1.025 0 270) (size 1.15 1.4) (layers F.Cu F.Paste F.Mask) (roundrect_rratio 0.217391)
       (net 5 "Net-(C4-Pad2)"))
@@
       (effects (font (size 1 1) (thickness 0.15)))
     )
-    (fp_text user %R (at 0 0 90) (layer F.Fab)
-      (effects (font (size 0.4 0.4) (thickness 0.06)))
-    )
     (fp_line (start 1.397 0.762) (end -1.397 0.762) (layer F.CrtYd) (width 0.05))
     (fp_line (start 1.397 -0.762) (end 1.397 0.762) (layer F.CrtYd) (width 0.05))
@@
     (fp_line (start -0.8 -0.4) (end 0.8 -0.4) (layer F.Fab) (width 0.1))
     (fp_line (start -0.8 0.4) (end -0.8 -0.4) (layer F.Fab) (width 0.1))
+    (fp_text user %R (at 0 0 90) (layer F.Fab)
+      (effects (font (size 0.4 0.4) (thickness 0.06)))
+    )
     (pad 2 smd trapezoid (at 0.9525 0 270) (size 0.7 1.3) (layers F.Cu F.Paste F.Mask)
       (net 13 "Net-(F1-Pad1)"))
@@
     (fp_line (start -0.35 0) (end -0.35 0.55) (layer F.SilkS) (width 0.1))
     (fp_line (start -0.75 0) (end -0.35 0) (layer F.SilkS) (width 0.1))
-    (fp_text user %R (at 0 -2.286 90) (layer F.Fab)
-      (effects (font (size 1 1) (thickness 0.15)))
-    )
     (fp_line (start -3.048 -1.36) (end -3.048 1.36) (layer F.SilkS) (width 0.12))
     (fp_line (start 0.25 0) (end 0.75 0) (layer F.Fab) (width 0.1))
@@
     (fp_line (start -2.286 -1.524) (end 3.048 -1.524) (layer F.CrtYd) (width 0.12))
     (fp_line (start 3.048 -1.524) (end 3.048 1.524) (layer F.CrtYd) (width 0.12))
+    (fp_text user %R (at 0 -2.286 90) (layer F.Fab)
+      (effects (font (size 1 1) (thickness 0.15)))
+    )
     (pad 1 smd rect (at -2.032 0 270) (size 1.6 2) (layers F.Cu F.Paste F.Mask)
       (net 15 "Net-(D4-Pad1)"))
@@
     (fp_line (start -0.35 0) (end -0.35 0.55) (layer F.SilkS) (width 0.1))
     (fp_line (start -0.75 0) (end -0.35 0) (layer F.SilkS) (width 0.1))
-    (fp_text user %R (at 0 -2.286) (layer F.Fab)
-      (effects (font (size 1 1) (thickness 0.15)))
-    )
     (fp_line (start -3.048 -1.36) (end -3.048 1.36) (layer F.SilkS) (width 0.12))
     (fp_line (start 0.25 0) (end 0.75 0) (layer F.Fab) (width 0.1))
@@
     (fp_line (start -2.286 -1.524) (end 3.048 -1.524) (layer F.CrtYd) (width 0.12))
     (fp_line (start 3.048 -1.524) (end 3.048 1.524) (layer F.CrtYd) (width 0.12))
+    (fp_text user %R (at 0 -2.286) (layer F.Fab)
+      (effects (font (size 1 1) (thickness 0.15)))
+    )
     (pad 1 smd rect (at -2.032 0 180) (size 1.6 2) (layers F.Cu F.Paste F.Mask)
       (net 2 +12V))
@@
     (fp_text value 100nF (at 0 0) (layer F.Fab)
       (effects (font (size 1 1) (thickness 0.15)))
-    )
-    (fp_text user %R (at 0 0) (layer F.Fab)
-      (effects (font (size 0.5 0.5) (thickness 0.08)))
     )
     (fp_line (start 1.85 0.95) (end -1.85 0.95) (layer F.CrtYd) (width 0.05))
@@
     (fp_line (start -1 -0.6) (end 1 -0.6) (layer F.Fab) (width 0.1))
     (fp_line (start -1 0.6) (end -1 -0.6) (layer F.Fab) (width 0.1))
+    (fp_text user %R (at 0 0) (layer F.Fab)
+      (effects (font (size 0.5 0.5) (thickness 0.08)))
+    )
     (pad 2 smd roundrect (at 1.025 0 180) (size 1.15 1.4) (layers F.Cu F.Paste F.Mask) (roundrect_rratio 0.217391)
       (net 1 GND))
@@
     (fp_text value 100nF (at 0 1.65 90) (layer F.Fab)
       (effects (font (size 1 1) (thickness 0.15)))
-    )
-    (fp_text user %R (at 0 0 90) (layer F.Fab)
-      (effects (font (size 0.5 0.5) (thickness 0.08)))
     )
     (fp_line (start 1.68 0.95) (end -1.68 0.95) (layer F.CrtYd) (width 0.05))
@@
     (fp_line (start -1 -0.6) (end 1 -0.6) (layer F.Fab) (width 0.1))
     (fp_line (start -1 0.6) (end -1 -0.6) (layer F.Fab) (width 0.1))
+    (fp_text user %R (at 0 0 90) (layer F.Fab)
+      (effects (font (size 0.5 0.5) (thickness 0.08)))
+    )
     (pad 2 smd roundrect (at 0.9375 0 270) (size 0.975 1.4) (layers F.Cu F.Paste F.Mask) (roundrect_rratio 0.25)
       (net 25 "Net-(C8-Pad2)"))
@@
       (effects (font (size 1 1) (thickness 0.15)))
     )
-    (fp_text user %R (at 0 0) (layer F.Fab)
-      (effects (font (size 0.98 0.98) (thickness 0.15)))
-    )
     (fp_line (start 0 2.56) (end 1.95 2.56) (layer F.SilkS) (width 0.12))
     (fp_line (start 0 2.56) (end -1.95 2.56) (layer F.SilkS) (width 0.12))
@@
     (fp_line (start 3.7 2.7) (end 3.7 -2.7) (layer F.CrtYd) (width 0.05))
     (fp_line (start 3.7 -2.7) (end -3.7 -2.7) (layer F.CrtYd) (width 0.05))
+    (fp_text user %R (at 0 0) (layer F.Fab)
+      (effects (font (size 0.98 0.98) (thickness 0.15)))
+    )
     (pad 8 smd roundrect (at 2.475 -1.905 180) (size 1.95 0.6) (layers F.Cu F.Paste F.Mask) (roundrect_rratio 0.25)
       (net 20 "Net-(R2-Pad1)"))
@@
   )
   (module e-Power:Logo_UFRGS_14.7x8.0mm_SilkS (layer F.Cu)
-    (at 153.2 99.475)
+    (at 149.86 99.06)
     (tags "logo UFRGS")
     (attr virtual)
@@
   )
   (module e-Power:Logo_e-Power_16.5x8.0mm_SilkS (layer F.Cu)
-    (at 170.375 98.975)
+    (at 165.1 98.975)
     (attr virtual)
     (fp_text reference G2 (at -5.08 -3.81) (layer F.SilkS) hide
