File: BMS_temperatura/temperature_sensors.sch (KiCad schematic (older format))
At the start: 0 parts

Commit message: layout final bms temp
Parts:
- added J1: TEMP_IDC_26_CONN, Connector_IDC:IDC-Header_2x13_P2.54mm_Horizontal, symbol Connector:Conn_01x26_Female
Connections:
- net TS_1: now also J1.25 (Pin_25)
- net TS_10: now also J1.22 (Pin_22)
- net TS_11: now also J1.19 (Pin_19)
- net TS_12: now also J1.20 (Pin_20)
- net TS_13: now also J1.14 (Pin_14)
- net TS_14: now also J1.13 (Pin_13)
- net TS_15: now also J1.3 (Pin_3)
- net TS_16: now also J1.4 (Pin_4)
- net TS_17: now also J1.12 (Pin_12)
- net TS_18: now also J1.11 (Pin_11)
- net TS_19: now also J1.5 (Pin_5)
- net TS_2: now also J1.26 (Pin_26)
- net TS_20: now also J1.6 (Pin_6)
- net TS_21: now also J1.10 (Pin_10)
- net TS_22: now also J1.9 (Pin_9)
- net TS_23: now also J1.7 (Pin_7)
- net TS_24: now also J1.8 (Pin_8)
- net TS_3: now also J1.15 (Pin_15)
- net TS_4: now also J1.16 (Pin_16)
- net TS_5: now also J1.23 (Pin_23)
- net TS_6: now also J1.24 (Pin_24)
- net TS_7: now also J1.17 (Pin_17)
- net TS_8: now also J1.18 (Pin_18)
- net TS_9: now also J1.21 (Pin_21)
- new net GND: J1.1 (Pin_1), J1.2 (Pin_2)
Changed lines of the file:
@@
 Text HLabel 5550 2200 2    50   Output ~ 0
 T18
+$Comp
+L Connector:Conn_01x26_Female J1
+U 1 1 60562961
+P 7450 2250
+F 0 "J1" H 7478 2226 50  0000 L CNN
+F 1 "TEMP_IDC_26_CONN" H 6800 850 50  0000 L CNN
+F 2 "Connector_IDC:IDC-Header_2x13_P2.54mm_Horizontal" H 7450 2250 50  0001 C CNN
+F 3 "~" H 7450 2250 50  0001 C CNN
+	1    7450 2250
+	1    0    0    -1
+$EndComp
+Wire Wire Line
+	7150 3450 7250 3450
+Text HLabel 7150 3450 0    50   Input ~ 0
+TS_1
+Wire Wire Line
+	7150 3550 7250 3550
+Text HLabel 7150 3550 0    50   Input ~ 0
+TS_2
+Wire Wire Line
+	7150 3350 7250 3350
+Text HLabel 7150 3350 0    50   Input ~ 0
+TS_6
+Wire Wire Line
+	7150 3250 7250 3250
+Text HLabel 7150 3250 0    50   Input ~ 0
+TS_5
+Wire Wire Line
+	7150 3150 7250 3150
+Text HLabel 7150 3150 0    50   Input ~ 0
+TS_10
+Wire Wire Line
+	7150 3050 7250 3050
+Text HLabel 7150 3050 0    50   Input ~ 0
+TS_9
+Wire Wire Line
+	7150 2950 7250 2950
+Text HLabel 7150 2950 0    50   Input ~ 0
+TS_12
+Wire Wire Line
+	7150 2850 7250 2850
+Text HLabel 7150 2850 0    50   Input ~ 0
+TS_11
+Wire Wire Line
+	7150 2750 7250 2750
+Text HLabel 7150 2750 0    50   Input ~ 0
+TS_8
+Wire Wire Line
+	7150 2650 7250 2650
+Text HLabel 7150 2650 0    50   Input ~ 0
+TS_7
+Wire Wire Line
+	7150 2550 7250 2550
+Wire Wire Line
+	7150 2450 7250 2450
+Text HLabel 7150 2450 0    50   Input ~ 0
+TS_3
+Wire Wire Line
+	7150 2350 7250 2350
+Text HLabel 7150 2350 0    50   Input ~ 0
+TS_13
+Wire Wire Line
+	7150 2250 7250 2250
+Text HLabel 7150 2250 0    50   Input ~ 0
+TS_14
+Wire Wire Line
+	7150 2150 7250 2150
+Text HLabel 7150 2150 0    50   Input ~ 0
+TS_17
+Wire Wire Line
+	7150 2050 7250 2050
+Text HLabel 7150 2050 0    50   Input ~ 0
+TS_18
+Wire Wire Line
+	7150 1950 7250 1950
+Text HLabel 7150 1950 0    50   Input ~ 0
+TS_21
+Wire Wire Line
+	7150 1850 7250 1850
+Wire Wire Line
+	7150 1750 7250 1750
+Text HLabel 7150 1750 0    50   Input ~ 0
+TS_24
+Wire Wire Line
+	7150 1650 7250 1650
+Text HLabel 7150 1650 0    50   Input ~ 0
+TS_23
+Wire Wire Line
+	7150 1550 7250 1550
+Text HLabel 7150 1550 0    50   Input ~ 0
+TS_20
+Wire Wire Line
+	7150 1450 7250 1450
+Text HLabel 7150 1450 0    50   Input ~ 0
+TS_19
+Wire Wire Line
+	7150 1350 7250 1350
+Text HLabel 7150 1350 0    50   Input ~ 0
+TS_16
+Wire Wire Line
+	7150 1250 7250 1250
+Text HLabel 7150 1250 0    50   Input ~ 0
+TS_15
+Wire Wire Line
+	7150 1150 7250 1150
+Text HLabel 7150 2550 0    50   Input ~ 0
+TS_4
+$Comp
+L power:GND #PWR?
+U 1 1 60567A6E
+P 7050 1050
+AR Path="/5EA47040/60567A6E" Ref="#PWR?"  Part="1"
+AR Path="/5EA471BF/60567A6E" Ref="#PWR?"  Part="1"
+AR Path="/5EEF4361/60567A6E" Ref="#PWR?"  Part="1"
+AR Path="/5EEF524D/60567A6E" Ref="#PWR?"  Part="1"
+AR Path="/5EC044AE/5EC054C7/60567A6E" Ref="#PWR?"  Part="1"
+AR Path="/5EC044AE/5EC39151/60567A6E" Ref="#PWR?"  Part="1"
+AR Path="/5EC24961/5EC054C7/60567A6E" Ref="#PWR?"  Part="1"
+AR Path="/5EC24961/5EC3A225/60567A6E" Ref="#PWR?"  Part="1"
+AR Path="/5EC24961/5EC4031A/60567A6E" Ref="#PWR?"  Part="1"
+AR Path="/5EC24961/5EC462FD/60567A6E" Ref="#PWR?"  Part="1"
+AR Path="/5EC24961/5EC4BDFE/60567A6E" Ref="#PWR?"  Part="1"
+AR Path="/5EC24961/5EC51A1F/60567A6E" Ref="#PWR?"  Part="1"
+AR Path="/5EC24961/5EC574F6/60567A6E" Ref="#PWR?"  Part="1"
+AR Path="/5EC24961/5EC5D2D3/60567A6E" Ref="#PWR?"  Part="1"
+AR Path="/5EC24961/5EC62E5E/60567A6E" Ref="#PWR?"  Part="1"
+AR Path="/5EC24961/5EC6897D/60567A6E" Ref="#PWR?"  Part="1"
+AR Path="/5EC24961/5EC6E4EA/60567A6E" Ref="#PWR?"  Part="1"
+AR Path="/5EC24961/5EC74033/60567A6E" Ref="#PWR?"  Part="1"
+AR Path="/5EC24961/5EC79B70/60567A6E" Ref="#PWR?"  Part="1"
+AR Path="/5EC24961/5EC7F6A7/60567A6E" Ref="#PWR?"  Part="1"
+AR Path="/5EC24961/5EC85226/60567A6E" Ref="#PWR?"  Part="1"
+AR Path="/5EC24961/5F2675E0/60567A6E" Ref="#PWR?"  Part="1"
+AR Path="/5EC24961/5F26D4B2/60567A6E" Ref="#PWR?"  Part="1"
+AR Path="/5EC24961/5F646961/60567A6E" Ref="#PWR?"  Part="1"
+AR Path="/5EC24961/5F656EA4/60567A6E" Ref="#PWR?"  Part="1"
+AR Path="/5EC24961/5F675FE6/60567A6E" Ref="#PWR?"  Part="1"
+AR Path="/5EC24961/5F67B671/60567A6E" Ref="#PWR?"  Part="1"
+AR Path="/5EC24961/5F6A1F0B/60567A6E" Ref="#PWR?"  Part="1"
+AR Path="/5EC24961/60567A6E" Ref="#PWR0103"  Part="1"
+F 0 "#PWR0103" H 7050 800 50  0001 C CNN
+F 1 "GND" V 7150 1050 50  0000 C CNN
+F 2 "" H 7050 1050 50  0001 C CNN
+F 3 "" H 7050 1050 50  0001 C CNN
+	1    7050 1050
+	0    1    1    0
+$EndComp
+Wire Wire Line
+	7050 1050 7150 1050
+Wire Wire Line
+	7150 1150 7150 1050
+Connection ~ 7150 1050
+Wire Wire Line
+	7150 1050 7250 1050
+Text HLabel 7150 1850 0    50   Input ~ 0
+TS_22
 $EndSCHEMATC

Commit message: Add files via upload
Divisor de tensão
Parts:
- J1: symbol Connector:Conn_01x26_Female -> BMS_temperatura-rescue:Conn_01x26_Female-Connector
Changed lines of the file:
@@
 T18
 $Comp
-L Connector:Conn_01x26_Female J1
+L BMS_temperatura-rescue:Conn_01x26_Female-Connector J1
 U 1 1 60562961
 P 7450 2250
@@
 TS_4
 $Comp
-L power:GND #PWR?
+L BMS_temperatura-rescue:GND-power #PWR?
 U 1 1 60567A6E
 P 7050 1050
