File: BMS_temperatura/voltage_references.sch (KiCad schematic (older format))
At the start: 12 parts, among them U201 LM324, U203 TL431

Commit message: layout att.1
Parts:
- gave numbers to parts that had none: 1
Changed lines of the file:
@@
 P 2900 2050
 AR Path="/5ED9340F/6193203A" Ref="TP?"  Part="1"
-AR Path="/5EC1D7DE/6193203A" Ref="TP?"  Part="1"
-F 0 "TP?" H 2850 2250 50  0000 L CNN
+AR Path="/5EC1D7DE/6193203A" Ref="TP23"  Part="1"
+F 0 "TP23" H 2850 2250 50  0000 L CNN
 F 1 "2.2727V" H 2550 2100 50  0000 L CNN
 F 2 "e-Power:TestPoint_Pad_D1.0mm" H 3100 2050 50  0001 C CNN

Commit message: Add files via upload
Divisor de tensão
Parts:
- C205, C206, C207, C208, C211: symbol Device:C -> BMS_temperatura-rescue:C-Device
- R201, R210, R229, R230: symbol Device:R -> BMS_temperatura-rescue:R-Device
- TP23: symbol Connector:TestPoint -> BMS_temperatura-rescue:TestPoint-Connector
- U201: symbol e-Power:LM324 -> BMS_temperatura-rescue:LM324-e-Power
- U203: symbol Reference_Voltage:TL432DBZ -> BMS_temperatura-rescue:TL432DBZ-Reference_Voltage
Changed lines of the file:
@@
 $EndDescr
 $Comp
-L Device:R R201
+L BMS_temperatura-rescue:R-Device R201
 U 1 1 5EAE3031
 P 1000 950
@@
 2.2727V
 $Comp
-L e-Power:LM324 U201
+L BMS_temperatura-rescue:LM324-e-Power U201
 U 1 1 5EAE9BFA
 P 2300 2000
@@
 $EndComp
 $Comp
-L power:+5V #PWR0201
+L BMS_temperatura-rescue:+5V-power #PWR0201
 U 1 1 5EB89179
 P 1000 750
@@
 $EndComp
 $Comp
-L Device:R R210
+L BMS_temperatura-rescue:R-Device R210
 U 1 1 5EB8AA78
 P 1000 1300
@@
 $EndComp
 $Comp
-L power:GND #PWR0208
+L BMS_temperatura-rescue:GND-power #PWR0208
 U 1 1 5EB8BCC6
 P 1000 1850
@@
 	1000 1500 1000 1550
 $Comp
-L Device:C C206
+L BMS_temperatura-rescue:C-Device C206
 U 1 1 5EB8E025
 P 850 1650
@@
 $EndComp
 $Comp
-L Device:C C205
+L BMS_temperatura-rescue:C-Device C205
 U 1 1 5EB8ED80
 P 650 1650
@@
 2.5V
 $Comp
-L power:GND #PWR0212
+L BMS_temperatura-rescue:GND-power #PWR0212
 U 1 1 5EB956D1
 P 2300 2400
@@
 $EndComp
 $Comp
-L Device:R R229
+L BMS_temperatura-rescue:R-Device R229
 U 1 1 5EBB0544
 P 1650 2400
@@
 $EndComp
 $Comp
-L Device:R R230
+L BMS_temperatura-rescue:R-Device R230
 U 1 1 5EBB1776
 P 2050 2400
@@
 	1150 2400 1500 2400
 $Comp
-L Device:C C208
+L BMS_temperatura-rescue:C-Device C208
 U 1 1 5EBBB1C2
 P 1550 2100
@@
 $EndComp
 $Comp
-L Device:C C207
+L BMS_temperatura-rescue:C-Device C207
 U 1 1 5EBBBF29
 P 1550 1900
@@
 $EndComp
 $Comp
-L power:GND #PWR0210
+L BMS_temperatura-rescue:GND-power #PWR0210
 U 1 1 5EBBC902
 P 1300 2150
@@
 2.2727V
 $Comp
-L power:+12V #PWR0214
+L BMS_temperatura-rescue:+12V-power #PWR0214
 U 1 1 5ED9B422
 P 2650 3000
@@
 $EndComp
 $Comp
-L power:GND #PWR0215
+L BMS_temperatura-rescue:GND-power #PWR0215
 U 1 1 5ED9CE9B
 P 1850 3100
@@
 $EndComp
 $Comp
-L Device:C C211
+L BMS_temperatura-rescue:C-Device C211
 U 1 1 5ED9DBAA
 P 2650 3300
@@
 Connection ~ 1850 1900
 $Comp
-L power:GND #PWR0216
+L BMS_temperatura-rescue:GND-power #PWR0216
 U 1 1 5ED9FCD3
 P 2650 3500
@@
 $EndComp
 $Comp
-L e-Power:LM324 U201
+L BMS_temperatura-rescue:LM324-e-Power U201
 U 5 1 5EAEE4D6
 P 2250 3200
@@
 	2900 2000 2950 2000
 $Comp
-L Reference_Voltage:TL432DBZ U203
+L BMS_temperatura-rescue:TL432DBZ-Reference_Voltage U203
 U 1 1 5FB99557
 P 1000 1650
@@
 	2650 2000 2900 2000
 $Comp
-L Connector:TestPoint TP?
+L BMS_temperatura-rescue:TestPoint-Connector TP?
 U 1 1 6193203A
 P 2900 2050
