File: Charger_Shutdown/Charger_Shuwdown.sch (KiCad schematic (older format))
At the start: 39 parts, among them J1 BMS, J2 CHARGER_SHTDNW, J3 IMD, J8 voltage supply, K4 RELAY_19.1x15.5mm, K5 RELAY_19.1x15.5mm, Q1 MMBT5551, Q3 MMBT5551, Q4 Si2302DS, Q5 Si2302DS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

Commit message: charger atualizacao
Parts:
- removed C4: 10nF, Capacitor_SMD:C_0805_2012Metric, symbol Device:C
- removed C5: 220uF, Capacitor_SMD:CP_Elec_8x10, symbol Device:CP
- removed D6: SS54HF, e-Power:DO-214AC, symbol e-Power:1N5819
- added J5: IMD_SHTDNW, e-Power:TerminalBlock_Phoenix_MKDS-1,5-2_1x02_P5.08mm_Horizontal, symbol Connector:Screw_Terminal_01x02
- J2: value CHARGER_SHTDNW -> BMS_SHTDNW
- renumbered J8 to J4
Connections:
- net Input_Power: now also F1.1
- net at K5.1: now also J2.2 (Pin_2); no longer K4.4
- net at K4.1: now also J5.2 (Pin_2); no longer J2.2 (Pin_2)
- new net: J5.1 (Pin_1), K4.4
Other:
- moved on the sheet: C3, F1, J2, TP10, TP2
Changed lines of the file:
@@
 	3700 4250 3700 4500
 NoConn ~ 3400 2000
-Wire Wire Line
-	4500 1300 4500 1400
 Wire Notes Line
 	800  3100 800  5400
@@
 	800  750  800  3000
 $Comp
-L power:GND #PWR0108
-U 1 1 5F0D3617
-P 10300 1750
-F 0 "#PWR0108" H 10300 1500 50  0001 C CNN
-F 1 "GND" H 10305 1577 50  0000 C CNN
-F 2 "" H 10300 1750 50  0001 C CNN
-F 3 "" H 10300 1750 50  0001 C CNN
-	1    10300 1750
-	1    0    0    -1
-$EndComp
-$Comp
 L power:GND #PWR0109
 U 1 1 5F0E50A5
-P 9900 1750
-F 0 "#PWR0109" H 9900 1500 50  0001 C CNN
-F 1 "GND" H 9905 1577 50  0000 C CNN
-F 2 "" H 9900 1750 50  0001 C CNN
-F 3 "" H 9900 1750 50  0001 C CNN
-	1    9900 1750
-	1    0    0    -1
-$EndComp
-$Comp
-L power:GND #PWR0110
-U 1 1 5F0E51BF
-P 10650 1750
-F 0 "#PWR0110" H 10650 1500 50  0001 C CNN
-F 1 "GND" H 10655 1577 50  0000 C CNN
-F 2 "" H 10650 1750 50  0001 C CNN
-F 3 "" H 10650 1750 50  0001 C CNN
-	1    10650 1750
+P 9150 1500
+F 0 "#PWR0109" H 9150 1250 50  0001 C CNN
+F 1 "GND" H 9155 1327 50  0000 C CNN
+F 2 "" H 9150 1500 50  0001 C CNN
+F 3 "" H 9150 1500 50  0001 C CNN
+	1    9150 1500
 	1    0    0    -1
 $EndComp
@@
 L Device:C C3
 U 1 1 5F0E535B
-P 9900 1600
-F 0 "C3" H 9900 1700 50  0000 L CNN
-F 1 "100nF" H 9900 1500 50  0000 L CNN
-F 2 "Capacitor_SMD:C_0805_2012Metric" H 9938 1450 50  0001 C CNN
-F 3 "~" H 9900 1600 50  0001 C CNN
-	1    9900 1600
-	1    0    0    -1
-$EndComp
-$Comp
-L Device:C C4
-U 1 1 5F0E5904
-P 10300 1600
-F 0 "C4" H 10300 1700 50  0000 L CNN
-F 1 "10nF" H 10300 1500 50  0000 L CNN
-F 2 "Capacitor_SMD:C_0805_2012Metric" H 10338 1450 50  0001 C CNN
-F 3 "~" H 10300 1600 50  0001 C CNN
-	1    10300 1600
-	1    0    0    -1
-$EndComp
-$Comp
-L Device:CP C5
-U 1 1 5F0E5A69
-P 10650 1600
-F 0 "C5" H 10500 1650 50  0000 R CNN
-F 1 "220uF" H 10500 1550 50  0000 R CNN
-F 2 "Capacitor_SMD:CP_Elec_8x10" H 10688 1450 50  0001 C CNN
-F 3 "~" H 10650 1600 50  0001 C CNN
-	1    10650 1600
-	-1   0    0    -1
+P 9150 1350
+F 0 "C3" H 9150 1450 50  0000 L CNN
+F 1 "100nF" H 9150 1250 50  0000 L CNN
+F 2 "Capacitor_SMD:C_0805_2012Metric" H 9188 1200 50  0001 C CNN
+F 3 "~" H 9150 1350 50  0001 C CNN
+	1    9150 1350
+	1    0    0    -1
 $EndComp
 $Comp
 L e-Power:Fuse_1206 F1
 U 1 1 5F0E7C9E
-P 9200 1200
-F 0 "F1" V 9400 1150 50  0000 L CNN
-F 1 "Fuse_1206" V 9300 1000 50  0000 L CNN
-F 2 "e-Power:FUSE_1206_3216Metric" V 9130 1200 50  0001 C CNN
-F 3 "" H 9200 1200 50  0001 C CNN
-	1    9200 1200
+P 8700 1150
+F 0 "F1" V 8800 1100 50  0000 L CNN
+F 1 "Fuse_1206" V 8600 950 50  0000 L CNN
+F 2 "e-Power:FUSE_1206_3216Metric" V 8630 1150 50  0001 C CNN
+F 3 "" H 8700 1150 50  0001 C CNN
+	1    8700 1150
 	0    -1   -1   0
 $EndComp
-Wire Wire Line
-	9900 1450 10100 1450
-Wire Wire Line
-	10100 1200 10100 1450
-Connection ~ 10100 1450
-Wire Wire Line
-	10100 1450 10300 1450
-Connection ~ 10100 1200
-Wire Wire Line
-	10100 1200 10650 1200
-Wire Wire Line
-	10650 1200 10650 1450
 $Comp
 L Connector:Screw_Terminal_01x02 J1
@@
 $EndComp
 $Comp
-L Connector:Screw_Terminal_01x02 J8
+L Connector:Screw_Terminal_01x02 J4
 U 1 1 5F372D5C
 P 8400 1950
-F 0 "J8" H 8400 1650 50  0000 C CNN
+F 0 "J4" H 8400 1650 50  0000 C CNN
 F 1 "voltage supply" H 8350 1750 50  0000 C CNN
 F 2 "e-Power:TerminalBlock_Phoenix_MKDS-1,5-2_1x02_P5.08mm_Horizontal" H 8400 1950 50  0001 C CNN
@@
 L power:+12V #PWR0117
 U 1 1 5F2696FA
-P 10100 1100
-F 0 "#PWR0117" H 10100 950 50  0001 C CNN
-F 1 "+12V" H 10115 1273 50  0000 C CNN
-F 2 "" H 10100 1100 50  0001 C CNN
-F 3 "" H 10100 1100 50  0001 C CNN
-	1    10100 1100
-	1    0    0    -1
-$EndComp
-Wire Wire Line
-	10100 1200 10100 1100
+P 9150 1050
+F 0 "#PWR0117" H 9150 900 50  0001 C CNN
+F 1 "+12V" H 9165 1223 50  0000 C CNN
+F 2 "" H 9150 1050 50  0001 C CNN
+F 3 "" H 9150 1050 50  0001 C CNN
+	1    9150 1050
+	1    0    0    -1
+$EndComp
+Wire Wire Line
+	9150 1150 9150 1050
 Text GLabel 8950 1850 2    50   Input ~ 0
 Input_Power
-Text GLabel 8550 1200 0    50   Input ~ 0
+Text GLabel 8350 1150 0    50   Input ~ 0
 Input_Power
 $Comp
@@
 L Connector:TestPoint TP2
 U 1 1 5F3C6F55
-P 10650 1100
-F 0 "TP2" H 10708 1218 50  0000 L CNN
-F 1 "+12V" H 10708 1127 50  0000 L CNN
-F 2 "e-Power:TestPoint_Pad_D1.0mm" H 10850 1100 50  0001 C CNN
-F 3 "~" H 10850 1100 50  0001 C CNN
-	1    10650 1100
-	1    0    0    -1
-$EndComp
-Wire Wire Line
-	10650 1100 10650 1200
-Connection ~ 10650 1200
+P 9400 1050
+F 0 "TP2" H 9458 1168 50  0000 L CNN
+F 1 "+12V" H 9458 1077 50  0000 L CNN
+F 2 "e-Power:TestPoint_Pad_D1.0mm" H 9600 1050 50  0001 C CNN
+F 3 "~" H 9600 1050 50  0001 C CNN
+	1    9400 1050
+	1    0    0    -1
+$EndComp
+Wire Wire Line
+	9400 1050 9400 1150
 $Comp
 L Transistor_BJT:MMBT3904 Q3
@@
 $EndComp
 $Comp
-L e-Power:1N5819 D6
-U 1 1 5F598BC8
-P 8850 1200
-F 0 "D6" H 8800 1100 50  0000 L CNN
-F 1 "SS54HF" H 8700 1300 50  0000 L CNN
-F 2 "e-Power:DO-214AC" H 8850 1025 50  0001 C CNN
-F 3 "" H 8850 1200 50  0001 C CNN
-	1    8850 1200
-	-1   0    0    1
-$EndComp
-$Comp
 L Transistor_BJT:MMBT3904 Q1
 U 1 1 5F5A0EDA
@@
 $EndComp
 Wire Wire Line
-	8550 1200 8600 1200
+	8350 1150 8400 1150
 $Comp
 L Connector:TestPoint TP10
 U 1 1 5F7019CB
-P 8600 1050
-F 0 "TP10" H 8658 1168 50  0000 L CNN
-F 1 "+VIN" H 8658 1077 50  0000 L CNN
-F 2 "e-Power:TestPoint_Pad_D1.0mm" H 8800 1050 50  0001 C CNN
-F 3 "~" H 8800 1050 50  0001 C CNN
-	1    8600 1050
-	1    0    0    -1
-$EndComp
-Wire Wire Line
-	8600 1050 8600 1200
-Connection ~ 8600 1200
-Wire Wire Line
-	8600 1200 8700 1200
+P 8400 1000
+F 0 "TP10" H 8458 1118 50  0000 L CNN
+F 1 "+VIN" H 8458 1027 50  0000 L CNN
+F 2 "e-Power:TestPoint_Pad_D1.0mm" H 8600 1000 50  0001 C CNN
+F 3 "~" H 8600 1000 50  0001 C CNN
+	1    8400 1000
+	1    0    0    -1
+$EndComp
+Wire Wire Line
+	8400 1000 8400 1150
+Connection ~ 8400 1150
 $Comp
 L Connector:TestPoint TP3
@@
 	1500 1600 1500 2250
 Connection ~ 1500 2250
-Wire Wire Line
-	9000 1200 9050 1200
-$Comp
-L power:GND #PWR0107
-U 1 1 5F882C8C
-P 10300 1750
-F 0 "#PWR0107" H 10300 1500 50  0001 C CNN
-F 1 "GND" H 10305 1577 50  0000 C CNN
-F 2 "" H 10300 1750 50  0001 C CNN
-F 3 "" H 10300 1750 50  0001 C CNN
-	1    10300 1750
-	1    0    0    -1
-$EndComp
-Connection ~ 10300 1750
 NoConn ~ 9150 2350
 NoConn ~ 9350 2350
 Wire Wire Line
-	9350 1200 10100 1200
+	8850 1150 9150 1150
 Connection ~ 2950 2350
 Wire Wire Line
@@
 L Connector:Screw_Terminal_01x02 J2
 U 1 1 61594DD1
-P 5050 4400
-F 0 "J2" V 5014 4212 50  0000 R CNN
-F 1 "CHARGER_SHTDNW" V 5150 4600 50  0000 R CNN
-F 2 "e-Power:TerminalBlock_Phoenix_MKDS-1,5-2_1x02_P5.08mm_Horizontal" H 5050 4400 50  0001 C CNN
-F 3 "~" H 5050 4400 50  0001 C CNN
-	1    5050 4400
+P 4700 3550
+F 0 "J2" V 4664 3362 50  0000 R CNN
+F 1 "BMS_SHTDNW" V 4800 3750 50  0000 R CNN
+F 2 "e-Power:TerminalBlock_Phoenix_MKDS-1,5-2_1x02_P5.08mm_Horizontal" H 4700 3550 50  0001 C CNN
+F 3 "~" H 4700 3550 50  0001 C CNN
+	1    4700 3550
+	0    1    -1   0
+$EndComp
+$Comp
+L e-Power:RELAY_19.1x15.5mm K5
+U 1 1 5F46E112
+P 4400 4100
+F 0 "K5" H 4450 3850 50  0000 R CNN
+F 1 "RELAY_19.1x15.5mm" H 4750 4600 50  0001 R CNN
+F 2 "e-Power:Relay_SPDT_SANYOU_SRD" H 5670 4070 50  0001 C CNN
+F 3 "" H 4400 4100 50  0001 C CNN
+	1    4400 4100
 	1    0    0    1
 $EndComp
+Wire Wire Line
+	3700 3800 4200 3800
+Wire Wire Line
+	4200 4500 4200 4400
+Wire Wire Line
+	3700 4500 4200 4500
 $Comp
 L e-Power:RELAY_19.1x15.5mm K4
@@
 	1    0    0    1
 $EndComp
-$Comp
-L e-Power:RELAY_19.1x15.5mm K5
-U 1 1 5F46E112
-P 4400 4100
-F 0 "K5" H 4450 3850 50  0000 R CNN
-F 1 "RELAY_19.1x15.5mm" H 4750 4600 50  0001 R CNN
-F 2 "e-Power:Relay_SPDT_SANYOU_SRD" H 5670 4070 50  0001 C CNN
-F 3 "" H 4400 4100 50  0001 C CNN
-	1    4400 4100
-	1    0    0    1
-$EndComp
-Wire Wire Line
-	4850 4300 4850 1300
-Wire Wire Line
-	4600 2000 4600 3800
-Wire Wire Line
-	3700 3800 4200 3800
-Wire Wire Line
-	4200 4500 4200 4400
-Wire Wire Line
-	3700 4500 4200 4500
-Wire Wire Line
-	4500 1300 4850 1300
+Wire Wire Line
+	4850 4400 4850 3750
+Wire Wire Line
+	4850 3750 4700 3750
+Wire Wire Line
+	4600 3750 4600 3800
+$Comp
+L Connector:Screw_Terminal_01x02 J5
+U 1 1 614B3CEC
+P 4600 1150
+F 0 "J5" V 4564 962 50  0000 R CNN
+F 1 "IMD_SHTDNW" V 4700 1350 50  0000 R CNN
+F 2 "e-Power:TerminalBlock_Phoenix_MKDS-1,5-2_1x02_P5.08mm_Horizontal" H 4600 1150 50  0001 C CNN
+F 3 "~" H 4600 1150 50  0001 C CNN
+	1    4600 1150
+	0    1    -1   0
+$EndComp
+Wire Wire Line
+	4500 1350 4500 1400
+Wire Wire Line
+	4600 2000 4750 2000
+Wire Wire Line
+	4750 2000 4750 1350
+Wire Wire Line
+	4750 1350 4600 1350
+Wire Wire Line
+	8400 1150 8550 1150
+Connection ~ 9150 1150
+Wire Wire Line
+	9150 1150 9400 1150
+Wire Wire Line
+	9150 1150 9150 1200
 $EndSCHEMATC
